File: mikrobus.kicad_sch (KiCad schematic)
At the start: 1 part, among them CON1 MIKROBUS_HOST_CONN

Commit message: additional sheets added
Connections:
- net SDA: now reaches CON1.P11 (SDA)
- net SCL: now reaches CON1.P12 (SCL)
- net TX: now reaches CON1.P13 (TX)
- net RX: now reaches CON1.P14 (RX)
- net INT: now reaches CON1.P15 (INT)
- net PWM: now reaches CON1.P16 (PWM)
- net RST: now reaches CON1.P2 (RST)
- net CS: now reaches CON1.P3 (CS)
- net SCK: now reaches CON1.P4 (SCK)
- net MISO: now reaches CON1.P5 (MISO)
- net MOSI: now reaches CON1.P6 (MOSI)
- no-connect marks 1 -> 2
Changed lines of the file:
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@@
   (paper "A4")
   (no_connect (at 157.48 97.79))
+  (no_connect (at 119.38 67.31))
+  (wire (pts (xy 157.48 72.39) (xy 168.91 72.39))
+    (stroke (width 0) (type default) (color 0 0 0 0))
+  )
+  (wire (pts (xy 109.22 72.39) (xy 119.38 72.39))
+    (stroke (width 0) (type default) (color 0 0 0 0))
+  )
   (wire (pts (xy 160.02 102.87) (xy 157.48 102.87))
+    (stroke (width 0) (type default) (color 0 0 0 0))
+  )
+  (wire (pts (xy 157.48 77.47) (xy 168.91 77.47))
+    (stroke (width 0) (type default) (color 0 0 0 0))
+  )
+  (wire (pts (xy 157.48 82.55) (xy 168.91 82.55))
+    (stroke (width 0) (type default) (color 0 0 0 0))
+  )
+  (wire (pts (xy 109.22 87.63) (xy 119.38 87.63))
+    (stroke (width 0) (type default) (color 0 0 0 0))
+  )
+  (wire (pts (xy 109.22 82.55) (xy 119.38 82.55))
     (stroke (width 0) (type default) (color 0 0 0 0))
   )
@@
     (stroke (width 0) (type default) (color 0 0 0 0))
   )
+  (wire (pts (xy 109.22 92.71) (xy 119.38 92.71))
+    (stroke (width 0) (type default) (color 0 0 0 0))
+  )
+  (wire (pts (xy 157.48 92.71) (xy 168.91 92.71))
+    (stroke (width 0) (type default) (color 0 0 0 0))
+  )
+  (wire (pts (xy 157.48 67.31) (xy 168.91 67.31))
+    (stroke (width 0) (type default) (color 0 0 0 0))
+  )
+  (wire (pts (xy 109.22 77.47) (xy 119.38 77.47))
+    (stroke (width 0) (type default) (color 0 0 0 0))
+  )
+  (wire (pts (xy 157.48 87.63) (xy 168.91 87.63))
+    (stroke (width 0) (type default) (color 0 0 0 0))
+  )
   (wire (pts (xy 116.84 102.87) (xy 116.84 105.41))
     (stroke (width 0) (type default) (color 0 0 0 0))
   )
+  (hierarchical_label "SCL" (shape bidirectional) (at 168.91 87.63 0)
+    (effects (font (size 1.27 1.27)) (justify left))
+  )
+  (hierarchical_label "SDA" (shape bidirectional) (at 168.91 92.71 0)
+    (effects (font (size 1.27 1.27)) (justify left))
+  )
+  (hierarchical_label "MOSI" (shape input) (at 109.22 92.71 180)
+    (effects (font (size 1.27 1.27)) (justify right))
+  )
+  (hierarchical_label "PWM" (shape input) (at 168.91 67.31 0)
+    (effects (font (size 1.27 1.27)) (justify left))
+  )
+  (hierarchical_label "TX" (shape output) (at 168.91 82.55 0)
+    (effects (font (size 1.27 1.27)) (justify left))
+  )
+  (hierarchical_label "SCK" (shape input) (at 109.22 82.55 180)
+    (effects (font (size 1.27 1.27)) (justify right))
+  )
+  (hierarchical_label "RX" (shape input) (at 168.91 77.47 0)
+    (effects (font (size 1.27 1.27)) (justify left))
+  )
+  (hierarchical_label "INT" (shape output) (at 168.91 72.39 0)
+    (effects (font (size 1.27 1.27)) (justify left))
+  )
+  (hierarchical_label "RST" (shape input) (at 109.22 72.39 180)
+    (effects (font (size 1.27 1.27)) (justify right))
+  )
+  (hierarchical_label "MISO" (shape output) (at 109.22 87.63 180)
+    (effects (font (size 1.27 1.27)) (justify right))
+  )
+  (hierarchical_label "CS" (shape input) (at 109.22 77.47 180)
+    (effects (font (size 1.27 1.27)) (justify right))
+  )
   (symbol (lib_id "power:GND") (at 160.02 105.41 0) (unit 1)
