File: mikrobus.kicad_sch (KiCad schematic)
At the start: 1 part, among them CON1 MIKROBUS_HOST_CONN

Commit message: added solderpad license text to each sheet
Other:
- note added: "Copyright and related rights are licensed under the Solderpad Hardware License, Version 0.51 (the "License"); you may not use this file except in compliance with the License. You may obtain a copy of the License at http://solderpad.org/licenses/SHL-0.51. Unless required by applicable law or agreed to in writing, software, hardware and materials distributed under this License is distributed on an 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"
Changed lines of the file:
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@@
     (stroke (width 0) (type default) (color 0 0 0 0))
+  )
+  (text "Copyright and related rights are licensed under the Solderpad Hardware License, Version 0.51 (the \"License\");\nyou may not use this file except in compliance with the License.  You may obtain a copy of the License at\nhttp://solderpad.org/licenses/SHL-0.51. Unless required by applicable law or agreed to in writing, software,\nhardware and materials distributed under this License is distributed on an \"AS IS\" BASIS, WITHOUT WARRANTIES OR\nCONDITIONS OF ANY KIND, either express or implied. See the License for the specific language governing\npermissions and limitations under the License.\n"
+    (at 179.07 177.8 0)
+    (effects (font (size 1 1)) (justify left bottom))
   )
   (symbol (lib_id "power:GND") (at 160.02 105.41 0) (unit 1)

Commit message: added the camera, temperature sensor and basic MCU symbol
Parts:
- added C32, C35: 100n, Capacitor_SMD:C_0603_1608Metric, symbol Device:C
- added C33: 10uF, Capacitor_SMD:C_0603_1608Metric, symbol Device:C
- added JP3, JP4, JP5: SolderJumper_2_Open, Jumper:SolderJumper-2_P1.3mm_Open_RoundedPad1.0x1.5mm, symbol Jumper:SolderJumper_2_Open
- added R11, R12, R13, R14: 47k, Resistor_SMD:R_0603_1608Metric, symbol Device:R
- added U11: MCP9808, Package_DFN_QFN:DFN-8-1EP_3x2mm_P0.5mm_EP1.7x1.4mm, symbol Sensor_Temperature:MCP9808_DFN
Connections:
- net +3V3: now also C32.1, C33.1, C35.1, JP3.2 (B), JP4.2 (B), JP5.2 (B), R14.1, U11.8 (VDD)
- net GND: now also C32.2, C33.2, C35.2, R11.2, R12.2, R13.2, U11.4 (GND), U11.9 (EP/GND)
- net click_an: now reaches CON1.P1 (AN)
- net sda: now reaches CON1.P11 (SDA)
- net sda: now also U11.1 (SDA)
- net scl: now reaches CON1.P12 (SCL)
- net scl: now also U11.2 (SCL)
- net click_tx: now reaches CON1.P13 (TX)
- net click_rx: now reaches CON1.P14 (RX)
- net click_int: now reaches CON1.P15 (INT)
- net click_pwm: now reaches CON1.P16 (PWM)
- net click_rst: now reaches CON1.P2 (RST)
- net click_cs: now reaches CON1.P3 (CS)
- net click_sck: now reaches CON1.P4 (SCK)
- net click_miso: now reaches CON1.P5 (MISO)
- net click_mosi: now reaches CON1.P6 (MOSI)
- new net: JP5.1 (A), R13.1, U11.7 (A0)
- new net: JP3.1 (A), R11.1, U11.5 (A2)
- new net: JP4.1 (A), R12.1, U11.6 (A1)
- new net temperature_alert: R14.2, U11.3 (Alert)
Other:
- note added: "Copyright and related rights are licensed under the Solderpad Hardware License, Version 2.1 (the "License"); you may not use this file except in compliance with the License. You may obtain a copy of the License at http://solderpad.org/licenses/SHL-2.1. Unless required by applicable law or agreed to in writing, software, hardware and materials distributed under this License is distributed on an "A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"
- note added: "MCP9808 I2C Address 0011 A2 A1 A0 Default 0011 0 0 0"
- note removed: "Copyright and related rights are licensed under the Solderpad Hardware License, Version 0.51 (the "License"); you may not use this file except in compliance with the License. You may obtain a copy of the License at http://solderpad.org/licenses/SHL-0.51. Unless required by applicable law or agreed to in writing, software, hardware and materials distributed under this License is distributed on an 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"
- moved on the sheet: CON1

Commit message: updated footprints, added the barrel power connector and test points
Parts:
- CON1: footprint mikroBUS:MIKROBUS_HOST_CONN -> mikroBus:MIKROBUS_HOST_CONN
Changed lines of the file:
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@@
-    )
-  )
-  (symbol (lib_id "mikrobus:MIKROBUS_HOST_CONN") (at 62.23 109.22 0) (unit 1)
-    (in_bom yes) (on_board yes) (dnp no) (fields_autoplaced)
-    (property "Reference" "CON1" (at 76.2 64.8802 0)
-      (effects (font (size 1.27 1.27)))
-    )
-    (property "Value" "MIKROBUS_HOST_CONN" (at 76.2 67.4171 0)
-      (effects (font (size 1.27 1.27)))
-    )
-    (property "Footprint" "mikroBUS:MIKROBUS_HOST_CONN" (at 66.04 73.66 0)
-      (effects (font (size 1.27 1.27)) (justify left bottom) hide)
-    )
-    (property "Datasheet" "" (at 62.23 109.22 0)
-      (effects (font (size 1.27 1.27)) hide)
-    )
-    (pin "P1")
-    (pin "P10")
-    (pin "P11")
-    (pin "P12")
-    (pin "P13")
-    (pin "P14")
-    (pin "P15")
-    (pin "P16")
-    (pin "P2")
-    (pin "P3")
-    (pin "P4")
-    (pin "P5")
-    (pin "P6")
-    (pin "P7")
-    (pin "P8")
-    (pin "P9")
-    (instances
-      (project "OpenHW DevKit"
-        (path "/b0906e10-2fbc-4309-a8b4-6fc4cd1a5490/43d030b0-c46c-4448-bc9e-987f12c7559d"
-          (reference "CON1") (unit 1)
-        )
-      )
     )
   )
@@
         )
       )
+    )
+  )
+  (symbol (lib_id "mikrobus:MIKROBUS_HOST_CONN") (at 62.23 109.22 0) (unit 1)
+    (in_bom yes) (on_board yes) (dnp no) (fields_autoplaced)
+    (property "Reference" "CON1" (at 76.2 64.8802 0)
+      (effects (font (size 1.27 1.27)))
+    )
+    (property "Value" "MIKROBUS_HOST_CONN" (at 76.2 67.4171 0)
+      (effects (font (size 1.27 1.27)))
+    )
+    (property "Footprint" "mikroBus:MIKROBUS_HOST_CONN" (at 66.04 73.66 0)
+      (effects (font (size 1.27 1.27)) (justify left bottom) hide)
+    )
+    (property "Datasheet" "" (at 62.23 109.22 0)
+      (effects (font (size 1.27 1.27)) hide)
+    )
+    (pin "P1")
+    (pin "P10")
+    (pin "P11")
+    (pin "P12")
+    (pin "P13")
+    (pin "P14")
+    (pin "P15")
+    (pin "P16")
+    (pin "P2")
+    (pin "P3")
+    (pin "P4")
+    (pin "P5")
+    (pin "P6")
+    (pin "P7")
+    (pin "P8")
+    (pin "P9")
+    (instances
+      (project "OpenHW DevKit"
+        (path "/b0906e10-2fbc-4309-a8b4-6fc4cd1a5490/43d030b0-c46c-4448-bc9e-987f12c7559d"
+          (reference "CON1") (unit 1)
+        )
+        (path "/b0906e10-2fbc-4309-a8b4-6fc4cd1a5490/0f04658e-bc58-402e-baec-b0a803f67eac"
+          (reference "CON1") (unit 1)
+        )
+      )
