File: jtag.kicad_sch (KiCad schematic)
At the start: 38 parts, among them J3 USB_C_Receptacle, J4 Conn_01x02_Male, J5 3220-10-0100-00, U2 FT2232HL-REEL, U3 74LVC125ADRG3, Y2 12MHz

Commit message: additional sheets added
Connections:
- net +1V8: no longer C9.1, U2.12 (VCORE-1), U2.37 (VCORE-2), U2.49 (VREGOUT), U2.64 (VCORE-3)
- new net FTDI_1v8: C9.1, U2.12 (VCORE-1), U2.37 (VCORE-2), U2.49 (VREGOUT), U2.64 (VCORE-3)
Other:
- note added: "TODO: activity LED's for JTAG?"
- note added: "https://riscv.org/wp-content/uploads/2019/03/riscv-debug-release.pdf"
- note removed: "activity LED's for JTAG?"
- moved on the sheet: C21, U3E

Commit message: updates to the jtag interface
Parts:
- removed U3: 74LVC125ADRG3, Package_SO:SOIC-14_3.9x8.7mm_P1.27mm, symbol 74xx:74LVC125
- added C22, C23, C24, C25: 100nF, Capacitor_SMD:C_0603_1608Metric_Pad1.08x0.95mm_HandSolder, symbol Device:C_Small
- added D7: LED_Small, LED_SMD:LED_0603_1608Metric, symbol Device:LED_Small
- added JP2: SolderJumper_2_Bridged, Jumper:SolderJumper-2_P1.3mm_Bridged_RoundedPad1.0x1.5mm, symbol Jumper:SolderJumper_2_Bridged
- added R9: 2.2k, Resistor_SMD:R_0603_1608Metric_Pad0.98x0.95mm_HandSolder, symbol Device:R
- added U4, U5, U6, U7, U8: 74LVC1G125, Package_TO_SOT_SMD:SOT-353_SC-70-5, symbol 74xGxx:74LVC1G125
- D5, D6: footprint LED_SMD:LED_0201_0603Metric_Pad0.64x0.40mm_HandSolder -> LED_SMD:LED_0603_1608Metric
Connections:
- net +3V3: now also JP2.2 (B), R9.2; no longer C21.1
- net GND: now also C22.2, C23.2, C24.2, C25.2, U4.3 (GND), U5.3 (GND), U6.3 (GND), U7.3 (GND), U8.3 (GND)
- net TCK: now also U5.4
- net TDI: now also U4.2
- net TDO: now also U6.4
- net TMS: now also U7.4
- net nRESET: now also U8.4
- net at J4.2 (Pin_2), R8.2: now also U4.1, U5.1, U6.1, U7.1, U8.1
- net at U2.29 (ACBUS3): now also D7.1 (K)
- net at U2.16 (ADBUS0): now also U5.2
- net at U2.17 (ADBUS1): now also U4.4
- net at U2.18 (ADBUS2): now also U6.2
- net at U2.19 (ADBUS3): now also U7.2
- net at U2.23 (ADBUS6): now also U8.2
- new net: D7.2 (A), R9.1
- new net VCC: C21.1, C22.1, C23.1, C24.1, C25.1, JP2.1 (A), U4.5 (VCC), U5.5 (VCC), U6.5 (VCC), U7.5 (VCC), U8.5 (VCC)
- no-connect marks 11 -> 22
Other:
- note removed: "TODO: Verify the nRESET and how to use FTDI with it."
- note removed: "TODO: activity LED's for JTAG?"
- moved on the sheet: C21, C6, C9, J5, R8

Commit message: Edits to JTAG
Other:
- note added: "Note: 74lvc1g125 use hidden vcc pin for power"
- moved on the sheet: C21, C22, C23, C24, C25
