File: jtag.kicad_sch (KiCad schematic)
At the start: 38 parts, among them J3 USB_C_Receptacle, J4 Conn_01x02_Male, J5 3220-10-0100-00, U2 FT2232HL-REEL, U3 74LVC125ADRG3, Y2 12MHz

Commit message: updates jtag sheet
Parts:
- removed U3: 74LVC125ADRG3, Package_SO:SOIC-14_3.9x8.7mm_P1.27mm, symbol 74xx:74LVC125
- added C22, C23, C24, C25: 100nF, Capacitor_SMD:C_0603_1608Metric_Pad1.08x0.95mm_HandSolder, symbol Device:C_Small
- added D7: LED_Small, LED_SMD:LED_0603_1608Metric, symbol Device:LED_Small
- added JP2: SolderJumper_2_Bridged, Jumper:SolderJumper-2_P1.3mm_Bridged_RoundedPad1.0x1.5mm, symbol Jumper:SolderJumper_2_Bridged
- added R9: 2.2k, Resistor_SMD:R_0603_1608Metric_Pad0.98x0.95mm_HandSolder, symbol Device:R
- added U3, U4, U5, U6, U7: 74LVC1G125, Package_TO_SOT_SMD:SOT-353_SC-70-5, symbol 74xGxx:74LVC1G125
- D5, D6: footprint LED_SMD:LED_0201_0603Metric_Pad0.64x0.40mm_HandSolder -> LED_SMD:LED_0603_1608Metric
Connections:
- net +3V3: now also JP2.1 (A), R9.2; no longer C21.1
- net GND: now also C22.2, C23.2, C24.2, C25.2, U3.3 (GND), U4.3 (GND), U5.3 (GND), U6.3 (GND), U7.3 (GND)
- net TCK: now also U4.4
- net TDI: now also U3.2
- net TDO: now also U5.4
- net TMS: now also U6.4
- net nRESET: now also U7.4
- net at J4.2 (Pin_2), R8.2: now also U3.1, U4.1, U5.1, U6.1, U7.1
- net at U2.29 (ACBUS3): now also D7.1 (K)
- net at U2.16 (ADBUS0): now also U4.2
- net at U2.17 (ADBUS1): now also U3.4
- net at U2.18 (ADBUS2): now also U5.2
- net at U2.19 (ADBUS3): now also U6.2
- net at U2.23 (ADBUS6): now also U7.2
- net +1V8 renamed ft_1v8
- new net: D7.2 (A), R9.1
- new net VCC: C21.1, C22.1, C23.1, C24.1, C25.1, JP2.2 (B), U3.5 (VCC), U4.5 (VCC), U5.5 (VCC), U6.5 (VCC), U7.5 (VCC)
- no-connect marks 11 -> 24
Other:
- note removed: "TODO: Verify the nRESET and how to use FTDI with it."
- note removed: "activity LED's for JTAG?"
- moved on the sheet: C14, C15, C16, C17, C18, C19, C20, C21, C6, C9, J5

Commit message: added solderpad license text to each sheet
Other:
- note added: "Copyright and related rights are licensed under the Solderpad Hardware License, Version 0.51 (the "License"); you may not use this file except in compliance with the License. You may obtain a copy of the License at http://solderpad.org/licenses/SHL-0.51. Unless required by applicable law or agreed to in writing, software, hardware and materials distributed under this License is distributed on an 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"
Changed lines of the file:
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@@
     (effects (font (size 1.27 1.27)) (justify left bottom))
+  )
+  (text "Copyright and related rights are licensed under the Solderpad Hardware License, Version 0.51 (the \"License\");\nyou may not use this file except in compliance with the License.  You may obtain a copy of the License at\nhttp://solderpad.org/licenses/SHL-0.51. Unless required by applicable law or agreed to in writing, software,\nhardware and materials distributed under this License is distributed on an \"AS IS\" BASIS, WITHOUT WARRANTIES OR\nCONDITIONS OF ANY KIND, either express or implied. See the License for the specific language governing\npermissions and limitations under the License.\n"
+    (at 179.07 177.8 0)
+    (effects (font (size 1 1)) (justify left bottom))
   )
   (label "d-" (at 54.61 87.63 0)

Commit message: added the camera, temperature sensor and basic MCU symbol
Parts:
- removed Y2: 12MHz, Crystal:Crystal_SMD_HC49-SD, symbol Device:Crystal_Small
- added Y2: 12MHz, Crystal:Crystal_SMD_Abracon_ABM8G-4Pin_3.2x2.5mm, symbol Device:Crystal_GND24_Small
Connections:
- net GND: now also Y2.2, Y2.4
- net osci: now also Y2.1
- net osco: now also Y2.3
Other:
- note added: "Copyright and related rights are licensed under the Solderpad Hardware License, Version 2.1 (the "License"); you may not use this file except in compliance with the License. You may obtain a copy of the License at http://solderpad.org/licenses/SHL-2.1. Unless required by applicable law or agreed to in writing, software, hardware and materials distributed under this License is distributed on an "A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"
- note removed: "Copyright and related rights are licensed under the Solderpad Hardware License, Version 0.51 (the "License"); you may not use this file except in compliance with the License. You may obtain a copy of the License at http://solderpad.org/licenses/SHL-0.51. Unless required by applicable law or agreed to in writing, software, hardware and materials distributed under this License is distributed on an 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"
Changed lines of the file:
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@@
   (junction (at 59.69 90.17) (diameter 0) (color 0 0 0 0)
   )
+  (junction (at 31.75 166.37) (diameter 0) (color 0 0 0 0)
+  )
   (junction (at 237.49 123.19) (diameter 0) (color 0 0 0 0)
   )
@@
   )
   (junction (at 237.49 109.22) (diameter 0) (color 0 0 0 0)
-  )
-  (junction (at 31.75 166.37) (diameter 0) (color 0 0 0 0)
   )
   (no_connect (at 158.75 110.49))
@@
     (stroke (width 0) (type default) (color 0 0 0 0))
   )
+  (wire (pts (xy 22.86 163.83) (xy 29.21 163.83))
+    (stroke (width 0) (type default) (color 0 0 0 0))
+  )
   (wire (pts (xy 158.75 125.73) (xy 209.55 125.73))
     (stroke (width 0) (type default) (color 0 0 0 0))
@@
     (stroke (width 0) (type default) (color 0 0 0 0))
   )
-  (wire (pts (xy 31.75 168.91) (xy 31.75 166.37))
+  (wire (pts (xy 31.75 170.18) (xy 31.75 166.37))
     (stroke (width 0) (type default) (color 0 0 0 0))
   )
@@
     (stroke (width 0) (type default) (color 0 0 0 0))
   )
-  (wire (pts (xy 31.75 158.75) (xy 31.75 161.29))
+  (wire (pts (xy 31.75 157.48) (xy 31.75 161.29))
     (stroke (width 0) (type default) (color 0 0 0 0))
   )
@@
     (stroke (width 0) (type default) (color 0 0 0 0))
   )
+  (wire (pts (xy 34.29 163.83) (xy 48.26 163.83))
+    (stroke (width 0) (type default) (color 0 0 0 0))
+  )
   (wire (pts (xy 179.07 25.4) (xy 179.07 87.63))
     (stroke (width 0) (type default) (color 0 0 0 0))
@@
     (stroke (width 0) (type default) (color 0 0 0 0))
   )
-  (wire (pts (xy 40.64 158.75) (xy 31.75 158.75))
+  (wire (pts (xy 38.1 157.48) (xy 31.75 157.48))
     (stroke (width 0) (type default) (color 0 0 0 0))
   )
@@
     (stroke (width 0) (type default) (color 0 0 0 0))
   )
-  (wire (pts (xy 40.64 168.91) (xy 31.75 168.91))
+  (wire (pts (xy 38.1 170.18) (xy 31.75 170.18))
     (stroke (width 0) (type default) (color 0 0 0 0))
   )
@@
     (effects (font (size 1.27 1.27)) (justify left bottom))
   )
-  (text "Copyright and related rights are licensed under the Solderpad Hardware License, Version 0.51 (the \"License\");\nyou may not use this file except in compliance with the License.  You may obtain a copy of the License at\nhttp://solderpad.org/licenses/SHL-0.51. Unless required by applicable law or agreed to in writing, software,\nhardware and materials distributed under this License is distributed on an \"AS IS\" BASIS, WITHOUT WARRANTIES OR\nCONDITIONS OF ANY KIND, either express or implied. See the License for the specific language governing\npermissions and limitations under the License.\n"
-    (at 179.07 177.8 0)
+  (text "Copyright and related rights are licensed under the Solderpad Hardware License, Version 2.1 (the \"License\");\nyou may not use this file except in compliance with the License.  You may obtain a copy of the License at\nhttp://solderpad.org/licenses/SHL-2.1. Unless required by applicable law or agreed to in writing, software,\nhardware and materials distributed under this License is distributed on an \"AS IS\" BASIS, WITHOUT WARRANTIES OR\nCONDITIONS OF ANY KIND, either express or implied. See the License for the specific language governing\npermissions and limitations under the License.\n"
+    (at 180.34 179.07 0)
     (effects (font (size 1 1)) (justify left bottom))
   )
@@
     (effects (font (size 1.27 1.27)) (justify left bottom))
   )
-  (global_label "osci" (shape input) (at 40.64 168.91 0) (fields_autoplaced)
+  (global_label "osci" (shape input) (at 38.1 170.18 0) (fields_autoplaced)
     (effects (font (size 1.27 1.27)) (justify left))
-    (property "Intersheet References" "${INTERSHEET_REFS}" (id 0) (at 46.9236 168.8306 0)
+    (property "Intersheet References" "${INTERSHEET_REFS}" (id 0) (at 44.3836 170.1006 0)
       (effects (font (size 1.27 1.27)) (justify left) hide)
     )
@@
     )
   )
-  (global_label "osco" (shape input) (at 40.64 158.75 0) (fields_autoplaced)
+  (global_label "osco" (shape input) (at 38.1 157.48 0) (fields_autoplaced)
     (effects (font (size 1.27 1.27)) (justify left))
-    (property "Intersheet References" "${INTERSHEET_REFS}" (id 0) (at 47.4679 158.6706 0)
+    (property "Intersheet References" "${INTERSHEET_REFS}" (id 0) (at 44.9279 157.4006 0)
       (effects (font (size 1.27 1.27)) (justify left) hide)
     )
@@
     (pin "2")
   )
-  (symbol (lib_id "Device:Crystal_Small") (at 31.75 163.83 270) (unit 1)
-    (in_bom yes) (on_board yes)
-    (property "Reference" "Y2" (id 0) (at 33.9852 162.6616 90)
-      (effects (font (size 1.27 1.27)) (justify left))
-    )
-    (property "Value" "12MHz" (id 1) (at 33.9852 164.973 90)
-      (effects (font (size 1.27 1.27)) (justify left))
-    )
-    (property "Footprint" "Crystal:Crystal_SMD_HC49-SD" (id 2) (at 31.75 163.83 0)
-      (effects (font (size 1.27 1.27)) hide)
-    )
-    (property "Datasheet" "~" (id 3) (at 31.75 163.83 0)
-      (effects (font (size 1.27 1.27)) hide)
-    )
-    (pin "1")
-    (pin "2")
-  )
   (symbol (lib_id "power:+3.3V") (at 255.27 22.86 0) (unit 1)
     (in_bom yes) (on_board yes)
@@
     (pin "1")
     (pin "2")
+  )
+  (symbol (lib_id "Device:Crystal_GND24_Small") (at 31.75 163.83 90) (unit 1)
+    (in_bom yes) (on_board yes)
+    (property "Reference" "Y2" (id 0) (at 34.29 161.29 90))
+    (property "Value" "12MHz" (id 1) (at 35.56 166.37 90))
+    (property "Footprint" "Crystal:Crystal_SMD_Abracon_ABM8G-4Pin_3.2x2.5mm" (id 2) (at 31.75 163.83 0)
+      (effects (font (size 1.27 1.27)) hide)
+    )
+    (property "Datasheet" "~" (id 3) (at 31.75 163.83 0)
+      (effects (font (size 1.27 1.27)) hide)
+    )
+    (pin "1")
+    (pin "2")
+    (pin "3")
+    (pin "4")
   )
   (symbol (lib_id "power:+3.3V") (at 265.43 22.86 0) (unit 1)
@@
       (effects (font (size 1.27 1.27)) hide)
     )
+    (pin "1")
+  )
+  (symbol (lib_id "power:GND") (at 48.26 163.83 0) (unit 1)
+    (in_bom yes) (on_board yes)
+    (property "Reference" "#PWR0150" (id 0) (at 48.26 170.18 0)
+      (effects (font (size 1.27 1.27)) hide)
+    )
+    (property "Value" "GND" (id 1) (at 48.387 168.2242 0))
+    (property "Footprint" "" (id 2) (at 48.26 163.83 0)
+      (effects (font (size 1.27 1.27)) hide)
+    )
+    (property "Datasheet" "" (id 3) (at 48.26 163.83 0)
+      (effects (font (size 1.27 1.27)) hide)
+    )

Commit message: MCU pinout finalized
Connections:
- net +3V3: no longer J5.1
Changed lines of the file:
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@@
-    (pin "1")
-  )
-  (symbol (lib_id "power:+3.3V") (at 255.27 132.08 0) (unit 1)
-    (in_bom yes) (on_board yes)
-    (property "Reference" "#PWR0106" (id 0) (at 255.27 135.89 0)
-      (effects (font (size 1.27 1.27)) hide)
-    )
-    (property "Value" "+3.3V" (id 1) (at 255.651 127.6858 0))
-    (property "Footprint" "" (id 2) (at 255.27 132.08 0)
-      (effects (font (size 1.27 1.27)) hide)
-    )
-    (property "Datasheet" "" (id 3) (at 255.27 132.08 0)
-      (effects (font (size 1.27 1.27)) hide)
-    )
     (pin "1")
   )

Commit message: Power and Level Shifter updates
Parts:
- removed C6, C9: 4.7uF, Capacitor_SMD:C_0603_1608Metric_Pad1.08x0.95mm_HandSolder, symbol Device:C_Small
- removed JP2: SolderJumper_2_Bridged, Jumper:SolderJumper-2_P1.3mm_Bridged_RoundedPad1.0x1.5mm, symbol Jumper:SolderJumper_2_Bridged
- removed R8: 10k, Resistor_SMD:R_0603_1608Metric_Pad0.98x0.95mm_HandSolder, symbol Device:R
- removed U3, U4, U5, U6, U7: 74LVC1G125, Package_TO_SOT_SMD:SOT-353_SC-70-5, symbol 74xGxx:74LVC1G125
- added C?: 100nF, Capacitor_SMD:C_0603_1608Metric_Pad1.08x0.95mm_HandSolder, symbol Device:C_Small
- added R?: 10k, Resistor_SMD:R_0603_1608Metric_Pad0.98x0.95mm_HandSolder, symbol Device:R
- added U? (x3): PI4ULS3V302XVEX, PSON40P160X120X55-8N, symbol PI4ULS3V302XVEX:PI4ULS3V302XVEX
Connections:
- net +3V3: now also C24.1, C25.1, C?.1, U?.8 (VCCB), U?.8 (VCCB), U?.8 (VCCB); no longer J4.1 (Pin_1), U2.50 (VREGIN)
- net GND: now also J4.2 (Pin_2), C?.2, U?.4 (GND), U?.4 (GND), U?.4 (GND), U?.6 (B2)
- net TCK: now also U?.2 (A1)
- net TDI: now also U?.3 (A2)
- net TDO: now also U?.2 (A1)
- net TMS: now also U?.3 (A2)
- net nRESET: now also U?.2 (A1)
- net at U2.19 (ADBUS3): now also U?.6 (B2)
- net at U2.23 (ADBUS6): now also U?.7 (B1)
- net at U2.18 (ADBUS2): now also U?.7 (B1)
- net +1V8: now reaches J5.1
- net +1V8: now also C18.1, C19.1, C20.1, C21.1, C22.1, C23.1, U2.12 (VCORE-1), U2.37 (VCORE-2), U2.64 (VCORE-3), R?.2, U?.1 (VCCA), U?.1 (VCCA), U?.1 (VCCA)
- net at U2.16 (ADBUS0): now also U?.7 (B1)
- net at U2.17 (ADBUS1): now also U?.6 (B2)
- removed net VCC: C21.1, C22.1, C23.1, C24.1, C25.1
- removed net ft_1v8: C18.1, C19.1, C20.1, U2.12 (VCORE-1), U2.37 (VCORE-2), U2.49 (VREGOUT), U2.64 (VCORE-3)
- new net: J4.1 (Pin_1), R?.1, U?.5 (EN), U?.5 (EN), U?.5 (EN)
- no-connect marks 24 -> 27
Other:
- moved on the sheet: C18, C19, C20, C21, C22, C23, C24, C25, D7, J4, J5, R9

Commit message: updates to the footprints
Parts:
- C10, C11, C12, C13, C14, C15, C16, C17, C18, C19, C20, C21, C22, C23, C24, C25, C5, C7, C8: footprint Capacitor_SMD:C_0603_1608Metric_Pad1.08x0.95mm_HandSolder -> Capacitor_SMD:C_0603_1608Metric
- C68: renamed from C?; footprint Capacitor_SMD:C_0603_1608Metric_Pad1.08x0.95mm_HandSolder -> Capacitor_SMD:C_0603_1608Metric
- U20, U21, U22: renamed from U?; footprint PSON40P160X120X55-8N -> pi4uls3v302:PSON40P160X120X55-8N
- gave numbers to parts that had none: 1

Commit message: pcb updates including level shifter adjustments
Connections:
- net VBUS: now reaches D1.1 (A1), D3.A, J3.A4 (VBUS), J3.A9 (VBUS), J3.B4 (VBUS), J3.B9 (VBUS)
Changed lines of the file:
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@@
+    (effects (font (size 1.27 1.27)) (justify left bottom))
+  )
+  (label "VBUS" (at 46.99 60.96 0)
     (effects (font (size 1.27 1.27)) (justify left bottom))
   )
