File: jtag.kicad_sch (KiCad schematic)
At the start: 45 parts, among them J3 USB_C_Receptacle, J4 Conn_01x02_Male, J5 3220-10-0100-00, U2 FT2232HL-REEL, U20 PI4ULS3V302XVEX, U21 PI4ULS3V302XVEX, U22 PI4ULS3V302XVEX, Y2 12MHz

Commit message: Changed to KiCAD 7 and updated to final pinout.
Parts:
- removed C21, C22, C23, C24, C25: 100nF, Capacitor_SMD:C_0603_1608Metric, symbol Device:C_Small
- removed U20, U21, U22: PI4ULS3V302XVEX, pi4uls3v302:PSON40P160X120X55-8N, symbol PI4ULS3V302XVEX:PI4ULS3V302XVEX
- added U10, U13: NTB0104BQ,115, NTB0104:NXP_Semiconductors-SOT762-1-08_2019-0-MFG, symbol NTB0104:NTB0104BQ,115
Connections:
- net +1V8: now also U10.1 (VCC(A)), U13.1 (VCC(A))
- net +3V3: now also U10.14 (VCC(B)), U13.14 (VCC(B))
- net GND: now also U10.15 (GND), U10.7 (GND), U13.15 (GND), U13.7 (GND)
- net TCK: now also U10.2 (A1)
- net TDI: now also U10.3 (A2)
- net TDO: now also U10.4 (A3)
- net TMS: now also U10.5 (A4)
- net nRESET: now also U13.2 (A1)
- net at J4.1 (Pin_1), R29.1: now also U10.8 (OE), U13.8 (OE)
- net at U2.23 (ADBUS6): now also U13.13 (B1)
- net at U2.17 (ADBUS1): now also U10.12 (B2)
- net at U2.16 (ADBUS0): now also U10.13 (B1)
- net at U2.19 (ADBUS3): now also U10.10 (B4)
- net at U2.18 (ADBUS2): now also U10.11 (B3)
- no-connect marks 27 -> 29
Other:
- moved on the sheet: C68, J4, J5, R29

Commit message: updated pinout changes
Parts:
- added C26: 3.3uF, Capacitor_SMD:C_0603_1608Metric, symbol Device:C_Small
Connections:
- net +1V8: no longer C18.1, C19.1, C20.1, U2.12 (VCORE-1), U2.37 (VCORE-2), U2.64 (VCORE-3)
- net +3V3: now also U2.50 (VREGIN)
- net GND: now also C26.2
- net TCK: now also U10.4 (A3); no longer U10.2 (A1)
- net TDI: now also U10.2 (A1); no longer U10.3 (A2)
- net TDO: now also U10.3 (A2); no longer U10.4 (A3)
- net nRESET: now also U13.5 (A4); no longer U13.2 (A1)
- net at U10.11 (B3): now also U2.16 (ADBUS0); no longer U2.18 (ADBUS2)
- net at U10.12 (B2): now also U2.18 (ADBUS2); no longer U2.17 (ADBUS1)
- net at U10.13 (B1): now also U2.17 (ADBUS1); no longer U2.16 (ADBUS0)
- net at U13.10 (B4): now also U2.23 (ADBUS6)
- net at U13.13 (B1): no longer U2.23 (ADBUS6)
- net at U2.49 (VREGOUT): now also C18.1, C19.1, C20.1, U2.12 (VCORE-1), U2.37 (VCORE-2), U2.64 (VCORE-3), C26.1
- no-connect marks 29 -> 25
Other:
- note added: "TCK TDI TDO TMS"
- note added: "TDI TDO TCK TMS"
- moved on the sheet: C18, C19, C20

Commit message: updated the QR code and added shield coupling to the usb connector
Parts:
- added C27, C30: 12.5pF, Capacitor_SMD:C_0603_1608Metric, symbol Device:C_Small
- added R24: 1M, Resistor_SMD:R_0603_1608Metric_Pad0.98x0.95mm_HandSolder, symbol Device:R
Connections:
- net GND: now also C27.2, C30.2, R24.2; no longer J3.S1 (SHIELD)
- new net shield: C27.1, C30.1, J3.S1 (SHIELD), R24.1
- no-connect marks 25 -> 30
Other:
- moved on the sheet: C7, C8, Y2

Commit message: Updates to the JTAG interface
Parts:
- added R26: 2.2k, Resistor_SMD:R_0603_1608Metric_Pad0.98x0.95mm_HandSolder, symbol Device:R
- added R27, R28, R42: 10k, Resistor_SMD:R_0603_1608Metric_Pad0.98x0.95mm_HandSolder, symbol Device:R
- added U17: 93C56, Package_SO:SOIC-8_3.9x4.9mm_P1.27mm, symbol Memory_EEPROM:93CxxB
- D5: Function TX -> RX
- D6: Function RX -> TX
Connections:
- net +3V3: now also R27.2, R28.2, R42.2, U17.8 (VCC)
- net FT_RXD: now also U2.39 (BDBUS1); no longer U2.52 (BCBUS1)
- net FT_TXD: now also U2.38 (BDBUS0); no longer U2.48 (BCBUS0)
- net GND: now also U17.5 (GND)
- net at D5.1 (K): now also U2.54 (BCBUS3); no longer U2.41 (BDBUS3)
- net at D6.1 (K): now also U2.55 (BCBUS4); no longer U2.43 (BDBUS4)
- net EE_DATA: now reaches U2.61 (EEDATA)
- net EE_DATA: now also R26.1, U17.3 (DI)
- net EE_SCLK: now reaches U2.62 (EECLK)
- net EE_SCLK: now also R27.1, U17.2 (SCLK)
- net EE_CS: now reaches U2.63 (EECS)
- net EE_CS: now also R42.1, U17.1 (CS)
- new net: R26.2, R28.1, U17.4 (DO)
Other:
- moved on the sheet: C7, C8, D5, D6, R6, R7, Y2

Commit message: pullup resistors on JTAG signals
Parts:
- added D10, D11: BAT760-7, Diode_SMD:SOD2513X120N, symbol bat760:BAT760-7
Connections:
- net GND: now also U13.12 (B2), U13.13 (B1)
- net nRESET: now also U13.4 (A3); no longer J5.10, U13.5 (A4)
- net at U13.10 (B4): now also D10.A; no longer U2.23 (ADBUS6)
- net at U13.11 (B3): now also D11.A
- new net: D11.C, U2.23 (ADBUS6)
- new net nTRST: J5.10, U13.5 (A4)
Other:
- note added: "Connecting resets through shifters to ensure they are disabled with the jumper"
- note added: "Diodes ensure resets are only active low."
- note removed: "TDI TDO TCK TMS"
- moved on the sheet: J4

Commit message: routed the Opella changes
Parts:
- removed D10, D11: BAT760-7, Diode_SMD:SOD2513X120N, symbol bat760:BAT760-7
- added D10, D12: 1N914WT, Diode_SMD:D_SOD-523, symbol Diode:1N914WT
Connections:
- net at U13.10 (B4): now also D12.2 (A)
- net at U13.11 (B3): now also D10.2 (A)
- net at U2.23 (ADBUS6): now also D10.1 (K)
- net at U2.22 (ADBUS5): now also D12.1 (K)
- no-connect marks 30 -> 29
Other:
- moved on the sheet: J4, J5

Commit message: updated footprints, added the barrel power connector and test points
Parts:
- removed D3: BAT760-7, Diode_SMD:SOD2513X120N, symbol bat760:BAT760-7
- removed J3: USB_C_Receptacle, Connector_USB:USB_C_Receptacle_Amphenol_12401610E4-2A, symbol Connector:USB_C_Receptacle
- added D3: BAT760-7, diode:Diodes-SOD323-03_2017-0-0, symbol diode:BAT760-7
- added J3: USB4105-GF-A, GCT_USB4105-GF-A, symbol usb:USB4105-GF-A
Connections:
- net GND: now also J3.A1_B12 (GND), J3.B1_A12 (GND__1)
- net VBUS: now also D3.2 (ANODE), J3.A4_B9 (VBUS), J3.B4_A9 (VBUS__1)
- net d+: now also J3.A6 (DP1), J3.B6 (DP2)
- net d-: now also J3.A7 (DN1), J3.B7 (DN2)
- net shield: now also J3.S1 (SHELL_GND), J3.S2 (SHELL_GND__1), J3.S3 (SHELL_GND__2), J3.S4 (SHELL_GND__3)
- net at R3.1: now also J3.A5 (CC1)
- net at R2.1: now also J3.B5 (CC2)
- net +5V renamed +VDC
- net +VDC: now also D3.1 (CATHODE)
Other:
- moved on the sheet: C27, C30, C5, D1, D2, D4, R2, R24, R3

Commit message: updated 3d models and cleaned up the DRC
Parts:
- removed J5: 3220-10-0100-00, footprints:3220-10-0100-00, symbol cnc_tech_connector:3220-10-0100-00
- added J5: 3220-10-0100-00, CONN_3220-10-0100-00_CNC, symbol jtag header:3220-10-0100-00
Connections:
- net +1V8: now also J5.1
- net GND: now also J5.3, J5.5, J5.7, J5.9
- net TCK: now also J5.4
- net TDI: now also J5.8
- net TDO: now also J5.6
- net TMS: now also J5.2
- net nTRST: now also J5.10
Changed lines of the file:
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@@
+    )
+  )
+  (symbol (lib_id "jtag header:3220-10-0100-00") (at 264.16 132.08 0) (unit 1)
+    (in_bom yes) (on_board yes) (dnp no)
+    (property "Reference" "J5" (at 277.5585 142.763 0)
+      (effects (font (size 1.524 1.524)) (justify left))
+    )
+    (property "Value" "3220-10-0100-00" (at 261.62 158.75 0)
+      (effects (font (size 1.524 1.524)) (justify left) hide)
+    )
+    (property "Footprint" "CONN_3220-10-0100-00_CNC" (at 264.16 132.08 0)
+      (effects (font (size 1.27 1.27) italic) hide)
+    )
+    (property "Datasheet" "3220-10-0100-00" (at 264.16 132.08 0)
+      (effects (font (size 1.27 1.27) italic) hide)
+    )
+    (pin "1")
+    (pin "10")
+    (pin "2")
+    (pin "3")
+    (pin "4")
+    (pin "5")
+    (pin "6")
+    (pin "7")
+    (pin "8")
+    (pin "9")
+    (instances
+      (project "OpenHW DevKit"
+        (path "/b0906e10-2fbc-4309-a8b4-6fc4cd1a5490/05c5e7d7-6e8b-47d0-a3ba-1eadff858466"
+          (reference "J5") (unit 1)
+        )
+      )
     )
   )
@@
         )
       )
-    )
-  )
-  (symbol (lib_id "cnc_tech_connector:3220-10-0100-00") (at 264.16 132.08 0) (unit 1)
-    (in_bom yes) (on_board yes) (dnp no)
-    (property "Reference" "J5" (at 277.5585 142.5338 0)
-      (effects (font (size 1.524 1.524)) (justify left))
-    )
-    (property "Value" "3220-10-0100-00" (at 261.62 160.02 0)
-      (effects (font (size 1.524 1.524)) (justify left))
-    )
-    (property "Footprint" "footprints:3220-10-0100-00" (at 274.32 143.764 0)
-      (effects (font (size 1.524 1.524)) hide)
-    )
-    (property "Datasheet" "" (at 264.16 132.08 0)
-      (effects (font (size 1.524 1.524)))
-    )
-    (pin "1")
-    (pin "10")
-    (pin "2")
-    (pin "3")
-    (pin "4")
-    (pin "5")
-    (pin "6")
-    (pin "7")
-    (pin "8")
-    (pin "9")
-    (instances
-      (project "OpenHW DevKit"
-        (path "/b0906e10-2fbc-4309-a8b4-6fc4cd1a5490/05c5e7d7-6e8b-47d0-a3ba-1eadff858466"
-          (reference "J5") (unit 1)
-        )
-      )
