File: OpenHW DevKit.kicad_pcb (KiCad board)
At the start: 4 copper layers, 100 x 75 mm, 54 parts, among them CON1 MIKROBUS_HOST_CONN, J1 Conn_02x05_Odd_Even, J2 Conn_02x03_Odd_Even, J3 USB_C_Receptacle, J4 Conn_01x02_Male, J5 3220-10-0100-00, J6 Barrel_Jack, U1 ESP32-C3-MINI-1, U2 FT2232HL-REEL, U3 74LVC125ADRG3, Y1 32.768kHz, Y2 12MHz

Commit message: updates jtag sheet
Parts:
- added C22: 100nF, Capacitor_SMD:C_0603_1608Metric_Pad1.08x0.95mm_HandSolder, F.Cu at (120.8, 107.3)
- added C23: 100nF, Capacitor_SMD:C_0603_1608Metric_Pad1.08x0.95mm_HandSolder, F.Cu at (125.1, 102.3)
- added C24: 100nF, Capacitor_SMD:C_0603_1608Metric_Pad1.08x0.95mm_HandSolder, F.Cu at (120.8, 102.3)
- added C25: 100nF, Capacitor_SMD:C_0603_1608Metric_Pad1.08x0.95mm_HandSolder, F.Cu at (120.8, 104.8)
- added D7: LED_Small, LED_SMD:LED_0603_1608Metric, F.Cu at (129.3, 102.3)
- added JP2: SolderJumper_2_Bridged, Jumper:SolderJumper-2_P1.3mm_Bridged_RoundedPad1.0x1.5mm, F.Cu at (134.0, 96.9)
- added R9: 2.2k, Resistor_SMD:R_0603_1608Metric_Pad0.98x0.95mm_HandSolder, F.Cu at (125.1, 104.8)
- added U4: 74LVC1G125, Package_TO_SOT_SMD:SOT-353_SC-70-5, F.Cu at (128.0, 108.4)
- added U5: 74LVC1G125, Package_TO_SOT_SMD:SOT-353_SC-70-5, F.Cu at (133.0, 102.6)
- added U6: 74LVC1G125, Package_TO_SOT_SMD:SOT-353_SC-70-5, F.Cu at (124.6, 107.6)
- added U7: 74LVC1G125, Package_TO_SOT_SMD:SOT-353_SC-70-5, F.Cu at (129.0, 105.2)
- D5, D6: footprint LED_SMD:LED_0201_0603Metric_Pad0.64x0.40mm_HandSolder -> LED_SMD:LED_0603_1608Metric
- U3: value 74LVC125ADRG3 -> 74LVC1G125; footprint Package_SO:SOIC-14_3.9x8.7mm_P1.27mm -> Package_TO_SOT_SMD:SOT-353_SC-70-5
- moved U3 19.7 mm to (134.4, 107.2)
Connections:
- net +1V8 renamed /jtag and uart/ft_1v8
- C21 pad 1: +3V3 -> VCC
- U2 pad 16: unconnected-(U2-Pad16) -> Net-(U2-Pad16)
- U2 pad 17: unconnected-(U2-Pad17) -> Net-(U2-Pad17)
- U2 pad 18: unconnected-(U2-Pad18) -> Net-(U2-Pad18)
- U2 pad 19: unconnected-(U2-Pad19) -> Net-(U2-Pad19)
- U2 pad 23: unconnected-(U2-Pad23) -> Net-(U2-Pad23)
- U2 pad 26: Net-(U2-Pad26) -> unconnected-(U2-Pad26)
- U2 pad 27: Net-(U2-Pad27) -> unconnected-(U2-Pad27)
- U2 pad 28: Net-(U2-Pad28) -> unconnected-(U2-Pad28)
- U3 pad 2: Net-(U2-Pad26) -> /jtag and uart/TDI
- U3 pad 3: /jtag and uart/TCK -> GND
- U3 pad 4: Net-(J4-Pad2) -> Net-(U2-Pad17)
- U3 pad 5: Net-(U2-Pad27) -> VCC

Commit message: adjustments
Parts:
- moved C21 1.94 mm to (151.8, 94.6)
Changed lines of the file:
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@@
   )
   (footprint "Capacitor_SMD:C_0603_1608Metric_Pad1.08x0.95mm_HandSolder" (layer "F.Cu")
-    (at 152.146 92.71)
+    (at 151.765 94.615)
     (descr "Capacitor SMD 0603 (1608 Metric), square (rectangular) end terminal, IPC_7351 nominal with elongated pad for handsoldering. (Body size source: IPC-SM-782 page 76, https://www.pcb-3d.com/wordpress/wp-content/uploads/ipc-sm-782a_amendment_1_and_2.pdf), generated with kicad-footprint-generator")
     (tags "capacitor handsolder")

Commit message: added logs and 3d model updates
Parts:
- added G***: LOGO, logos:core-v, F.Cu at (187.3, 129.4)
- added G***: LOGO, logos:openhw_group_small, F.Cu at (124.0, 129.5)
- moved C25 43.4 mm to (163.3, 96.3), turned to 180 degrees
- moved C24 39.7 mm to (160.0, 96.3), turned to 180 degrees
- moved U7 36.1 mm to (163.3, 94.0)
- moved C22 34.5 mm to (153.4, 96.3), turned to 180 degrees
- moved C23 32.2 mm to (156.7, 96.3), turned to 180 degrees
- moved U4 29.2 mm to (153.4, 94.0)
- moved U6 28.9 mm to (150.1, 94.0)
- moved U3 28.9 mm to (160.0, 94.0)
- moved U5 25.2 mm to (156.7, 94.0)
- moved R8 17.1 mm to (165.9, 94.4), turned to 90 degrees
- moved D5 17.1 mm to (118.6, 95.0)
- moved D6 17.1 mm to (118.6, 92.7)
- moved R6 17.1 mm to (122.2, 95.2)
- moved R7 17.1 mm to (122.2, 92.5)
- moved D7 16.6 mm to (118.6, 89.7)
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Other:
- outline, holes or cut-outs redrawn

Commit message: updates to the images and place holders for MCU footprint
Parts:
- added C26: 1uF, Capacitor_SMD:C_0603_1608Metric, F.Cu at (111.3, 80.8)
- added C27: 1uF, Capacitor_SMD:C_0603_1608Metric, F.Cu at (103.6, 92.7)
- added C28: 1uF, Capacitor_SMD:C_0603_1608Metric, F.Cu at (115.3, 96.8)
- added C29: 1uF, Capacitor_SMD:C_0603_1608Metric, F.Cu at (115.3, 80.8)
- added C30: 1uF, Capacitor_SMD:C_0603_1608Metric, F.Cu at (107.7, 92.7)
- added C31: 1uF, Capacitor_SMD:C_0603_1608Metric, F.Cu at (115.3, 98.3)
- added C32: 1uF, Capacitor_SMD:C_0603_1608Metric, F.Cu at (103.6, 80.8)
- added C33: 1uF, Capacitor_SMD:C_0603_1608Metric, F.Cu at (107.7, 80.8)
- added C34: 10uF, Capacitor_SMD:C_0603_1608Metric_Pad1.08x0.95mm_HandSolder, F.Cu at (147.6, 73.4)
- added D8: BAT760-7, Diode_SMD:SOD2513X120N, F.Cu at (109.2, 75.7)
- added D9: MMBD4448HADW, Package_TO_SOT_SMD:SOT-363_SC-70-6, F.Cu at (113.3, 92.2)
- added G***: LOGO, LOGO, F.Cu at (182.6, 112.0)
- added G***: LOGO, logos:mcu_devkit_bold_275_reverse, F.Cu at (120.7, 115.6)
- added J10: PinHeader_1x20_P1.00mm_Vertical, Connector_PinHeader_1.00mm:PinHeader_1x20_P1.00mm_Vertical, F.Cu at (143.2, 100.3)
- added J11: PinHeader_1x20_P1.00mm_Vertical, Connector_PinHeader_1.00mm:PinHeader_1x20_P1.00mm_Vertical, F.Cu at (141.1, 102.6)
- added J12: PinHeader_1x20_P1.00mm_Vertical, Connector_PinHeader_1.00mm:PinHeader_1x20_P1.00mm_Vertical, F.Cu at (143.2, 124.0)
- added J13: PinHeader_1x20_P1.00mm_Vertical, Connector_PinHeader_1.00mm:PinHeader_1x20_P1.00mm_Vertical, F.Cu at (164.2, 102.6)
- added J20: PinHeader_2x20_P2.54mm_Vertical, Connector_PinHeader_2.54mm:PinHeader_2x20_P2.54mm_Vertical, F.Cu at (129.3, 131.3)
- added R10: 1M, Resistor_SMD:R_0603_1608Metric_Pad0.98x0.95mm_HandSolder, F.Cu at (150.1, 77.7)
- added U10: TLV71209_SOT23-5, Package_TO_SOT_SMD:SOT-23-5, F.Cu at (112.0, 97.0)
- added U100: LQFP-80_12x12mm_P0.5mm, Package_QFP:LQFP-80_12x12mm_P0.5mm, F.Cu at (152.6, 111.9)
- added U11: LM1117-5.0, Package_TO_SOT_SMD:SOT-223-3_TabPin2, F.Cu at (105.7, 86.1)
- added U8: LM1117-3.3, Package_TO_SOT_SMD:SOT-223-3_TabPin2, F.Cu at (113.3, 86.1)
- added U9: LM1117-1.8, Package_TO_SOT_SMD:SOT-223-3_TabPin2, F.Cu at (105.7, 98.0)
- moved G*** 68.9 mm to (121.4, 109.5)
- moved C21 13.3 mm to (163.3, 94.7)
- moved C25 13.3 mm to (150.1, 94.7)
- moved U6 13.3 mm to (163.3, 92.5)
- moved U7 13.3 mm to (150.1, 92.5)
- moved G*** 8.45 mm to (119.4, 122.4)
- moved D7 8.19 mm to (123.5, 96.3), turned to 180 degrees
- moved R9 6.98 mm to (119.9, 96.3), turned to 180 degrees
- moved D5 6.84 mm to (123.5, 90.2), turned to 180 degrees
- moved C22 6.78 mm to (160.0, 94.7)
- moved C24 6.78 mm to (153.4, 94.7)
- moved U3 6.78 mm to (153.4, 92.5)
- moved U4 6.78 mm to (160.0, 92.5)
- moved J5 6.02 mm to (159.5, 86.1), turned to 180 degrees
- moved R6 5.56 mm to (119.9, 90.2), turned to 180 degrees
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Connections:
- J6 pad 1: unconnected-(J6-Pad1) -> Net-(J6-Pad1)
- J6 pad 2: unconnected-(J6-Pad2) -> GND
Routing:
- net +5V: track 4.55 -> 60.8 mm
- net GND: track 51.8 -> 106.8 mm, vias 23 -> 42
- net +3V3: track 21.7 -> 67.1 mm, vias 0 -> 7
- net Net-(J4-Pad2): track 0.00 -> 29.3 mm, vias 0 -> 8
- net Net-(D7-Pad1): track 0.00 -> 24.0 mm, vias 0 -> 2
- net VCC: track 0.00 -> 17.0 mm
- net +1V8: track 0.00 -> 15.5 mm
- net Net-(D6-Pad1): track 0.00 -> 13.7 mm, vias 0 -> 2
- net Net-(J6-Pad1): track 0.00 -> 12.5 mm
- net Net-(J1-Pad6): track 0.00 -> 12.3 mm, vias 0 -> 1
- net Net-(J2-Pad3): track 0.00 -> 11.9 mm, vias 0 -> 1
- net Net-(J1-Pad4): track 0.00 -> 11.1 mm, vias 0 -> 1
- net Net-(J1-Pad2): track 0.00 -> 11.0 mm, vias 0 -> 1
- net Net-(C32-Pad1): track 0.00 -> 10.9 mm
- net Net-(D5-Pad1): track 0.00 -> 10.7 mm, vias 0 -> 2
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- added copper zone on In2.Cu, net +1V8
- added copper zone on In2.Cu, net +3V3
- added copper zone on In1.Cu, net GND
Other:
- outline, holes or cut-outs redrawn
- board text added: "Ashling Opella-LD Debug"
- board text added: "JTAG"

Commit message: added the camera, temperature sensor and basic MCU symbol
Parts:
- removed D8: BAT760-7, Diode_SMD:SOD2513X120N
- removed J10, J11, J12, J13: PinHeader_1x20_P1.00mm_Vertical, Connector_PinHeader_1.00mm:PinHeader_1x20_P1.00mm_Vertical
- removed J20: PinHeader_2x20_P2.54mm_Vertical, Connector_PinHeader_2.54mm:PinHeader_2x20_P2.54mm_Vertical
- removed U100: LQFP-80_12x12mm_P0.5mm, Package_QFP:LQFP-80_12x12mm_P0.5mm
- added C35: 100n, Capacitor_SMD:C_0603_1608Metric, F.Cu at (192.1, 109.3)
- added C36: 1uF, Capacitor_SMD:C_0603_1608Metric, F.Cu at (175.1, 122.8)
- added C37: 1uF, Capacitor_SMD:C_0603_1608Metric, F.Cu at (183.5, 122.9)
- added JP3: SolderJumper_2_Open, Jumper:SolderJumper-2_P1.3mm_Open_RoundedPad1.0x1.5mm, B.Cu at (195.7, 88.8)
- added JP4: SolderJumper_2_Open, Jumper:SolderJumper-2_P1.3mm_Open_RoundedPad1.0x1.5mm, B.Cu at (195.7, 96.3)
- added JP5: SolderJumper_2_Open, Jumper:SolderJumper-2_P1.3mm_Open_RoundedPad1.0x1.5mm, B.Cu at (195.7, 92.6)
- added R11: 47k, Resistor_SMD:R_0603_1608Metric, F.Cu at (194.4, 94.6)
- added R12: 47k, Resistor_SMD:R_0603_1608Metric, F.Cu at (196.0, 94.6)
- added R13: 47k, Resistor_SMD:R_0603_1608Metric, F.Cu at (197.5, 94.6)
- added R14: 47k, Resistor_SMD:R_0603_1608Metric, F.Cu at (192.9, 94.6)
- added R15: 4.7k, Resistor_SMD:R_0603_1608Metric, F.Cu at (142.1, 49.1)
- added R16: 4.7k, Resistor_SMD:R_0603_1608Metric, F.Cu at (146.1, 49.1)
- added U12: AP2127K-2.8, Package_TO_SOT_SMD:SOT-23-5, F.Cu at (179.2, 123.2)
- C32: value 1uF -> 100n
- C33: value 1uF -> 10uF
- J6: value Barrel_Jack -> Conn_01x24; footprint Connector_BarrelJack:BarrelJack_CLIFF_FC681465S_SMT_Horizontal -> Connector_FFC-FPC:Hirose_FH12-24S-0.5SH_1x24-1MP_P0.50mm_Horizontal
- U11: value LM1117-5.0 -> MCP9808; footprint Package_TO_SOT_SMD:SOT-223-3_TabPin2 -> Package_DFN_QFN:DFN-8-1EP_3x2mm_P0.5mm_EP1.7x1.4mm
- Y2: footprint Crystal:Crystal_SMD_HC49-SD -> Crystal:Crystal_SMD_Abracon_ABM8G-4Pin_3.2x2.5mm
- moved C32 95.8 mm to (196.1, 105.8), turned to 0 degrees
- moved U11 89.7 mm to (195.2, 91.3), turned to 0 degrees
- moved C33 88.5 mm to (193.3, 103.3)
- moved J6 82.2 mm to (179.7, 115.7), turned to 180 degrees
- moved G*** 67.9 mm to (114.8, 114.2)
- moved C27 51.2 mm to (146.1, 121.4)
- moved C30 51.2 mm to (150.1, 121.4)
- moved C28 51.2 mm to (157.7, 125.5)
- moved C29 51.2 mm to (157.7, 109.5)
- moved C31 51.2 mm to (157.7, 127.0)
- moved C26 51.2 mm to (153.7, 109.5)
- moved D9 51.2 mm to (155.7, 120.9)
- moved FB2 51.2 mm to (156.7, 104.6)
- moved U10 51.2 mm to (154.4, 125.7)
- moved U8 51.2 mm to (155.7, 114.8)
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Connections:
- C32 pad 1: Net-(C32-Pad1) -> +3V3
- C33 pad 1: +5V -> +3V3
- CON1 pad P1: unconnected-(CON1-PadP1) -> /mikrobus and sensors/click_an
- CON1 pad P11: unconnected-(CON1-PadP11) -> sda
- CON1 pad P12: unconnected-(CON1-PadP12) -> scl
- CON1 pad P13: unconnected-(CON1-PadP13) -> /mikrobus and sensors/click_tx
- CON1 pad P14: unconnected-(CON1-PadP14) -> /mikrobus and sensors/click_rx
- CON1 pad P15: unconnected-(CON1-PadP15) -> /mikrobus and sensors/click_int
- CON1 pad P16: unconnected-(CON1-PadP16) -> /mikrobus and sensors/click_pwm
- CON1 pad P2: unconnected-(CON1-PadP2) -> /mikrobus and sensors/click_rst
- CON1 pad P3: unconnected-(CON1-PadP3) -> /mikrobus and sensors/click_cs
- CON1 pad P4: unconnected-(CON1-PadP4) -> /mikrobus and sensors/click_sck
- CON1 pad P5: unconnected-(CON1-PadP5) -> /mikrobus and sensors/click_miso
- CON1 pad P6: unconnected-(CON1-PadP6) -> /mikrobus and sensors/click_mosi
- D9 pad 1: Net-(C32-Pad1) -> (no net)
- J6 pad 1: Net-(J6-Pad1) -> unconnected-(J6-Pad1)
- J6 pad 3: (no net) -> /camera/camera_d1
- U11 pad 1: GND -> sda
- U11 pad 2: +5V -> scl
- U11 pad 3: Net-(C32-Pad1) -> /mikrobus and sensors/temperature_alert
- Y2 pad 1: osco -> osci
- Y2 pad 2: osci -> GND
Routing:
- net +5V: track 60.8 -> 0.00 mm
- net Net-(J6-Pad1): track 12.5 -> 0.00 mm
- net Net-(C32-Pad1): track 10.9 -> 0.00 mm
- net +3V3: track 67.1 -> 59.4 mm
- net osci: track 20.6 -> 16.3 mm
- net osco: track 14.1 -> 12.1 mm
- net GND: track 106.8 -> 105.8 mm
Other:
- outline, holes or cut-outs redrawn

Commit message: MCU pinout finalized
Parts:
- added U13: W25Q128JVS, Package_SO:SOIC-8_5.23x5.23mm_P1.27mm, F.Cu at (150.8, 124.2)
- added U14: CV32E40P, Package_QFP:LQFP-80_12x12mm_P0.5mm, F.Cu at (150.8, 109.3)
- added X1: SG-8002LB, Oscillator:Oscillator_SMD_SeikoEpson_SG8002LB-4Pin_5.0x3.2mm, F.Cu at (163.9, 109.5)
- moved R15 64.1 mm to (185.2, 96.6)
- moved R16 64.1 mm to (189.2, 96.6)
- moved FB2 36.8 mm to (120.8, 96.6)
- moved G*** 35.2 mm to (168.8, 91.2)
- moved R8 32.2 mm to (133.7, 91.2), turned to 0 degrees
- moved C21 32.1 mm to (131.8, 88.6), turned to 90 degrees
- moved C22 29.7 mm to (131.8, 85.3), turned to 90 degrees
- moved U6 29.5 mm to (134.1, 88.6), turned to -90 degrees
- moved C23 27.9 mm to (131.8, 82.0), turned to 90 degrees
- moved C24 26.9 mm to (131.8, 78.7), turned to 90 degrees
- moved U4 26.9 mm to (134.1, 85.3), turned to -90 degrees
- moved C25 26.6 mm to (131.8, 75.4), turned to 90 degrees
- moved U5 24.9 mm to (134.1, 82.0), turned to -90 degrees
- moved C29 24.4 mm to (135.4, 99.6)
- moved U8 24.4 mm to (133.3, 104.9)
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Connections:
- net /ExpressLink/EL_EVENT renamed el_event
- net /ExpressLink/EL_RXD renamed el_rx
- net /ExpressLink/EL_TXD renamed el_tx
- net /ExpressLink/EL_WAKE renamed el_wake
- net /ExpressLink/~{EL_RESET} renamed el_reset
- net /camera/camera_int renamed camera_int
- net /camera/camera_pclk renamed camera_pclk
- net /camera/camera_trig renamed camera_trig
- net /jtag and uart/TCK renamed TCK
- net /jtag and uart/TDI renamed TDI
- net /jtag and uart/TDO renamed TDO
- net /jtag and uart/TMS renamed TMS
- net /mikrobus and sensors/click_cs renamed CS0
- net /mikrobus and sensors/click_rx renamed click_rx
- net /mikrobus and sensors/click_sck renamed SCLK0
- net /mikrobus and sensors/click_tx renamed click_tx
- net /mikrobus and sensors/temperature_alert renamed temp_alert
- net scl renamed SCL0
- net sda renamed SDA0
- CON1 pad P15: /mikrobus and sensors/click_int -> irq
- CON1 pad P16: /mikrobus and sensors/click_pwm -> pwm
- CON1 pad P2: /mikrobus and sensors/click_rst -> reset
- CON1 pad P5: /mikrobus and sensors/click_miso -> MOSI0
- CON1 pad P6: /mikrobus and sensors/click_mosi -> MOSI0
- J6 pad 14: /camera/camera_d0 -> camera_d0
- J6 pad 16: /camera/camera_hsync -> camera_hsync
- J6 pad 6: /camera/camera_vsync -> camera_vsync
- J6 pad 8: /camera/camera_mclk -> camera_mclk
- U2 pad 48: /jtag and uart/FT_TXD -> console_tx
- U2 pad 52: /jtag and uart/FT_RXD -> console_rx
Routing:
- net GND: track 105.8 -> 95.6 mm, vias 42 -> 40
- net osco: track 12.1 -> 4.24 mm
- net osci: track 16.3 -> 9.76 mm
- net +1V8: track 15.5 -> 9.00 mm
- net Net-(J4-Pad2): track 29.3 -> 23.0 mm
- net +3V3: track 59.4 -> 56.7 mm

Commit message: updates to the footprints
Parts:
- removed the G*** at (114.8, 114.2)
- removed JP2: SolderJumper_2_Bridged, Jumper:SolderJumper-2_P1.3mm_Bridged_RoundedPad1.0x1.5mm
- added C38: 100nF, Capacitor_SMD:C_0603_1608Metric, F.Cu at (222.9, 94.1)
- added C39: 100nF, Capacitor_SMD:C_0603_1608Metric, F.Cu at (222.7, 84.0)
- added C40: 100nF, Capacitor_SMD:C_0603_1608Metric, F.Cu at (218.0, 99.1)
- added C41: 100nF, Capacitor_SMD:C_0603_1608Metric, F.Cu at (227.0, 84.0)
- added C42: 100nF, Capacitor_SMD:C_0603_1608Metric, F.Cu at (227.3, 91.6)
- added C43: 100nF, Capacitor_SMD:C_0603_1608Metric, F.Cu at (231.4, 86.6)
- added C44: 100nF, Capacitor_SMD:C_0603_1608Metric, F.Cu at (227.0, 86.6)
- added C45: 100nF, Capacitor_SMD:C_0603_1608Metric, F.Cu at (222.7, 86.6)
- added C46: 100nF, Capacitor_SMD:C_0603_1608Metric, F.Cu at (213.7, 100.5)
- added C47: 100nF, Capacitor_SMD:C_0603_1608Metric, F.Cu at (209.3, 99.0)
- added C48: 100nF, Capacitor_SMD:C_0603_1608Metric, F.Cu at (231.9, 79.0)
- added C49: 100nF, Capacitor_SMD:C_0603_1608Metric, F.Cu at (218.3, 86.0)
- added C50: 100nF, Capacitor_SMD:C_0603_1608Metric, F.Cu at (214.2, 92.9)
- added C51: 100nF, Capacitor_SMD:C_0603_1608Metric, F.Cu at (236.3, 79.0)
- added C52: 100nF, Capacitor_SMD:C_0603_1608Metric, F.Cu at (214.2, 90.4)
- added C53: 100nF, Capacitor_SMD:C_0603_1608Metric, F.Cu at (236.3, 81.5)
- added C54: 100nF, Capacitor_SMD:C_0603_1608Metric, F.Cu at (223.2, 79.0)
- added C55: 100nF, Capacitor_SMD:C_0603_1608Metric, F.Cu at (222.9, 91.6)
- added C56: 100nF, Capacitor_SMD:C_0603_1608Metric, F.Cu at (218.3, 83.5)
- added C57: 100nF, Capacitor_SMD:C_0603_1608Metric, F.Cu at (222.9, 89.1)
- added C58: 100nF, Capacitor_SMD:C_0603_1608Metric, F.Cu at (205.0, 96.5)
- added C59: 100nF, Capacitor_SMD:C_0603_1608Metric, F.Cu at (231.4, 84.0)
- added C60: 100nF, Capacitor_SMD:C_0603_1608Metric, F.Cu at (213.7, 95.5)
- added C61: 100nF, Capacitor_SMD:C_0603_1608Metric, F.Cu at (205.0, 99.0)
- added C62: 100nF, Capacitor_SMD:C_0603_1608Metric, F.Cu at (227.6, 81.5)
- added C63: 100nF, Capacitor_SMD:C_0603_1608Metric, F.Cu at (223.2, 81.5)
- added C64: 100nF, Capacitor_SMD:C_0603_1608Metric, F.Cu at (218.6, 91.6)
- added C65: 100nF, Capacitor_SMD:C_0603_1608Metric, F.Cu at (218.6, 89.1)
- added C66: 100nF, Capacitor_SMD:C_0603_1608Metric, F.Cu at (212.7, 87.9)
- added C67: 100nF, Capacitor_SMD:C_0603_1608Metric, F.Cu at (218.0, 96.6)
- added C68: 100nF, Capacitor_SMD:C_0603_1608Metric, F.Cu at (251.9, 81.5)
- added C69: 10uF, Capacitor_SMD:C_0603_1608Metric, F.Cu at (114.4, 115.2)
- added C70: 10uF, Capacitor_SMD:C_0603_1608Metric, F.Cu at (114.4, 117.7)
- added C71: 10uF, Capacitor_SMD:C_0603_1608Metric, F.Cu at (124.5, 109.7)
- added C72: 100nF, Capacitor_SMD:C_0603_1608Metric, F.Cu at (123.7, 111.8)
- added C73: 100nF, Capacitor_SMD:C_0603_1608Metric, F.Cu at (107.5, 120.4)
- added C74: 100nF, Capacitor_SMD:C_0603_1608Metric, F.Cu at (109.9, 120.4)
- added C75: 22uF, Capacitor_SMD:C_0603_1608Metric, F.Cu at (254.5, 63.6)
- added C76: 22uF, Capacitor_SMD:C_0603_1608Metric, F.Cu at (240.8, 64.3)
- added C77: 22uF, Capacitor_SMD:C_0603_1608Metric, F.Cu at (231.6, 60.4)
- added C78: 22uF, Capacitor_SMD:C_0603_1608Metric, F.Cu at (222.2, 60.7)
- added C79: 22uF, Capacitor_SMD:C_0603_1608Metric, F.Cu at (213.7, 65.7)
- added C80: 22uF, Capacitor_SMD:C_0603_1608Metric, F.Cu at (233.1, 70.1)
- added C81: 22uF, Capacitor_SMD:C_0603_1608Metric, F.Cu at (253.2, 71.9)
- added C82: 22uF, Capacitor_SMD:C_0603_1608Metric, F.Cu at (240.8, 71.6)
- added C83: 22uF, Capacitor_SMD:C_0603_1608Metric, F.Cu at (242.1, 67.5)
- added D10: LED, LED_SMD:LED_0603_1608Metric, F.Cu at (226.6, 65.7)
- added D11: LED, LED_SMD:LED_0603_1608Metric, F.Cu at (218.7, 65.2)
- added D8: LED, LED_SMD:LED_0603_1608Metric, F.Cu at (237.0, 67.0)
- added L1: 3.3uH, Inductor_SMD:L_Bourns-SRN4018, F.Cu at (115.4, 111.2)
- added L2: 3.3uH, Inductor_SMD:L_Bourns-SRN4018, F.Cu at (109.3, 116.8)
- added L3: 3.3uH, Inductor_SMD:L_Bourns-SRN4018, F.Cu at (109.3, 111.2)
- added Q1: MMBT3904, Package_TO_SOT_SMD:SOT-23, F.Cu at (218.6, 80.0)
- added Q2: MMBT3904, Package_TO_SOT_SMD:SOT-23, F.Cu at (213.7, 80.0)
- added Q3: MMBT3904, Package_TO_SOT_SMD:SOT-23, F.Cu at (205.2, 93.0)
- added Q4: MMBT3904, Package_TO_SOT_SMD:SOT-23, F.Cu at (213.7, 84.4)
- added R17: 220, Resistor_SMD:R_0603_1608Metric, F.Cu at (244.4, 81.5)
- added R18: 200k, Resistor_SMD:R_0603_1608Metric, F.Cu at (235.5, 84.0)
- added R19: 4.7k, Resistor_SMD:R_0603_1608Metric, F.Cu at (231.4, 91.6)
- added R20: 4.7k, Resistor_SMD:R_0603_1608Metric, F.Cu at (235.5, 86.6)
- added R21: 1k, Resistor_SMD:R_0603_1608Metric, F.Cu at (235.5, 89.1)
- added R22: 220, Resistor_SMD:R_0603_1608Metric, F.Cu at (239.6, 84.0)
- added R23: 100, Resistor_SMD:R_0603_1608Metric, F.Cu at (231.4, 89.1)
- added R24: 1k, Resistor_SMD:R_0603_1608Metric, F.Cu at (227.1, 94.1)
- added R25: 4.7k, Resistor_SMD:R_0603_1608Metric, F.Cu at (222.2, 100.9)
- added R26: 220, Resistor_SMD:R_0603_1608Metric, F.Cu at (231.1, 94.1)
- added R27: 1k, Resistor_SMD:R_0603_1608Metric, F.Cu at (239.6, 86.6)
- added R28: 220, Resistor_SMD:R_0603_1608Metric, F.Cu at (240.4, 81.5)
- added R29: 10k, Resistor_SMD:R_0603_1608Metric_Pad0.98x0.95mm_HandSolder, F.Cu at (251.9, 79.0)
- added R30: 31k, Resistor_SMD:R_0603_1608Metric, F.Cu at (120.5, 109.7)
- added R31: 10k, Resistor_SMD:R_0603_1608Metric, F.Cu at (114.4, 120.3)
- added R32: 13k, Resistor_SMD:R_0603_1608Metric, F.Cu at (118.4, 115.2)
- added R33: 10k, Resistor_SMD:R_0603_1608Metric, F.Cu at (120.5, 112.2)
- added SW1: SW_Push, Button_Switch_SMD:SW_Push_1P1T-SH_NO_CK_KMR2xxG, F.Cu at (209.9, 70.1)
- added SW2: SW_Push, Button_Switch_SMD:SW_Push_1P1T-SH_NO_CK_KMR2xxG, F.Cu at (216.5, 70.1)
- added U15: PI4ULS3V302XVEX, pi4uls3v302:PSON40P160X120X55-8N, F.Cu at (210.1, 127.7)
- added U16: PI4ULS3V302XVEX, pi4uls3v302:PSON40P160X120X55-8N, F.Cu at (216.7, 127.7)
- added U17: PI4ULS3V302XVEX, pi4uls3v302:PSON40P160X120X55-8N, F.Cu at (210.1, 134.1)
- added U18: PI4ULS3V302XVEX, pi4uls3v302:PSON40P160X120X55-8N, F.Cu at (216.7, 130.9)
- added U19: PI4ULS3V302XVEX, pi4uls3v302:PSON40P160X120X55-8N, F.Cu at (216.7, 134.1)
- added U20: PI4ULS3V302XVEX, pi4uls3v302:PSON40P160X120X55-8N, F.Cu at (233.7, 127.7)
- added U21: PI4ULS3V302XVEX, pi4uls3v302:PSON40P160X120X55-8N, F.Cu at (237.0, 127.7)
- added U22: PI4ULS3V302XVEX, pi4uls3v302:PSON40P160X120X55-8N, F.Cu at (230.3, 127.7)
- added U23: AP62300Z6, Package_TO_SOT_SMD:SOT-563, F.Cu at (122.3, 115.1)
- added U24: AP62300Z6, Package_TO_SOT_SMD:SOT-563, F.Cu at (105.0, 116.7)
- added U25: AP62300Z6, Package_TO_SOT_SMD:SOT-563, F.Cu at (104.7, 111.2)
- added U7: PI4ULS3V302XVEX, pi4uls3v302:PSON40P160X120X55-8N, F.Cu at (220.0, 130.9)
- C1, C10, C11, C12, C13, C14, C15, C16, C17, C18, C19, C2, C20, C21, C22, C23, C24, C25, C3, C34, C4, C5, C7, C8: footprint Capacitor_SMD:C_0603_1608Metric_Pad1.08x0.95mm_HandSolder -> Capacitor_SMD:C_0603_1608Metric
- C26, C27, C28, C29, C30, C31: value 1uF -> 100nF
- C6, C9: value 4.7uF -> 100nF; footprint Capacitor_SMD:C_0603_1608Metric_Pad1.08x0.95mm_HandSolder -> Capacitor_SMD:C_0603_1608Metric
- D9: value MMBD4448HADW -> LED; footprint Package_TO_SOT_SMD:SOT-363_SC-70-6 -> LED_SMD:LED_0603_1608Metric
- R8: value 10k -> 1k; footprint Resistor_SMD:R_0603_1608Metric_Pad0.98x0.95mm_HandSolder -> Resistor_SMD:R_0603_1608Metric
- U10: value TLV71209_SOT23-5 -> PI4ULS3V302XVEX; footprint Package_TO_SOT_SMD:SOT-23-5 -> pi4uls3v302:PSON40P160X120X55-8N
- U13: value W25Q128JVS -> PI4ULS3V302XVEX; footprint Package_SO:SOIC-8_5.23x5.23mm_P1.27mm -> pi4uls3v302:PSON40P160X120X55-8N
- U14: value CV32E40P -> CORE-V-MCU
- U3: value 74LVC1G125 -> W25Q32JWZP; footprint Package_TO_SOT_SMD:SOT-353_SC-70-5 -> Package_SON:WSON-8-1EP_6x5mm_P1.27mm_EP3.4x4.3mm
- U4: value 74LVC1G125 -> PI6ULS5V9306WEX; footprint Package_TO_SOT_SMD:SOT-353_SC-70-5 -> Package_SO:SOIC-8_3.9x4.9mm_P1.27mm
- U5: value 74LVC1G125 -> MAX6842DUKD0+T; footprint Package_TO_SOT_SMD:SOT-353_SC-70-5 -> MAX6842:MAX6842DUKD0&plus_T
- U6, U7: value 74LVC1G125 -> PI4ULS3V302XVEX; footprint Package_TO_SOT_SMD:SOT-353_SC-70-5 -> pi4uls3v302:PSON40P160X120X55-8N
- U8: value LM1117-3.3 -> PI4ULS3V302XVEX; footprint Package_TO_SOT_SMD:SOT-223-3_TabPin2 -> pi4uls3v302:PSON40P160X120X55-8N
- U9: value LM1117-1.8 -> PI4ULS3V302XVEX; footprint Package_TO_SOT_SMD:SOT-223-3_TabPin2 -> pi4uls3v302:PSON40P160X120X55-8N
- X1: value SG-8002LB -> ECS-2520MVLC-100-CN; footprint Oscillator:Oscillator_SMD_SeikoEpson_SG8002LB-4Pin_5.0x3.2mm -> Oscillator:Oscillator_SMD_ECS_2520MV-xxx-xx-4Pin_2.5x2.0mm
- moved D9 114.2 mm to (231.2, 66.0)
- moved C6 107.9 mm to (231.9, 81.5)
- moved C29 107.2 mm to (240.6, 79.0)
- moved C31 105.9 mm to (227.6, 79.0)
- moved C9 103.2 mm to (227.3, 89.1)
- moved R8 92.5 mm to (226.0, 96.6)
- moved U6 89.8 mm to (213.4, 130.9), turned to 0 degrees
- moved U8 89.6 mm to (220.0, 127.7), turned to 0 degrees
- moved C30 85.2 mm to (218.6, 94.1)
- moved C28 83.5 mm to (209.9, 92.0)
- moved C26 82.4 mm to (213.7, 98.0), turned to 0 degrees
- moved U9 80.8 mm to (213.4, 127.7), turned to 0 degrees
- moved C27 79.6 mm to (209.3, 96.5), turned to 0 degrees
- moved U10 78.7 mm to (210.1, 130.9), turned to 0 degrees
- moved U3 73.1 mm to (206.6, 87.5), turned to 0 degrees
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Connections:
- net Net-(U14-Pad48) renamed 10MHZ_CLOCK_SOC
- net camera_d0 renamed CAMERA_D0
- net camera_hsync renamed CAMERA_HSYNC
- net camera_int renamed /camera/camera_int
- net camera_trig renamed /camera/camera_trig
- net camera_vsync renamed CAMERA_VSYNC
- net el_reset renamed /ExpressLink/~{EL_RESET}
- C18 pad 1: /jtag and uart/ft_1v8 -> +1V8
- C19 pad 1: /jtag and uart/ft_1v8 -> +1V8
- C20 pad 1: /jtag and uart/ft_1v8 -> +1V8
- C21 pad 1: VCC -> +1V8
- C22 pad 1: VCC -> +1V8
- C23 pad 1: VCC -> +1V8
- C24 pad 1: VCC -> +3V3
- C25 pad 1: VCC -> +3V3
- C26 pad 1: +5V -> +1V8
- C27 pad 1: +5V -> +3V3
- C28 pad 1: +3V3 -> +1V8
- C31 pad 1: 0.9V -> Net-(C31-Pad1)
- C6 pad 1: +3V3 -> Net-(C6-Pad1)
- C9 pad 1: /jtag and uart/ft_1v8 -> +3V3
- CON1 pad P11: SDA0 -> SDA
- CON1 pad P12: SCL0 -> SCL
- CON1 pad P13: click_tx -> CLICK_TX
- CON1 pad P14: click_rx -> CLICK_RX
- CON1 pad P15: irq -> /mikrobus and sensors/click_int
- CON1 pad P16: pwm -> /mikrobus and sensors/click_pwm
- CON1 pad P2: reset -> /mikrobus and sensors/click_rst
- CON1 pad P3: CS0 -> /mikrobus and sensors/click_cs
- CON1 pad P4: SCLK0 -> /mikrobus and sensors/click_sck
- CON1 pad P5: MOSI0 -> /mikrobus and sensors/click_miso
- CON1 pad P6: MOSI0 -> /mikrobus and sensors/click_mosi
- D9 pad 1: (no net) -> Net-(D9-Pad1)
- D9 pad 2: +5V -> +3V3
- J4 pad 1: +3V3 -> Net-(J4-Pad1)
- J4 pad 2: Net-(J4-Pad2) -> GND
- J5 pad 1: +3V3 -> +1V8
- J5 pad 10: nRESET -> TRST
- J6 pad 12: /camera/camera_d4 -> CAMERA_D4
- J6 pad 13: /camera/camera_d7 -> CAMERA_D7
- J6 pad 17: camera_pclk -> CAMERA_PCLK
- J6 pad 19: /camera/camera_d6 -> CAMERA_D6
- J6 pad 20: /camera/camera_d5 -> CAMERA_D5
- J6 pad 21: SCL0 -> CAMERA_SCL
- J6 pad 22: SDA0 -> CAMERA_SDA
- J6 pad 3: /camera/camera_d1 -> CAMERA_D1
- J6 pad 5: /camera/camera_d3 -> CAMERA_D3
- J6 pad 8: camera_mclk -> CAMERA_MCLK
- J6 pad 9: /camera/camera_d2 -> CAMERA_D2
- R14 pad 2: temp_alert -> /mikrobus and sensors/temperature_alert
- R15 pad 1: +3V3 -> SCL0_SOC
- R15 pad 2: SCL0 -> +1V8
- R16 pad 1: +3V3 -> SDA0_SOC
- R16 pad 2: SDA0 -> +1V8
- R8 pad 1: GND -> Net-(Q1-Pad1)
- R8 pad 2: Net-(J4-Pad2) -> USER_LED_SOC
- U1 pad 16: el_event -> /ExpressLink/EL_EVENT
- U1 pad 26: el_tx -> EL_TX
- U1 pad 27: el_rx -> EL_RX
- U1 pad 6: el_wake -> /ExpressLink/EL_WAKE
- U10 pad 1: +3V3 -> +1V8
- U10 pad 2: GND -> SCLK0
- U10 pad 3: +3V3 -> MOSI0
- U10 pad 4: unconnected-(U10-Pad4) -> GND
- U10 pad 5: 0.9V -> +1V8
- U11 pad 1: SDA0 -> SDA
- U11 pad 2: SCL0 -> SCL
- U11 pad 3: temp_alert -> /mikrobus and sensors/temperature_alert
- U13 pad 1: unconnected-(U13-Pad1) -> +1V8
- U13 pad 2: unconnected-(U13-Pad2) -> MOSI0
- U13 pad 3: unconnected-(U13-Pad3) -> CLICK_PWM
- U13 pad 5: unconnected-(U13-Pad5) -> +1V8
- U13 pad 6: unconnected-(U13-Pad6) -> /mikrobus and sensors/click_pwm
- U13 pad 7: unconnected-(U13-Pad7) -> /mikrobus and sensors/click_mosi
- U14 pad 11: unconnected-(U14-Pad11) -> 0.8V
- U14 pad 13: unconnected-(U14-Pad13) -> 0.8V
- U14 pad 14: unconnected-(U14-Pad14) -> CLICK_RESET_SOC
- U14 pad 15: unconnected-(U14-Pad15) -> PGM_FLASH_DATA2_SOC
- U14 pad 16: unconnected-(U14-Pad16) -> PGM_FLASH_DATA3_SOC
- U14 pad 19: SCL0 -> SCL0_SOC
- U14 pad 20: SDA0 -> SDA0_SOC
- U14 pad 22: unconnected-(U14-Pad22) -> +1V8
- U14 pad 24: unconnected-(U14-Pad24) -> +1V8
- U14 pad 26: (no net) -> SCLK0_SOC
- U14 pad 27: (no net) -> MISO0_SOC
- U14 pad 28: (no net) -> FPGA_LED0
- U14 pad 3: unconnected-(U14-Pad3) -> RX1_MUX1_SOC
- U14 pad 31: unconnected-(U14-Pad31) -> 0.8V
- U14 pad 33: unconnected-(U14-Pad33) -> 0.8V
- U14 pad 34: (no net) -> CLICK_PWM_SOC
- U14 pad 35: (no net) -> EL_RESET_SOC
- U14 pad 36: (no net) -> USER_LED_SOC
- U14 pad 37: (no net) -> FPGA_LED1
- U14 pad 38: (no net) -> FPGA_LED2
- U14 pad 4: unconnected-(U14-Pad4) -> PGM_FLASH_CS
- U14 pad 41: (no net) -> unconnected-(U14-Pad41)
- U14 pad 42: (no net) -> unconnected-(U14-Pad42)
- U14 pad 43: TDO -> TCK
- U14 pad 45: TMS -> TDO
- U14 pad 46: TCK -> TMS
- U14 pad 47: unconnected-(U14-Pad47) -> TRST
- U14 pad 5: unconnected-(U14-Pad5) -> PGM_FLASH_DATA0
- U14 pad 51: unconnected-(U14-Pad51) -> 0.8V
- U14 pad 53: unconnected-(U14-Pad53) -> 0.8V
- U14 pad 55: unconnected-(U14-Pad55) -> nRESET_SOC
- U14 pad 56: console_tx -> RX0_SOC
- U14 pad 57: console_rx -> TX0_SOC
- U14 pad 58: TX1 -> TX1_MUX0_SOC
- U14 pad 59: RX1 -> RX1_MUX0_SOC
- U14 pad 6: unconnected-(U14-Pad6) -> PGM_FLASH_DATA1
- U14 pad 60: UART_MUX -> TX1_MUX1_SOC
- U14 pad 61: camera_mclk -> CAMERA_PCLK
- U14 pad 62: pwm -> CAMERA_MCLK
- U14 pad 63: irq -> EL_EVENT_SOC
- U14 pad 64: reset -> CLICK_IRQ_SOC
- U14 pad 66: unconnected-(U14-Pad66) -> CAMERA_D1
- U14 pad 67: unconnected-(U14-Pad67) -> CAMERA_D2
- U14 pad 68: unconnected-(U14-Pad68) -> CAMERA_D3
- U14 pad 7: unconnected-(U14-Pad7) -> PGM_FLASH_CLK
- U14 pad 71: unconnected-(U14-Pad71) -> 0.8V
- U14 pad 73: unconnected-(U14-Pad73) -> 0.8V
- U14 pad 74: unconnected-(U14-Pad74) -> CAMERA_D4
- U14 pad 75: unconnected-(U14-Pad75) -> CAMERA_D5
- U14 pad 76: unconnected-(U14-Pad76) -> CAMERA_D6
- U14 pad 77: unconnected-(U14-Pad77) -> CAMERA_D7
- U14 pad 78: unconnected-(U14-Pad78) -> EL_WAKE_SOC
- U14 pad 79: unconnected-(U14-Pad79) -> CS0_SOC
- U14 pad 8: unconnected-(U14-Pad8) -> USER_BUTTON
- U14 pad 80: unconnected-(U14-Pad80) -> MOSI0_SOC
- U2 pad 12: /jtag and uart/ft_1v8 -> +1V8
- U2 pad 37: /jtag and uart/ft_1v8 -> +1V8
- U2 pad 48: console_tx -> CONSOLE_TX
- U2 pad 49: /jtag and uart/ft_1v8 -> unconnected-(U2-Pad49)
- U2 pad 50: +3V3 -> unconnected-(U2-Pad50)
- U2 pad 52: console_rx -> CONSOLE_RX
- U2 pad 64: /jtag and uart/ft_1v8 -> +1V8
- U3 pad 1: Net-(J4-Pad2) -> PGM_FLASH_CS
- U3 pad 2: TDI -> PGM_FLASH_DATA1
- U3 pad 3: GND -> PGM_FLASH_DATA2
- U3 pad 4: Net-(U2-Pad17) -> GND
- U3 pad 5: VCC -> PGM_FLASH_DATA0
- U4 pad 1: Net-(J4-Pad2) -> GND
- U4 pad 2: Net-(U2-Pad16) -> +1V8
- U4 pad 3: GND -> SCL0_SOC
- U4 pad 4: TCK -> SDA0_SOC
- U4 pad 5: VCC -> SDA
- U5 pad 1: Net-(J4-Pad2) -> nRESET_SOC
- U5 pad 2: Net-(U2-Pad18) -> GND
- U5 pad 3: GND -> unconnected-(U5-Pad3)
- U5 pad 4: TDO -> Net-(SW2-Pad2)
- U5 pad 5: VCC -> +1V8
- U6 pad 1: Net-(J4-Pad2) -> +1V8
- U6 pad 2: Net-(U2-Pad19) -> TX0_SOC
- U6 pad 3: GND -> RX0_SOC
- U6 pad 4: TMS -> GND
- U6 pad 5: VCC -> +1V8
- U7 pad 1: Net-(J4-Pad2) -> +1V8
- U7 pad 2: Net-(U2-Pad23) -> TX1_MUX0_SOC
- U7 pad 3: GND -> RX1_MUX0_SOC
- U7 pad 4: nRESET -> GND
- U7 pad 5: VCC -> +1V8
- U8 pad 1: GND -> +1V8
- U8 pad 2: +3V3 -> TX1_MUX1_SOC
- U8 pad 3: +5V -> RX1_MUX1_SOC
- U9 pad 1: GND -> +1V8
- U9 pad 2: +1V8 -> TEMP_ALERT
- U9 pad 3: +5V -> CS0
- X1 pad 1: GND -> +1V8
- X1 pad 4: +3V3 -> +1V8
Routing:
- net GND: track 95.6 -> 0.00 mm, vias 40 -> 0
- net +3V3: track 56.7 -> 0.00 mm, vias 7 -> 0
- net Net-(D7-Pad1): track 24.0 -> 0.00 mm, vias 2 -> 0
- net Net-(J4-Pad2): track 23.0 -> 0.00 mm, vias 8 -> 0
- net /jtag and uart/ft_1v8: track 18.9 -> 0.00 mm
- net VCC: track 17.0 -> 0.00 mm
- net Net-(D1-Pad1): track 15.4 -> 0.00 mm
- net Net-(D6-Pad1): track 13.7 -> 0.00 mm, vias 2 -> 0
- net Net-(J1-Pad6): track 12.3 -> 0.00 mm, vias 1 -> 0
- net Net-(J2-Pad3): track 11.9 -> 0.00 mm, vias 1 -> 0
- net Net-(J3-PadA5): track 11.8 -> 0.00 mm
- net Net-(J3-PadB5): track 11.3 -> 0.00 mm, vias 2 -> 0
- net Net-(J1-Pad4): track 11.1 -> 0.00 mm, vias 1 -> 0
- net Net-(J1-Pad2): track 11.0 -> 0.00 mm, vias 1 -> 0
- net Net-(D5-Pad1): track 10.7 -> 0.00 mm, vias 2 -> 0
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