File: OpenHW DevKit.kicad_pcb (KiCad board)
At the start: 4 copper layers, 100 x 75 mm, 185 parts, among them CON1 MIKROBUS_HOST_CONN, J1 Conn_02x05_Odd_Even, J2 Conn_02x03_Odd_Even, J3 USB_C_Receptacle, J4 Conn_01x02_Male, J5 3220-10-0100-00, J6 Conn_01x24, Q1 MMBT3904, Q2 MMBT3904, Q3 MMBT3904, Q4 MMBT3904, SW1 SW_Push, SW2 SW_Push, U1 ESP32-C3-MINI-1, U10 PI4ULS3V302XVEX, U11 MCP9808, U12 AP2127K-2.8, U13 PI4ULS3V302XVEX, U14 CORE-V-MCU, U15 PI4ULS3V302XVEX, U16 PI4ULS3V302XVEX, U17 PI4ULS3V302XVEX, U18 PI4ULS3V302XVEX, U19 PI4ULS3V302XVEX, U2 FT2232HL-REEL, U20 PI4ULS3V302XVEX, U21 PI4ULS3V302XVEX, U22 PI4ULS3V302XVEX, U23 AP62300Z6, U24 AP62300Z6, U25 AP62300Z6, U3 W25Q32JWZP, U4 PI6ULS5V9306WEX, U5 MAX6842DUKD0+T, U6 PI4ULS3V302XVEX, U7 PI4ULS3V302XVEX, U8 PI4ULS3V302XVEX, U9 PI4ULS3V302XVEX, X1 ECS-2520MVLC-100-CN, Y1 32.768kHz, Y2 12MHz

Commit message: pcb updates including level shifter adjustments
Parts:
- removed the U7 at (134.1, 75.4)
- moved U21 146.2 mm to (99.5, 78.0)
- moved U20 138.3 mm to (105.6, 75.6)
- moved U22 133.3 mm to (105.6, 80.8)
- moved R29 125.4 mm to (126.8, 88.2)
- moved R23 109.0 mm to (128.7, 125.5)
- moved SW1 108.8 mm to (119.4, 130.6), turned to 180 degrees
- moved C31 107.7 mm to (128.6, 121.7)
- moved SW2 106.6 mm to (128.7, 130.6), turned to 180 degrees
- moved C83 103.4 mm to (151.1, 116.7), turned to -90 degrees
- moved R25 99.8 mm to (126.0, 127.3)
- moved C80 98.6 mm to (141.4, 106.3), turned to 180 degrees
- moved R27 96.0 mm to (155.2, 132.4)
- moved R28 95.7 mm to (156.8, 128.1)
- moved C29 94.8 mm to (146.7, 92.2)
- moved C77 90.4 mm to (148.7, 96.4), turned to 90 degrees
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Connections:
- net EL_RESET_SOC renamed ~{EL_RESET_SOC}
- net Net-(D1-Pad1) renamed /jtag and uart/VBUS
- net nRESET_SOC renamed ~{RESET_SOC}
- C34 pad 1: /ExpressLink/~{EL_RESET} -> /~{EL_RESET}
- CON1 pad P15: /mikrobus and sensors/click_int -> /CLICK_INT
- CON1 pad P16: /mikrobus and sensors/click_pwm -> /CLICK_PWM
- CON1 pad P2: /mikrobus and sensors/click_rst -> /CLICK_RST
- CON1 pad P3: /mikrobus and sensors/click_cs -> /CLICK_CS
- CON1 pad P4: /mikrobus and sensors/click_sck -> /CLICK_SCK
- CON1 pad P5: /mikrobus and sensors/click_miso -> /CLICK_MISO
- CON1 pad P6: /mikrobus and sensors/click_mosi -> /CLICK_MOSI
- R1 pad 2: /ExpressLink/~{EL_RESET} -> /~{EL_RESET}
- U1 pad 16: /ExpressLink/EL_EVENT -> /EL_EVENT
- U1 pad 26: EL_TX -> /EL_TXD
- U1 pad 27: EL_RX -> /EL_RXD
- U1 pad 6: /ExpressLink/EL_WAKE -> /EL_WAKE
- U1 pad 8: /ExpressLink/~{EL_RESET} -> /~{EL_RESET}
- U10 pad 2: SCLK0 -> CLICK_IRQ_SOC
- U10 pad 3: MOSI0 -> EL_EVENT_SOC
- U10 pad 6: /mikrobus and sensors/click_miso -> /EL_EVENT
- U10 pad 7: /mikrobus and sensors/click_sck -> /CLICK_PWM
- U13 pad 2: MOSI0 -> TX1_MUX1_SOC
- U13 pad 3: CLICK_PWM -> unconnected-(U13-Pad3)
- U13 pad 6: /mikrobus and sensors/click_pwm -> unconnected-(U13-Pad6)
- U13 pad 7: /mikrobus and sensors/click_mosi -> CLICK_RX
- U14 pad 11: 0.8V -> +0V8
- U14 pad 13: 0.8V -> +0V8
- U14 pad 15: PGM_FLASH_DATA2_SOC -> PGM_FLASH_DATA2
- U14 pad 16: PGM_FLASH_DATA3_SOC -> PGM_FLASH_DATA3
- U14 pad 31: 0.8V -> +0V8
- U14 pad 33: 0.8V -> +0V8
- U14 pad 51: 0.8V -> +0V8
- U14 pad 53: 0.8V -> +0V8
- U14 pad 71: 0.8V -> +0V8
- U14 pad 73: 0.8V -> +0V8
- U15 pad 2: CLICK_IRQ -> unconnected-(U15-Pad2)
- U15 pad 3: CLICK_RESET -> unconnected-(U15-Pad3)
- U15 pad 6: /mikrobus and sensors/click_rst -> unconnected-(U15-Pad6)
- U15 pad 7: /mikrobus and sensors/click_int -> unconnected-(U15-Pad7)
- U16 pad 2: TX1_MUX1_SOC -> unconnected-(U16-Pad2)
- U16 pad 3: RX1_MUX1_SOC -> unconnected-(U16-Pad3)
- U16 pad 6: CLICK_TX -> unconnected-(U16-Pad6)
- U16 pad 7: CLICK_RX -> unconnected-(U16-Pad7)
- U17 pad 2: TX1_MUX0_SOC -> unconnected-(U17-Pad2)
- U17 pad 3: RX1_MUX0_SOC -> unconnected-(U17-Pad3)
- U17 pad 6: EL_TX -> unconnected-(U17-Pad6)
- U17 pad 7: EL_RX -> unconnected-(U17-Pad7)
- U18 pad 2: EL_EVENT -> unconnected-(U18-Pad2)
- U18 pad 3: EL_WAKE -> unconnected-(U18-Pad3)
- U18 pad 6: /ExpressLink/EL_WAKE -> unconnected-(U18-Pad6)
- U18 pad 7: /ExpressLink/EL_EVENT -> unconnected-(U18-Pad7)
- U19 pad 2: EL_RESET -> unconnected-(U19-Pad2)
- U19 pad 7: /ExpressLink/~{EL_RESET} -> unconnected-(U19-Pad7)
- U6 pad 8: unconnected-(U6-Pad8) -> +3V3
- U7 pad 2: TX1_MUX0_SOC -> RX1_MUX0_SOC
- U7 pad 3: RX1_MUX0_SOC -> TX1_MUX0_SOC
- U7 pad 6: EL_TX -> EL_RX
- U7 pad 7: EL_RX -> EL_TX
- U8 pad 2: TX1_MUX1_SOC -> RX1_MUX1_SOC
- U8 pad 3: RX1_MUX1_SOC -> MOSI0_SOC
- U8 pad 6: CLICK_TX -> /CLICK_MOSI
- U8 pad 7: CLICK_RX -> CLICK_TX
- U9 pad 2: TEMP_ALERT -> CS0_SOC
- U9 pad 3: CS0 -> EL_WAKE_SOC
- U9 pad 6: /mikrobus and sensors/click_cs -> /EL_WAKE
- U9 pad 7: /mikrobus and sensors/temperature_alert -> /CLICK_CS
Routing:
- net GND: track 0.00 -> 54.0 mm, vias 0 -> 20
- net +1V8: track 0.00 -> 31.5 mm, vias 0 -> 6
- net osci: track 0.00 -> 13.6 mm
- net Net-(C10-Pad1): track 0.00 -> 13.1 mm
- net +0V8: track 0.00 -> 12.6 mm, vias 0 -> 2
- net Net-(J3-PadA5): track 0.00 -> 12.0 mm
- net osco: track 0.00 -> 10.3 mm
- net MOSI0_SOC: track 0.00 -> 9.85 mm
- net Net-(J3-PadB5): track 0.00 -> 9.85 mm
- net +3V3: track 0.00 -> 9.63 mm
- net RX1_MUX1_SOC: track 0.00 -> 9.57 mm
- net PGM_FLASH_DATA0: track 0.00 -> 8.98 mm
- net /jtag and uart/d-: track 0.00 -> 8.92 mm, vias 0 -> 2
- net PGM_FLASH_DATA3: track 0.00 -> 8.57 mm
- net /jtag and uart/d+: track 0.00 -> 8.26 mm, vias 0 -> 2
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