File: OpenHW DevKit.kicad_pcb (KiCad board)
At the start: 4 copper layers, 100 x 75 mm, 184 parts, among them CON1 MIKROBUS_HOST_CONN, J1 Conn_02x05_Odd_Even, J2 Conn_02x03_Odd_Even, J3 USB_C_Receptacle, J4 Conn_01x02_Male, J5 3220-10-0100-00, J6 Conn_01x24, Q1 MMBT3904, Q2 MMBT3904, Q3 MMBT3904, Q4 MMBT3904, SW1 SW_Push, SW2 SW_Push, U1 ESP32-C3-MINI-1, U10 PI4ULS3V302XVEX, U11 MCP9808, U12 AP2127K-2.8, U13 PI4ULS3V302XVEX, U14 CORE-V-MCU, U15 PI4ULS3V302XVEX, U16 PI4ULS3V302XVEX, U17 PI4ULS3V302XVEX, U18 PI4ULS3V302XVEX, U19 PI4ULS3V302XVEX, U2 FT2232HL-REEL, U20 PI4ULS3V302XVEX, U21 PI4ULS3V302XVEX, U22 PI4ULS3V302XVEX, U23 AP62300Z6, U24 AP62300Z6, U25 AP62300Z6, U3 W25Q32JWZP, U4 PI6ULS5V9306WEX, U5 MAX6842DUKD0+T, U6 PI4ULS3V302XVEX, U7 PI4ULS3V302XVEX, U8 PI4ULS3V302XVEX, U9 PI4ULS3V302XVEX, X1 ECS-2520MVLC-100-CN, Y1 32.768kHz, Y2 12MHz

Commit message: sync with schematic
Parts:
- moved U16 44.0 mm to (130.6, 100.1)
- moved U18 35.9 mm to (133.5, 96.6)
- moved C29 14.5 mm to (134.7, 100.3)
- moved R15 7.01 mm to (191.4, 99.9)
- moved U5 4.67 mm to (166.7, 109.3)
- moved R16 1.28 mm to (190.4, 97.2)
Routing:
- net CAMERA_D4: track 2.97 -> 65.4 mm, vias 0 -> 2
- net CAMERA_D3: track 4.20 -> 65.3 mm, vias 0 -> 2
- net CAMERA_D1: track 4.32 -> 64.9 mm, vias 0 -> 2
- net CAMERA_D5: track 2.92 -> 63.4 mm
- net CAMERA_D7: track 5.52 -> 65.8 mm
- net CAMERA_D6: track 5.52 -> 64.4 mm
- net CAMERA_D2: track 4.26 -> 62.6 mm, vias 0 -> 2
- net CAMERA_D0: track 4.38 -> 58.8 mm, vias 0 -> 2
- net CAMERA_MCLK: track 5.73 -> 49.8 mm, vias 0 -> 2
- net CAMERA_PCLK: track 5.57 -> 49.2 mm, vias 0 -> 2

Commit message: Update bottom and right edges of board wiring
Place components along bottom and right edge of board.
Parts:
- moved C55 56.2 mm to (160.1, 106.3)
- moved C82 46.8 mm to (163.2, 107.8), turned to 180 degrees
- moved U5 38.2 mm to (134.8, 130.3)
- moved R8 26.0 mm to (160.1, 121.7), turned to 90 degrees
- moved C35 25.2 mm to (193.0, 134.5)
- moved C33 25.2 mm to (194.2, 128.5)
- moved D10 24.3 mm to (151.5, 131.8), turned to 0 degrees
- moved R26 24.1 mm to (151.5, 130.2), turned to 180 degrees
- moved JP3 23.4 mm to (191.1, 111.7), turned to -90 degrees
- moved Q3 22.1 mm to (151.3, 126.5), turned to -90 degrees
- moved R21 22.0 mm to (149.9, 121.8), turned to 90 degrees
- moved C6 21.3 mm to (190.3, 90.9), turned to -90 degrees
- moved D8 20.6 mm to (161.2, 131.6), turned to 180 degrees
- moved R24 20.6 mm to (152.2, 121.8)
- moved R17 20.3 mm to (161.2, 130.0), turned to 180 degrees
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Routing:
- net GND: track 54.0 -> 106.4 mm, vias 20 -> 26
- net +3V3: track 9.63 -> 60.4 mm, vias 0 -> 3
- net SDA: track 0.00 -> 27.0 mm
- net SCL: track 0.00 -> 19.8 mm
- net +1V8: track 31.5 -> 46.3 mm, vias 6 -> 9
- net Net-(C6-Pad1): track 0.00 -> 8.09 mm
- net +0V8: track 12.6 -> 19.9 mm, vias 2 -> 3
- net Net-(JP3-Pad1): track 0.00 -> 6.84 mm
- net Net-(JP4-Pad1): track 0.00 -> 6.60 mm
- net Net-(JP5-Pad1): track 0.00 -> 6.56 mm
- net 10MHZ_CLOCK_SOC: track 0.00 -> 5.46 mm
- net Net-(Q1-Pad1): track 0.00 -> 4.10 mm
- net Net-(Q4-Pad1): track 0.00 -> 3.85 mm
- net Net-(Q2-Pad1): track 0.00 -> 3.78 mm
- net RX0_SOC: track 2.65 -> 6.12 mm
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
Commit message: Rework the SOC pinout
Parts:
- added C84: 100nF, Capacitor_SMD:C_0603_1608Metric, F.Cu at (148.8, 98.4)
- added C85: 100nF, Capacitor_SMD:C_0603_1608Metric, F.Cu at (157.7, 106.9)
- added C86: 100nF, Capacitor_SMD:C_0603_1608Metric, F.Cu at (147.5, 117.2)
- added C87: 100nF, Capacitor_SMD:C_0603_1608Metric, F.Cu at (139.5, 108.2)
- moved C65 79.7 mm to (135.2, 80.8), turned to 180 degrees
- moved C63 76.0 mm to (143.1, 80.8), turned to 180 degrees
- moved C49 75.1 mm to (139.0, 80.8), turned to 180 degrees
- moved C58 72.9 mm to (135.1, 77.0), turned to 180 degrees
- moved C59 70.3 mm to (141.5, 99.1), turned to 90 degrees
- moved C66 67.5 mm to (139.0, 77.0), turned to 180 degrees
- moved C79 65.1 mm to (145.0, 122.4)
- moved C60 64.7 mm to (143.1, 77.0), turned to 180 degrees
- moved C44 59.9 mm to (184.2, 76.1), turned to 180 degrees
- moved R25 59.0 mm to (184.8, 123.3)
- moved SW1 57.2 mm to (176.6, 131.8)
- moved C57 56.1 mm to (157.7, 108.5)
- moved R23 53.8 mm to (182.4, 127.4)
- moved SW2 53.8 mm to (182.5, 131.8)
- moved U15 49.9 mm to (184.0, 74.2)
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Connections:
- CON1 pad P13: CLICK_TX -> /CLICK_TX
- CON1 pad P14: CLICK_RX -> /CLICK_RX
- U10 pad 2: CLICK_IRQ_SOC -> CLICK_RESET_SOC
- U10 pad 3: EL_EVENT_SOC -> unconnected-(U10-Pad3)
- U10 pad 6: /EL_EVENT -> unconnected-(U10-Pad6)
- U10 pad 7: /CLICK_PWM -> /CLICK_RST
- U13 pad 2: TX1_MUX1_SOC -> CLICK_PWM_SOC
- U13 pad 3: unconnected-(U13-Pad3) -> CLICK_IRQ_SOC
- U13 pad 6: unconnected-(U13-Pad6) -> /CLICK_INT
- U13 pad 7: CLICK_RX -> /CLICK_PWM
- U14 pad 14: CLICK_RESET_SOC -> PGM_FLASH_DATA3
- U14 pad 15: PGM_FLASH_DATA2 -> PGM_FLASH_CLK
- U14 pad 16: PGM_FLASH_DATA3 -> PGM_FLASH_DATA0
- U14 pad 17: CAMERA_VSYNC -> TMS
- U14 pad 18: CAMERA_HSYNC -> TCK
- U14 pad 19: SCL0_SOC -> TDO
- U14 pad 20: SDA0_SOC -> TDI
- U14 pad 26: SCLK0_SOC -> TRST
- U14 pad 27: MISO0_SOC -> unconnected-(U14-Pad27)
- U14 pad 28: FPGA_LED0 -> unconnected-(U14-Pad28)
- U14 pad 3: RX1_MUX1_SOC -> SCLK0_SOC
- U14 pad 34: CLICK_PWM_SOC -> unconnected-(U14-Pad34)
- U14 pad 35: ~{EL_RESET_SOC} -> unconnected-(U14-Pad35)
- U14 pad 36: USER_LED_SOC -> unconnected-(U14-Pad36)
- U14 pad 37: FPGA_LED1 -> unconnected-(U14-Pad37)
- U14 pad 38: FPGA_LED2 -> unconnected-(U14-Pad38)
- U14 pad 4: PGM_FLASH_CS -> MISO0_SOC
- U14 pad 43: TCK -> unconnected-(U14-Pad43)
- U14 pad 44: TDI -> unconnected-(U14-Pad44)
- U14 pad 45: TDO -> unconnected-(U14-Pad45)
- U14 pad 46: TMS -> unconnected-(U14-Pad46)
- U14 pad 47: TRST -> unconnected-(U14-Pad47)
- U14 pad 5: PGM_FLASH_DATA0 -> MOSI0_SOC
- U14 pad 55: ~{RESET_SOC} -> unconnected-(U14-Pad55)
- U14 pad 56: RX0_SOC -> CAMERA_D5
- U14 pad 57: TX0_SOC -> CAMERA_D6
- U14 pad 58: TX1_MUX0_SOC -> CAMERA_PCLK
- U14 pad 59: RX1_MUX0_SOC -> CAMERA_HSYNC
- U14 pad 6: PGM_FLASH_DATA1 -> PGM_FLASH_DATA2
- U14 pad 60: TX1_MUX1_SOC -> CAMERA_D0
- U14 pad 61: CAMERA_PCLK -> CAMERA_D7
- U14 pad 62: CAMERA_MCLK -> CAMERA_D4
- U14 pad 63: EL_EVENT_SOC -> CAMERA_D2
- U14 pad 64: CLICK_IRQ_SOC -> CAMERA_MCLK
- U14 pad 65: CAMERA_D0 -> CAMERA_VSYNC
- U14 pad 66: CAMERA_D1 -> CAMERA_D3
- U14 pad 67: CAMERA_D2 -> CAMERA_D1
- U14 pad 68: CAMERA_D3 -> SCL0_SOC
- U14 pad 7: PGM_FLASH_CLK -> PGM_FLASH_DATA1
- U14 pad 74: CAMERA_D4 -> SDA0_SOC
- U14 pad 75: CAMERA_D5 -> TX1_MUX1_SOC
- U14 pad 76: CAMERA_D6 -> RX1_MUX1_SOC
- U14 pad 77: CAMERA_D7 -> CLICK_IRQ_SOC
- U14 pad 78: EL_WAKE_SOC -> CLICK_PWM_SOC
- U14 pad 79: CS0_SOC -> CLICK_RESET_SOC
- U14 pad 8: USER_BUTTON -> PGM_FLASH_CS
- U14 pad 80: MOSI0_SOC -> CS0_SOC
- U15 pad 2: unconnected-(U15-Pad2) -> RX1_MUX1_SOC
- U15 pad 3: unconnected-(U15-Pad3) -> TX1_MUX1_SOC
- U15 pad 6: unconnected-(U15-Pad6) -> /CLICK_TX
- U15 pad 7: unconnected-(U15-Pad7) -> /CLICK_RX
- U17 pad 2: unconnected-(U17-Pad2) -> RX1_MUX0_SOC
- U17 pad 3: unconnected-(U17-Pad3) -> TX1_MUX0_SOC
- U17 pad 6: unconnected-(U17-Pad6) -> /EL_RXD
- U17 pad 7: unconnected-(U17-Pad7) -> /EL_TXD
- U18 pad 2: unconnected-(U18-Pad2) -> EL_EVENT_SOC
- U18 pad 7: unconnected-(U18-Pad7) -> /EL_EVENT
- U19 pad 2: unconnected-(U19-Pad2) -> EL_WAKE_SOC
- U19 pad 3: unconnected-(U19-Pad3) -> ~{EL_RESET_SOC}
- U19 pad 6: unconnected-(U19-Pad6) -> /~{EL_RESET}
- U19 pad 7: unconnected-(U19-Pad7) -> /EL_WAKE
- U7 pad 2: RX1_MUX0_SOC -> unconnected-(U7-Pad2)
- U7 pad 3: TX1_MUX0_SOC -> unconnected-(U7-Pad3)
- U7 pad 6: EL_RX -> unconnected-(U7-Pad6)
- U7 pad 7: EL_TX -> unconnected-(U7-Pad7)
- U8 pad 2: RX1_MUX1_SOC -> SCLK0_SOC
- U8 pad 3: MOSI0_SOC -> CS0_SOC
- U8 pad 6: /CLICK_MOSI -> /CLICK_CS
- U8 pad 7: CLICK_TX -> /CLICK_SCK
- U9 pad 2: CS0_SOC -> MOSI0_SOC
- U9 pad 3: EL_WAKE_SOC -> MISO0_SOC
- U9 pad 6: /EL_WAKE -> /CLICK_MISO
- U9 pad 7: /CLICK_CS -> /CLICK_MOSI
Routing:
- net CLICK_PWM_SOC: track 0.00 -> 55.5 mm
- net CLICK_RESET_SOC: track 0.00 -> 53.5 mm
- net CLICK_IRQ_SOC: track 3.56 -> 55.6 mm
- net SCL0_SOC: track 2.05 -> 53.7 mm
- net SCLK0_SOC: track 0.00 -> 47.7 mm
- net TX1_MUX1_SOC: track 7.85 -> 51.0 mm
- net MISO0_SOC: track 0.00 -> 42.8 mm
- net CS0_SOC: track 5.24 -> 47.6 mm
- net SDA0_SOC: track 2.14 -> 43.8 mm
- net RX1_MUX1_SOC: track 9.57 -> 50.9 mm
- net CAMERA_D7: track 65.8 -> 24.7 mm
- net CAMERA_D4: track 65.4 -> 25.4 mm, vias 2 -> 0
- net CAMERA_D3: track 65.3 -> 28.8 mm, vias 2 -> 0
- net CAMERA_D2: track 62.6 -> 26.5 mm, vias 2 -> 0
- net CAMERA_D6: track 64.4 -> 29.0 mm
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- added copper zone on In2.Cu, net +0V8
- removed copper zone on In2.Cu, net +1V8

Commit message: New pinout (old symbol)
Parts:
- moved C42 7.75 mm to (124.8, 102.9)
- moved C32 7.75 mm to (130.1, 102.9)
- moved C41 7.75 mm to (126.4, 102.9)
- moved C82 7.75 mm to (121.1, 102.9)
- moved U6 7.75 mm to (122.9, 102.9)
- moved U7 7.75 mm to (128.3, 102.9)
Connections:
- U14 pad 27: unconnected-(U14-Pad27) -> TX1_MUX0_SOC
- U14 pad 28: unconnected-(U14-Pad28) -> RX1_MUX0_SOC
- U14 pad 34: unconnected-(U14-Pad34) -> EL_EVENT_SOC
- U14 pad 35: unconnected-(U14-Pad35) -> ~{EL_RESET_SOC}
- U14 pad 36: unconnected-(U14-Pad36) -> EL_WAKE_SOC
- U14 pad 37: unconnected-(U14-Pad37) -> RX0_SOC
- U14 pad 38: unconnected-(U14-Pad38) -> TX0_SOC
- U14 pad 43: unconnected-(U14-Pad43) -> USER_LED_SOC
- U14 pad 44: unconnected-(U14-Pad44) -> FPGA_LED0
- U14 pad 45: unconnected-(U14-Pad45) -> FPGA_LED1
- U14 pad 46: unconnected-(U14-Pad46) -> FPGA_LED2
- U14 pad 47: unconnected-(U14-Pad47) -> ~{RESET_SOC}
- U14 pad 55: unconnected-(U14-Pad55) -> USER_BUTTON
Routing:
- net EL_WAKE_SOC: track 19.7 -> 38.2 mm
- net ~{EL_RESET_SOC}: track 19.1 -> 37.1 mm
- net EL_EVENT_SOC: track 19.0 -> 36.2 mm
- net RX1_MUX0_SOC: track 22.3 -> 35.6 mm
- net TX1_MUX0_SOC: track 21.7 -> 34.4 mm
- net ~{RESET_SOC}: track 0.00 -> 11.0 mm
- net unconnected-(U14-Pad47): track 11.0 -> 0.00 mm
- net unconnected-(U14-Pad2): track 0.00 -> 3.10 mm

Commit message: revised pinout
Parts:
- moved R19 55.1 mm to (166.2, 122.4)
- moved R20 54.3 mm to (166.2, 124.0)
- moved R15 43.6 mm to (155.5, 122.5)
- moved C76 43.6 mm to (155.5, 120.9)
- moved R16 43.6 mm to (155.5, 124.1)
- moved U4 43.6 mm to (160.8, 121.9)
- moved C6 43.6 mm to (163.1, 118.3)
- moved R18 43.6 mm to (163.1, 116.7)
- moved C31 15.4 mm to (182.9, 132.0), turned to -90 degrees
- moved SW2 11.1 mm to (171.4, 131.9)
- moved C30 10.3 mm to (186.7, 127.5)
- moved C46 8.32 mm to (188.4, 99.3)
- moved JP3 8.32 mm to (181.0, 93.2)
- moved JP4 8.32 mm to (181.0, 96.0)
- moved JP5 8.32 mm to (181.0, 98.8)
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Connections:
- J6 pad 21: CAMERA_SCL -> SCL0_SOC
- J6 pad 22: CAMERA_SDA -> SDA0_SOC
- U14 pad 17: TMS -> RX0_SOC
- U14 pad 18: TCK -> TX0_SOC
- U14 pad 19: TDO -> TX1_MUX0_SOC
- U14 pad 20: TDI -> RX1_MUX0_SOC
- U14 pad 26: TRST -> SCLK0_SOC
- U14 pad 27: TX1_MUX0_SOC -> MISO0_SOC
- U14 pad 28: RX1_MUX0_SOC -> MOSI0_SOC
- U14 pad 3: SCLK0_SOC -> TX1_MUX1_SOC
- U14 pad 37: RX0_SOC -> USER_LED_SOC
- U14 pad 38: TX0_SOC -> FPGA_LED0
- U14 pad 4: MISO0_SOC -> RX1_MUX1_SOC
- U14 pad 43: USER_LED_SOC -> TMS
- U14 pad 44: FPGA_LED0 -> TCK
- U14 pad 45: FPGA_LED1 -> TDO
- U14 pad 46: FPGA_LED2 -> TDI
- U14 pad 47: ~{RESET_SOC} -> TRST
- U14 pad 5: MOSI0_SOC -> CLICK_RESET_SOC
- U14 pad 55: USER_BUTTON -> ~{RESET_SOC}
- U14 pad 56: CAMERA_D5 -> USER_BUTTON
- U14 pad 57: CAMERA_D6 -> SCL0_SOC
- U14 pad 58: CAMERA_PCLK -> SDA0_SOC
- U14 pad 60: CAMERA_D0 -> CAMERA_VSYNC
- U14 pad 61: CAMERA_D7 -> FPGA_LED1
- U14 pad 62: CAMERA_D4 -> FPGA_LED2
- U14 pad 63: CAMERA_D2 -> CAMERA_D5
- U14 pad 64: CAMERA_MCLK -> CAMERA_D6
- U14 pad 65: CAMERA_VSYNC -> CAMERA_PCLK
- U14 pad 66: CAMERA_D3 -> CAMERA_D0
- U14 pad 67: CAMERA_D1 -> CAMERA_D7
- U14 pad 68: SCL0_SOC -> CAMERA_D4
- U14 pad 74: SDA0_SOC -> CAMERA_D2
- U14 pad 75: TX1_MUX1_SOC -> CAMERA_MCLK
- U14 pad 76: RX1_MUX1_SOC -> CAMERA_D3
- U14 pad 77: CLICK_IRQ_SOC -> CAMERA_D1
- U14 pad 78: CLICK_PWM_SOC -> CLICK_IRQ_SOC
- U14 pad 79: CLICK_RESET_SOC -> CLICK_PWM_SOC
Routing:
- net USER_BUTTON: track 0.00 -> 36.8 mm
- net TMS: track 14.1 -> 46.5 mm
- net TCK: track 14.4 -> 46.7 mm
- net TDO: track 14.7 -> 46.9 mm
- net TDI: track 15.1 -> 47.1 mm
- net MOSI0_SOC: track 42.3 -> 73.7 mm
- net MISO0_SOC: track 42.8 -> 73.7 mm
- net SCLK0_SOC: track 47.7 -> 77.7 mm
- net Net-(SW2-Pad2): track 0.00 -> 27.7 mm
- net TRST: track 19.8 -> 47.3 mm
- net USER_LED_SOC: track 17.9 -> 34.8 mm, vias 0 -> 2
- net FPGA_LED0: track 14.1 -> 30.9 mm, vias 0 -> 2
- net SDA: track 34.7 -> 22.0 mm
- net GND: track 97.6 -> 109.9 mm, vias 35 -> 45
- net +1V8: track 52.6 -> 64.1 mm, vias 13 -> 18
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
Commit message: Changed to KiCAD 7 and updated to final pinout.
Parts:
- removed C21, C22, C23, C24, C25, C26, C27, C30, C38, C39, C42, C43, C44, C46, C47, C52, C53, C54, C56, C58, C60, C62, C64, C66, C67: 100nF, Capacitor_SMD:C_0603_1608Metric
- removed U15, U16, U17, U18, U19, U20, U21, U22: PI4ULS3V302XVEX, pi4uls3v302:PSON40P160X120X55-8N
- added J10: Conn_01x20, Connector_PinHeader_1.00mm:PinHeader_1x20_P1.00mm_Vertical, F.Cu at (138.5, 114.0)
- added J7: Conn_01x20, Connector_PinHeader_1.00mm:PinHeader_1x20_P1.00mm_Vertical, F.Cu at (160.0, 112.0)
- added J8: Conn_01x20, Connector_PinHeader_1.00mm:PinHeader_1x20_P1.00mm_Vertical, F.Cu at (157.5, 90.0)
- added J9: Conn_01x20, Connector_PinHeader_1.00mm:PinHeader_1x20_P1.00mm_Vertical, F.Cu at (136.0, 93.0)
- added JP2: SolderJumper_2_Bridged, Jumper:SolderJumper-2_P1.3mm_Bridged_RoundedPad1.0x1.5mm, F.Cu at (162.8, 112.9)
- added JP6: SolderJumper_2_Bridged, Jumper:SolderJumper-2_P1.3mm_Bridged_RoundedPad1.0x1.5mm, F.Cu at (162.8, 110.3)
- added JP7: SolderJumper_2_Bridged, Jumper:SolderJumper-2_P1.3mm_Bridged_RoundedPad1.0x1.5mm, F.Cu at (133.2, 91.4)
- added JP8: SolderJumper_2_Bridged, Jumper:SolderJumper-2_P1.3mm_Bridged_RoundedPad1.0x1.5mm, F.Cu at (133.2, 94.0)
- added SYM*1: ~, logos:devkits_qr, F.Cu at (149.6, 124.6)
- added TP1: TestPoint, TestPoint:TestPoint_Pad_D1.0mm, F.Cu at (133.7, 106.0)
- added TP2: 5v0, TestPoint:TestPoint_Loop_D2.54mm_Drill1.5mm_Beaded, F.Cu at (102.9, 98.3)
- added TP3: 3v3, TestPoint:TestPoint_Loop_D2.54mm_Drill1.5mm_Beaded, F.Cu at (102.9, 103.3)
- added TP4: 1v8, TestPoint:TestPoint_Loop_D2.54mm_Drill1.5mm_Beaded, F.Cu at (102.9, 108.4)
- added TP5: 0v8, TestPoint:TestPoint_Loop_D2.54mm_Drill1.5mm_Beaded, F.Cu at (102.9, 113.5)
- added TP6: GND, TestPoint:TestPoint_Loop_D2.54mm_Drill1.5mm_Beaded, F.Cu at (102.9, 118.5)
- C34: value 10uF -> 100nF
- JP3, JP4, JP5: moved to F.Cu
- SW1, SW2: footprint Button_Switch_SMD:SW_Push_1P1T-SH_NO_CK_KMR2xxG -> Button:TS204225WT160SMTTR
- U10, U13, U6, U7, U8, U9: value PI4ULS3V302XVEX -> NTB0104BQ,115; footprint pi4uls3v302:PSON40P160X120X55-8N -> NTB0104:NXP_Semiconductors-SOT762-1-08_2019-0-MFG
- U4: value PI6ULS5V9306WEX -> FXMA2102UMX; footprint Package_SO:SOIC-8_3.9x4.9mm_P1.27mm -> FXMA2102UMX:FXMA2102UMX
- moved C78 92.4 mm to (113.2, 101.9)
- moved C75 91.9 mm to (113.2, 100.4)
- moved C81 91.9 mm to (113.2, 103.4)
- moved C48 85.8 mm to (126.0, 97.5), turned to 180 degrees
- moved C68 80.0 mm to (126.0, 103.5), turned to 180 degrees
- moved U13 67.9 mm to (127.5, 106.5), turned to 90 degrees
- moved U6 62.0 mm to (174.8, 68.9), turned to 90 degrees
- moved C50 59.8 mm to (173.1, 72.0), turned to 180 degrees
- moved U10 57.2 mm to (127.5, 100.5), turned to 90 degrees
- moved C41 55.1 mm to (173.1, 73.7), turned to 180 degrees
- moved C33 54.4 mm to (162.7, 82.3), turned to -90 degrees
- moved U7 53.4 mm to (174.8, 76.7), turned to 90 degrees
- moved U9 49.8 mm to (127.5, 94.5), turned to 90 degrees
- moved C76 43.8 mm to (113.2, 109.6), turned to 0 degrees
- moved C32 39.8 mm to (164.3, 82.3), turned to -90 degrees
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Connections:
- C6 pad 1: Net-(C6-Pad1) -> Net-(U4-OE)
- J4 pad 1: Net-(J4-Pad1) -> Net-(J4-Pin_1)
- R18 pad 1: Net-(C6-Pad1) -> Net-(U4-OE)
- R29 pad 1: Net-(J4-Pad1) -> Net-(J4-Pin_1)
- U10 pad 2: CLICK_RESET_SOC -> TCK
- U10 pad 3: unconnected-(U10-Pad3) -> TDI
- U10 pad 4: GND -> TDO
- U10 pad 5: +1V8 -> TMS
- U10 pad 7: /CLICK_RST -> GND
- U10 pad 8: +3V3 -> Net-(J4-Pin_1)
- U13 pad 2: CLICK_PWM_SOC -> TRST
- U13 pad 3: CLICK_IRQ_SOC -> unconnected-(U13-A2-Pad3)
- U13 pad 4: GND -> unconnected-(U13-A3-Pad4)
- U13 pad 5: +1V8 -> unconnected-(U13-A4-Pad5)
- U13 pad 6: /CLICK_INT -> unconnected-(U13-NC-Pad6)
- U13 pad 7: /CLICK_PWM -> GND
- U13 pad 8: +3V3 -> Net-(J4-Pin_1)
- U14 pad 1: unconnected-(U14-Pad1) -> VPW_P
- U14 pad 14: PGM_FLASH_DATA3 -> PGM_FLASH_DATA0
- U14 pad 15: PGM_FLASH_CLK -> PGM_FLASH_DATA1
- U14 pad 16: PGM_FLASH_DATA0 -> CLICK_RESET_SOC
- U14 pad 17: RX0_SOC -> USER_BUTTON
- U14 pad 18: TX0_SOC -> SCL0_SOC
- U14 pad 19: TX1_MUX0_SOC -> SDA0_SOC
- U14 pad 2: unconnected-(U14-Pad2) -> VNW_N
- U14 pad 20: RX1_MUX0_SOC -> CAMERA_HSYNC
- U14 pad 22: +1V8 -> (no net)
- U14 pad 23: GND -> +1V8
- U14 pad 24: +1V8 -> GND
- U14 pad 25: (no net) -> +1V8
- U14 pad 26: SCLK0_SOC -> (no net)
- U14 pad 27: MISO0_SOC -> (no net)
- U14 pad 28: MOSI0_SOC -> SCLK0_SOC
- U14 pad 29: GND -> MISO0_SOC
- U14 pad 3: TX1_MUX1_SOC -> CAMERA_VSYNC
- U14 pad 30: GND -> CS0_SOC
- U14 pad 31: +0V8 -> GND
- U14 pad 32: +1V8 -> GND
- U14 pad 34: EL_EVENT_SOC -> +1V8
- U14 pad 35: ~{EL_RESET_SOC} -> +0V8
- U14 pad 36: EL_WAKE_SOC -> CAMERA_D5
- U14 pad 37: USER_LED_SOC -> ~{EL_RESET_SOC}
- U14 pad 38: FPGA_LED0 -> CLICK_IRQ_SOC
- U14 pad 39: unconnected-(U14-Pad39) -> EL_WAKE_SOC
- U14 pad 4: RX1_MUX1_SOC -> TX1_MUX1_SOC
- U14 pad 40: unconnected-(U14-Pad40) -> MOSI0_SOC
- U14 pad 41: unconnected-(U14-Pad41) -> NB
- U14 pad 42: unconnected-(U14-Pad42) -> PB
- U14 pad 43: TMS -> TDI
- U14 pad 44: TCK -> TMS
- U14 pad 46: TDI -> TCK
- U14 pad 5: CLICK_RESET_SOC -> PGM_FLASH_DATA3
- U14 pad 54: unconnected-(U14-Pad54) -> POWER_DETECT
- U14 pad 56: USER_BUTTON -> PGM_FLASH_CS
- U14 pad 57: SCL0_SOC -> TX1_MUX0_SOC
- U14 pad 58: SDA0_SOC -> RX1_MUX0_SOC
- U14 pad 59: CAMERA_HSYNC -> TX0_SOC
- U14 pad 6: PGM_FLASH_DATA2 -> PGM_FLASH_CLK
- U14 pad 60: CAMERA_VSYNC -> RX0_SOC
- U14 pad 61: FPGA_LED1 -> USER_LED_SOC
- U14 pad 62: FPGA_LED2 -> FPGA_LED0
- U14 pad 63: CAMERA_D5 -> CAMERA_MCLK
- U14 pad 64: CAMERA_D6 -> CAMERA_D3
- U14 pad 65: CAMERA_PCLK -> FPGA_LED1
- U14 pad 66: CAMERA_D0 -> CAMERA_PCLK
- U14 pad 67: CAMERA_D7 -> CAMERA_D1
- U14 pad 68: CAMERA_D4 -> CAMERA_D2
- U14 pad 7: PGM_FLASH_DATA1 -> PGM_FLASH_DATA2
- U14 pad 74: CAMERA_D2 -> CAMERA_D7
- U14 pad 75: CAMERA_MCLK -> FPGA_LED2
- U14 pad 76: CAMERA_D3 -> CAMERA_D4
- U14 pad 77: CAMERA_D1 -> CAMERA_D0
- U14 pad 78: CLICK_IRQ_SOC -> CAMERA_D6
- U14 pad 79: CLICK_PWM_SOC -> EL_EVENT_SOC
- U14 pad 8: PGM_FLASH_CS -> RX1_MUX1_SOC
- U14 pad 80: CS0_SOC -> CLICK_PWM_SOC
- U2 pad 16: Net-(U2-Pad16) -> Net-(U10-B1)
- U2 pad 17: Net-(U2-Pad17) -> Net-(U10-B2)
- U2 pad 18: Net-(U2-Pad18) -> Net-(U10-B3)
- U2 pad 19: Net-(U2-Pad19) -> Net-(U10-B4)
- U2 pad 23: Net-(U2-Pad23) -> Net-(U13-B1)
- U4 pad 1: GND -> Net-(U4-OE)
- U4 pad 2: +1V8 -> SCL
- U4 pad 3: SCL0_SOC -> SDA
- U4 pad 4: SDA0_SOC -> GND
- U4 pad 5: SDA -> Net-(U4-OE)
- U4 pad 6: SCL -> SDA0_SOC
- U4 pad 7: Net-(C6-Pad1) -> SCL0_SOC
- U4 pad 8: Net-(C6-Pad1) -> +1V8
- U6 pad 2: TX0_SOC -> EL_EVENT_SOC
- U6 pad 3: RX0_SOC -> RX1_MUX0_SOC
- U6 pad 4: GND -> TX1_MUX0_SOC
- U6 pad 5: +1V8 -> CLICK_RESET_SOC
- U6 pad 6: CONSOLE_TX -> unconnected-(U6-NC-Pad6)
- U6 pad 7: CONSOLE_RX -> GND
- U6 pad 8: +3V3 -> +1V8
- U7 pad 2: unconnected-(U7-Pad2) -> MOSI0_SOC
- U7 pad 3: unconnected-(U7-Pad3) -> MISO0_SOC
- U7 pad 4: GND -> SCLK0_SOC
- U7 pad 5: +1V8 -> CS0_SOC
- U7 pad 7: unconnected-(U7-Pad7) -> GND
- U7 pad 8: +3V3 -> +1V8
- U8 pad 2: SCLK0_SOC -> CLICK_PWM_SOC
- U8 pad 3: CS0_SOC -> CLICK_IRQ_SOC
- U8 pad 4: GND -> RX1_MUX1_SOC
- U8 pad 5: +1V8 -> TX1_MUX1_SOC
- U8 pad 6: /CLICK_CS -> unconnected-(U8-NC-Pad6)
- U8 pad 7: /CLICK_SCK -> GND
- U8 pad 8: +3V3 -> +1V8
- U9 pad 2: MOSI0_SOC -> TX0_SOC
- U9 pad 3: MISO0_SOC -> RX0_SOC
- U9 pad 4: GND -> EL_WAKE_SOC
- U9 pad 5: +1V8 -> ~{EL_RESET_SOC}
- U9 pad 6: /CLICK_MISO -> unconnected-(U9-NC-Pad6)
- U9 pad 7: /CLICK_MOSI -> GND
- U9 pad 8: +3V3 -> +1V8
Routing:
- net +1V8: track 64.1 -> 331.6 mm, vias 18 -> 36
- net TX1_MUX0_SOC: track 38.6 -> 111.9 mm, vias 2 -> 5
- net +3V3: track 33.5 -> 105.3 mm, vias 12 -> 28
- net RX1_MUX0_SOC: track 39.2 -> 108.9 mm, vias 2 -> 6
- net SCL: track 24.5 -> 88.8 mm, vias 0 -> 2
- net SDA: track 22.0 -> 86.1 mm
- net Net-(U13-B1): track 0.00 -> 55.1 mm, vias 0 -> 2
- net Net-(U10-B2): track 0.00 -> 52.8 mm, vias 0 -> 2
- net CAMERA_D5: track 21.9 -> 74.2 mm, vias 0 -> 3
- net Net-(U10-B3): track 0.00 -> 51.7 mm, vias 0 -> 2
- net Net-(U10-B4): track 0.00 -> 50.4 mm, vias 0 -> 2
- net Net-(U10-B1): track 0.00 -> 46.7 mm, vias 0 -> 2
- net ~{RESET_SOC}: track 6.67 -> 51.7 mm, vias 0 -> 2
- net +0V8: track 25.6 -> 69.6 mm, vias 4 -> 10
- net PGM_FLASH_CS: track 6.21 -> 45.0 mm, vias 0 -> 2
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- added copper zone on F.Cu, net +0V8
- added copper zone on F.Cu, net +1V8
- added copper zone on In2.Cu, net +1V8
- added copper zone on F.Cu, net +3V3
- added copper zone on In1.Cu, net +3V3
- added copper zone on F.Cu, net +5V
- added copper zone on F.Cu, net /jtag and uart/VBUS
- added copper zone on B.Cu, net GND
- added copper zone on F.Cu, net GND
Other:
- outline, holes or cut-outs redrawn
- board text added: "A0"
- board text added: "A1"
- board text added: "A2"
- board text added: "AWS IoT ExpressLink"
- board text added: "Ashling Opella-LD Onboard Debug"
- board text added: "CORE-V MCU"
- board text added: "CS"
- board text added: "Camera Interface"
- board text added: "EMPTY"
- board text added: "FPGA LED 0 IO47"
- board text added: "FPGA LED 1 IO25"
- board text added: "FPGA LED 2 IO26"
- board text added: "I2C Address 0011-A2-A1-A0 Default : 0011000 (0x18)"
- board text added: "INT"
- board text added: "IO12"
- board text added: "IO13"
- board text added: "IO14"
- board text added: "IO37"
- board text added: "IO38"
- board text added: "IO39"
- board text added: "IO40"
- board text added: "IO41"
- board text added: "IO42"
- board text added: "IO7 User Button"
- board text added: "IO8"
- board text added: "IO9"
- board text added: "MISO"
- board text added: "MOSI"
- board text added: "Opella-LD Disable"
- board text added: "RESET"
- board text added: "RST"
- board text added: "RX"
- board text added: "SCK"
- board text added: "TX"
- board text added: "Temperature Sensor MCP9808"
- board text added: "USER LED IO46"
- board text removed: "Ashling Opella-LD Debug"

Commit message: Updated camera and button models
Other:
- board text added: "+5V Not Connected"
Changed lines of the file:
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@@
     (pad "2" smd rect (at 2.075 1.075 270) (size 0.65 1.05) (layers "F.Cu" "F.Paste" "F.Mask")
       (net 36 "Net-(C31-Pad1)") (pinfunction "2") (pintype "passive"))
-    (model "TS20-42-25-WT-160-SMT-TR.stp"
+    (model "${KIPRJMOD}/project parts/3.2x4.2 button.step"
       (offset (xyz 0 0 0))
       (scale (xyz 1 1 1))
@@
       (rotate (xyz 0 90 180))
     )
-    (model "${KIPRJMOD}/project parts/HM01B0 Camera.step"
+    (model "${KIPRJMOD}/project parts/HIMAX Camera.step"
       (offset (xyz 3.5 -21.5 0.5))
       (scale (xyz 0.9 0.9 0.9))
@@
     (pad "2" smd rect (at 2.075 1.075 270) (size 0.65 1.05) (layers "F.Cu" "F.Paste" "F.Mask")
       (net 152 "Net-(U5-*MR)") (pinfunction "2") (pintype "passive"))
-    (model "TS20-42-25-WT-160-SMT-TR.stp"
+    (model "${KIPRJMOD}/project parts/3.2x4.2 button.step"
       (offset (xyz 0 0 0))
       (scale (xyz 1 1 1))
@@
     (effects (font (size 0.635 0.635) (thickness 0.127) bold))
   )
+  (gr_text "+5V Not Connected" (at 186.7 88.1) (layer "F.SilkS")
+    (effects (font (size 0.635 0.635) (thickness 0.127)))
+  )
   (gr_text "MISO" (at 170.4 76) (layer "F.SilkS")
