File: OpenHW DevKit.kicad_pcb (KiCad board)
At the start: 4 copper layers, 100 x 75 mm, 179 parts, among them CON1 MIKROBUS_HOST_CONN, J1 Conn_02x05_Odd_Even, J10 Conn_01x20, J11 Conn_01x02_Male, J2 Conn_02x03_Odd_Even, J3 USB_C_Receptacle, J4 Conn_01x02_Male, J5 3220-10-0100-00, J6 Conn_01x24, J7 Conn_01x20, J8 Conn_01x20, J9 Conn_01x20, Q1 MMBT3904, Q2 MMBT3904, SW1 SW_Push, SW2 SW_Push, U1 ESP32-C3-MINI-1, U10 NTB0104BQ,115, U11 MCP9808, U12 AP2127K-2.8, U13 NTB0104BQ,115, U14 CORE-V-MCU, U15 MP6400DG-01-LF-Z, U16 MP6400DG-01-LF-Z, U2 FT2232HL-REEL, U23 AP62300Z6, U24 AP62300Z6, U25 AP62300Z6, U3 W25Q32JWZP, U4 FXMA2102UMX, U5 MP6400DG-01-LF-Z, U6 NTB0104BQ,115, U7 NTB0104BQ,115, U8 NTB0104BQ,115, U9 NTB0104BQ,115, X1 ECS-2520MVLC-100-CN, Y1 32.768kHz, Y2 12MHz

Commit message: updated some text and removed an old picture
Routing:
- net +3V3: track 81.4 -> 94.7 mm, vias 30 -> 31
- net GND: track 66.7 -> 70.5 mm, vias 61 -> 62
- net /jtag and uart/d-: track 11.2 -> 11.8 mm
- net Net-(U13-B4): track 42.2 -> 42.7 mm

Commit message: updated the QR code and added shield coupling to the usb connector
Parts:
- added C27: 12.5pF, Capacitor_SMD:C_0603_1608Metric, F.Cu at (126.7, 64.3)
- added C30: 12.5pF, Capacitor_SMD:C_0603_1608Metric, F.Cu at (126.7, 66.0)
- added R24: 1M, Resistor_SMD:R_0603_1608Metric_Pad0.98x0.95mm_HandSolder, F.Cu at (126.9, 62.5)
- moved SYM*1 0.80 mm to (148.8, 124.6)
Connections:
- J3 pad S1: GND -> /jtag and uart/shield
Routing:
- net /jtag and uart/shield: track 0.00 -> 11.7 mm
- net USER_BUTTON: track 62.4 -> 63.1 mm
- added copper zone on B.Cu, net /jtag and uart/shield
- added copper zone on F.Cu, net /jtag and uart/shield

Commit message: adjusted track spacing and cleared DRC
Routing:
- net GND: track 70.5 -> 76.9 mm, vias 62 -> 68
- net CAMERA_D6: track 41.8 -> 45.4 mm
- net CAMERA_D5: track 42.6 -> 46.1 mm
- net CAMERA_D4: track 44.8 -> 43.1 mm
- net CAMERA_D7: track 45.5 -> 44.2 mm
- net CAMERA_D0: track 46.2 -> 44.9 mm
- net CAMERA_VSYNC: track 59.4 -> 60.6 mm
- net CAMERA_PCLK: track 46.0 -> 45.2 mm
- net CAMERA_HSYNC: track 57.8 -> 56.9 mm
- net Net-(U4-OE): track 10.6 -> 11.5 mm
- net TRST: track 30.0 -> 29.2 mm
- net /EL_TXD: track 15.5 -> 16.2 mm
- net CS0_SOC: track 66.7 -> 66.0 mm
- net CAMERA_D1: track 38.6 -> 39.3 mm
- net SDA0_SOC: track 52.2 -> 51.6 mm
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