File: OpenHW DevKit.kicad_sch (KiCad schematic)
At the start: 4 parts

Commit message: added solderpad license text to each sheet
Other:
- note added: "Copyright and related rights are licensed under the Solderpad Hardware License, Version 0.51 (the "License"); you may not use this file except in compliance with the License. You may obtain a copy of the License at http://solderpad.org/licenses/SHL-0.51. Unless required by applicable law or agreed to in writing, software, hardware and materials distributed under this License is distributed on an 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"
Changed lines of the file:
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@@
     )
+  )
+  (text "Copyright and related rights are licensed under the Solderpad Hardware License, Version 0.51 (the \"License\");\nyou may not use this file except in compliance with the License.  You may obtain a copy of the License at\nhttp://solderpad.org/licenses/SHL-0.51. Unless required by applicable law or agreed to in writing, software,\nhardware and materials distributed under this License is distributed on an \"AS IS\" BASIS, WITHOUT WARRANTIES OR\nCONDITIONS OF ANY KIND, either express or implied. See the License for the specific language governing\npermissions and limitations under the License.\n"
+    (at 179.07 177.8 0)
+    (effects (font (size 1 1)) (justify left bottom))
   )
   (symbol (lib_id "Mechanical:MountingHole") (at 22.86 149.86 0) (unit 1)

Commit message: added the camera, temperature sensor and basic MCU symbol
Parts:
- added R15, R16: 4.7k, Resistor_SMD:R_0603_1608Metric, symbol Device:R
- added U?: W25Q128JVS, Package_SO:SOIC-8_5.23x5.23mm_P1.27mm, symbol Memory_Flash:W25Q128JVS
- added U?: CV32E40P, Package_QFP:LQFP-80_12x12mm_P0.5mm, symbol OpenHW:CV32E40P
- added X?: SG-8002LB, Oscillator:Oscillator_SMD_SeikoEpson_SG8002LB-4Pin_5.0x3.2mm, symbol Oscillator:SG-8002LB
Connections:
- net ExpressLink/EL_EVENT: now also U?. (Vdd_3v3)
- net ExpressLink/EL_RXD: now also U?. (Vdd_3v3)
- net ExpressLink/EL_TXD: now also U?. (Vdd_3v3)
- net ExpressLink/EL_WAKE: now also U?. (Vdd_3v3)
- net ExpressLink/~{EL_RESET}: now also U?. (Vdd_3v3)
- net jtag and uart/FT_RXD: now also U?. (Vdd_3v3)
- net jtag and uart/FT_TXD: now also U?. (Vdd_3v3)
- net jtag and uart/TCK: now also U?. (Vdd_3v3)
- net jtag and uart/TDI: now also U?. (Vdd_3v3)
- net jtag and uart/TDO: now also U?. (Vdd_3v3)
- net jtag and uart/TMS: now also U?. (Vdd_3v3)
- new net: U?. (Vdd_3v3), U?.1 (~{CS})
- new net: U?. (Vdd_3v3), U?.2 (DO(IO1))
- new net: U?. (Vdd_3v3), U?.3 (IO2)
- new net: U?. (Vdd_3v3), U?.5 (DI(IO0))
- new net: U?. (Vdd_3v3), U?.6 (CLK)
- new net: U?. (Vdd_3v3), U?.7 (IO3)
- new net: U?. (Vdd_3v3), X?.3 (OUT)
- new net +1V8: U?. (Vdd_3v3)
- new net +3V3: R15.1, R16.1, U?. (Vdd_3v3), U?.8 (VCC), X?.4 (Vcc)
- new net 0.9V: U?. (Vdd_3v3)
- new net GND: U?. (Vdd_3v3), U?.4 (GND), X?.1 (OE), X?.2 (GND)
- new net RX1: U?. (Vdd_3v3)
- new net TX1: U?. (Vdd_3v3)
- new net camera/camera_d0: U?. (Vdd_3v3)
- new net camera/camera_d1: U?. (Vdd_3v3)
- new net camera/camera_d2: U?. (Vdd_3v3)
- new net camera/camera_d3: U?. (Vdd_3v3)
- new net camera/camera_d4: U?. (Vdd_3v3)
- new net camera/camera_d5: U?. (Vdd_3v3)
- new net camera/camera_d6: U?. (Vdd_3v3)
- new net camera/camera_d7: U?. (Vdd_3v3)
- new net camera/camera_hsync: U?. (Vdd_3v3)
- new net camera/camera_int: U?. (Vdd_3v3)
- new net camera/camera_mclk: U?. (Vdd_3v3)
- new net camera/camera_pclk: U?. (Vdd_3v3)
- new net camera/camera_trig: U?. (Vdd_3v3)
- new net camera/camera_vsync: U?. (Vdd_3v3)
- new net camera/i2c_scl: R15.2, U?. (Vdd_3v3)
- new net camera/i2c_sda: R16.2, U?. (Vdd_3v3)
- new net mikrobus and sensors/click_an: U?. (Vdd_3v3)
- new net mikrobus and sensors/click_cs: U?. (Vdd_3v3)
- new net mikrobus and sensors/click_int: U?. (Vdd_3v3)
- new net mikrobus and sensors/click_miso: U?. (Vdd_3v3)
- new net mikrobus and sensors/click_mosi: U?. (Vdd_3v3)
- new net mikrobus and sensors/click_pwm: U?. (Vdd_3v3)
- new net mikrobus and sensors/click_rst: U?. (Vdd_3v3)
- new net mikrobus and sensors/click_rx: U?. (Vdd_3v3)
- new net mikrobus and sensors/click_sck: U?. (Vdd_3v3)
- new net mikrobus and sensors/click_tx: U?. (Vdd_3v3)
- new net mikrobus and sensors/temperature_alert: U?. (Vdd_3v3)
Other:
- sheet mikrobus renamed mikrobus and sensors
- added sheet camera (camera.kicad_sch)
- sheet mikrobus and sensors ports: added click_an, click_cs, click_int, click_miso, click_mosi, click_pwm, click_rst, click_rx, click_sck, click_tx, scl, sda, temperature_alert; removed none
- note added: "Copyright and related rights are licensed under the Solderpad Hardware License, Version 2.1 (the "License"); you may not use this file except in compliance with the License. You may obtain a copy of the License at http://solderpad.org/licenses/SHL-2.1. Unless required by applicable law or agreed to in writing, software, hardware and materials distributed under this License is distributed on an "A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"
- note added: "NOTE: This symbol is representative of the final device and does not currently match the device in development."
- note removed: "Copyright and related rights are licensed under the Solderpad Hardware License, Version 0.51 (the "License"); you may not use this file except in compliance with the License. You may obtain a copy of the License at http://solderpad.org/licenses/SHL-0.51. Unless required by applicable law or agreed to in writing, software, hardware and materials distributed under this License is distributed on an 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"
- moved on the sheet: H1, H2, H3, H4

Commit message: MCU pinout finalized
Parts:
- removed U?: CV32E40P, Package_QFP:LQFP-80_12x12mm_P0.5mm, symbol OpenHW:CV32E40P
- added C?: 100nF, Capacitor_SMD:C_0603_1608Metric_Pad1.08x0.95mm_HandSolder, symbol Device:C_Small
- added JP? (x4): SolderJumper_2_Open, symbol Jumper:SolderJumper_2_Open
- added R? (x2): 4.7k, Resistor_SMD:R_0603_1608Metric, symbol Device:R
- added R? (x4): 100k, Resistor_SMD:R_0603_1608Metric, symbol Device:R
- added R?: 200k, Resistor_SMD:R_0603_1608Metric, symbol Device:R
- added U14: CORE-V-MCU, Package_QFP:LQFP-80_12x12mm_P0.5mm, symbol OpenHW:CV32E40P
- added U? (x13): PI4ULS3V302XVEX, PSON40P160X120X55-8N, symbol PI4ULS3V302XVEX:PI4ULS3V302XVEX
- added U?: PI6ULS5V9306WEX, Package_SO:SOIC-8_3.9x4.9mm_P1.27mm, symbol PI6ULS5V9306:PI6ULS5V9306WEX
- gave numbers to parts that had none: 2
Connections:
- net camera/i2c_scl is gone; now on net +1V8: R15.2
- net camera/i2c_sda is gone; now on net +1V8: R16.2
- net +1V8: now also U14.12 (VDDIOC), U14.22 (AVDD2), U14.24 (AVDD), U14.32 (VDDIOC), U14.52 (VDDIOC), U14.72 (VDDIOC), U?.2 (VREF1)
- net +3V3: now also R?.2, R?.2, R?.2, U?.8 (VCCB), U?.8 (VCCB), U?.8 (VCCB), U?.8 (VCCB), U?.8 (VCCB), U?.8 (VCCB), U?.8 (VCCB); no longer R15.1, R16.1
- net 0.9V: now also R?.1, R?.1, R?.1, R?.1, U14.11 (VDDC), U14.13 (VDD_FPGA), U14.31 (VDDC), U14.33 (VDD_FPGA), U14.51 (VDDC), U14.53 (VDD_FPGA), U14.71 (VDDC), U14.73 (VDD_FPGA), U?.1 (VCCA), U?.1 (VCCA), U?.1 (VCCA), U?.1 (VCCA), U?.1 (VCCA), U?.1 (VCCA), U?.1 (VCCA), U?.1 (VCCA), U?.1 (VCCA), U?.1 (VCCA)
- net ExpressLink/EL_EVENT: now also U?.7 (B1)
- net ExpressLink/EL_WAKE: now also U?.6 (B2)
- net ExpressLink/~{EL_RESET}: now also U?.7 (B1)
- net GND: now also C?.2, JP?.1 (A), JP?.1 (A), JP?.1 (A), JP?.1 (A), U14.10 (VSSC), U14.23 (AVSS), U14.29 (VSSIOC), U14.30 (VSSC), U14.49 (VSSIOC), U14.50 (VSSC), U14.69 (VSSIOC), U14.70 (VSSC), U14.9 (VSSIOC), U?.1 (GND), U?.4 (GND), U?.4 (GND), U?.4 (GND), U?.4 (GND), U?.4 (GND), U?.4 (GND), U?.4 (GND)
- net mikrobus and sensors/click_cs: now also U?.6 (B2)
- net mikrobus and sensors/click_int: now also U?.7 (B1)
- net mikrobus and sensors/click_miso: now also U?.6 (B2)
- net mikrobus and sensors/click_mosi: now also U?.7 (B1)
- net mikrobus and sensors/click_pwm: now also U?.6 (B2)
- net mikrobus and sensors/click_rst: now also U?.6 (B2)
- net mikrobus and sensors/click_sck: now also U?.7 (B1)
- net mikrobus and sensors/temperature_alert: now also U?.7 (B1)
- net PGM_FLASH_CS: now reaches U13.1 (~{CS})
- net PGM_FLASH_DATA1: now reaches U13.2 (DO(IO1))
- net PGM_FLASH_DATA2: now reaches U13.3 (IO2)
- net PGM_FLASH_DATA0: now reaches U13.5 (DI(IO0))
- net PGM_FLASH_CLK: now reaches U13.6 (CLK)
- net PGM_FLASH_DATA3: now reaches U13.7 (IO3)
- net at X1.3 (OUT): now also U?.7 (B1)
- new net: JP?.2 (B), R?.2, U?.5 (EN) (x4)
- new net: C?.1, R?.1, U?.7 (VREF2), U?.8 (EN)
- new net 10MHZ_CLOCK_SOC: U14.48 (IO5)
- new net CLICK_RX: U?.7 (B1)
- new net CLICK_TX: U?.6 (B2)
- new net CLOCK_SOC: U?.2 (A1)
- new net CONSOLE_RX: U?.7 (B1)
- new net CONSOLE_TX: U?.6 (B2)
- new net CS0: U?.3 (A2)
- new net EL_RX: U?.7 (B1)
- new net EL_TX: U?.6 (B2)
- new net IO5_SOC: U?.3 (A2)
- new net MOSI0: U?.2 (A1), U?.3 (A2)
- new net PGM_FLASH_CLK_SOC: U14.7 (IO16)
- new net PGM_FLASH_CS_SOC: U14.4 (IO13)
- new net PGM_FLASH_DATA0_SOC: U14.5 (IO14)
- new net PGM_FLASH_DATA1_SOC: U14.6 (IO15)
- new net PGM_FLASH_DATA2_SOC: U14.15 (IO19)
- new net PGM_FLASH_DATA3_SOC: U14.16 (IO20)
- new net RX0_SOC: U?.3 (A2)
- new net RX1_MUX0_SOC: U14.59 (IO10), U?.3 (A2)
- new net RX1_MUX1_SOC: U?.3 (A2)
- new net SCL: R?.1, U?.6 (SCL2)
- new net SCL0_SOC: R15.1, U14.19 (IO23), U?.3 (SCL1)
- new net SCLK0: U?.2 (A1)
- new net SDA: R?.1, U?.5 (SDA2)
- new net SDA0_SOC: R16.1, U14.20 (IO24), U?.4 (SDA1)
- new net TCK: U?.6 (B2)
- new net TCK_SOC: U?.3 (A2)
- new net TDI: U?.6 (B2)
- new net TDI_SOC: U?.3 (A2)
- new net TDO: U?.7 (B1)
- new net TDO_SOC: U?.2 (A1)
- new net TMS: U?.7 (B1)
- new net TMS_SOC: U?.2 (A1)
- new net TX0_SOC: U?.2 (A1)
- new net TX1_MUX0_SOC: U14.58 (IO9), U?.2 (A1)
- new net TX1_MUX1_SOC: U?.2 (A1)
- new net USER_BUTTON_SOC: U?.3 (A2)
- new net USER_LED_SOC: U?.2 (A1)
- new net el_event: U?.2 (A1)
- new net el_reset: U?.2 (A1)
- new net el_wake: U?.3 (A2)
- new net irq: U?.2 (A1)
- new net nRESET_SOC: U14.55 (IO6)
- new net pwm: U?.3 (A2)
- new net reset: U?.3 (A2)
- new net temp_alert: U?.2 (A1)
- no-connect marks 0 -> 1
Other:
- sheet jtag and uart ports: added nRESET; removed none
- note added: "10MHz clock for the SOC PLL"
- note added: "Clock from the Camera"
- note added: "Clock to the Camera"
- note added: "NOTE: RX/TX are swapped in the shifters"
- note added: "Questions: 1) POWER_DETECT 2) VPW_P, VNW_N, NB, PB voltages 3) U_RDOUT, U_RDIN"
- note added: "SOC Reset Input"
- note added: "TODO MODIFY JTAG for 1.8v I/O Find 10MHz 1.8v oscillator Find 1.8v QSPI Flash memory Fix Camera voltages Get SOC voltages sorted out"
- note removed: "NOTE: This symbol is representative of the final device and does not currently match the device in development."
- moved on the sheet: H1, H2, H3, H4, R15, R16, U13, X1

Commit message: Power and Level Shifter updates
Parts:
- removed JP? (x4): SolderJumper_2_Open, symbol Jumper:SolderJumper_2_Open
- removed R? (x4): 100k, Resistor_SMD:R_0603_1608Metric, symbol Device:R
- removed U13: W25Q128JVS, Package_SO:SOIC-8_5.23x5.23mm_P1.27mm, symbol Memory_Flash:W25Q128JVS
- removed U? (x4): PI4ULS3V302XVEX, PSON40P160X120X55-8N, symbol PI4ULS3V302XVEX:PI4ULS3V302XVEX
- removed X1: SG-8002LB, Oscillator:Oscillator_SMD_SeikoEpson_SG8002LB-4Pin_5.0x3.2mm, symbol Oscillator:SG-8002LB
- added C? (x37): 100nF, Capacitor_SMD:C_0603_1608Metric_Pad1.08x0.95mm_HandSolder, symbol Device:C_Small
- added D? (x4): LED, symbol Device:LED
- added Q? (x4): MMBT3904, Package_TO_SOT_SMD:SOT-23, symbol Transistor_BJT:MMBT3904
- added R? (x4): 220, Resistor_SMD:R_0603_1608Metric, symbol Device:R
- added R? (x4): 1k, Resistor_SMD:R_0603_1608Metric, symbol Device:R
- added R?: 4.7k, Resistor_SMD:R_0603_1608Metric, symbol Device:R
- added R?: 100, Resistor_SMD:R_0603_1608Metric, symbol Device:R
- added SW? (x2): SW_Push, symbol Switch:SW_Push
- added U? (x2): PI4ULS3V302XVEX, PSON40P160X120X55-8N, symbol PI4ULS3V302XVEX:PI4ULS3V302XVEX
- added U?: W25Q32JWZP, Package_SON:WSON-8-1EP_6x5mm_P1.27mm_EP3.4x4.3mm, symbol Memory_Flash:W25Q32JVZP
- added U?: MAX6842DUKD0+T, 21-0057_U5-1_MXM, symbol MAX6842:MAX6842DUKD0+T
- added X?: ECS-2520MVLC-100-CN, Oscillator:Oscillator_SMD_ECS_2520MV-xxx-xx-4Pin_2.5x2.0mm, symbol Oscillator:ECS-2520MV-xxx-xx
Connections:
- net PGM_FLASH_CLK_SOC is gone; now on net PGM_FLASH_CLK: U14.7 (IO16)
- net PGM_FLASH_CS_SOC is gone; now on net PGM_FLASH_CS: U14.4 (IO13)
- net PGM_FLASH_DATA0_SOC is gone; now on net PGM_FLASH_DATA0: U14.5 (IO14)
- net PGM_FLASH_DATA1_SOC is gone; now on net PGM_FLASH_DATA1: U14.6 (IO15)
- net +1V8: now also U?.1 (VCCA), U?.1 (VCCA), U?.1 (VCCA), U?.1 (VCCA), U?.1 (VCCA), U?.1 (VCCA), U?.1 (VCCA), U?.1 (VCCA), U?.1 (VCCA), U?.5 (EN), U?.5 (EN), U?.5 (EN), U?.5 (EN), U?.5 (EN), U?.5 (EN), U?.5 (EN), U?.5 (EN), U?.5 (EN), C?.1, C?.1, C?.1, C?.1, C?.1, C?.1, C?.1, C?.1, C?.1, C?.1, C?.1, C?.1, C?.1, C?.1, C?.1, C?.1, C?.1, C?.1, R?.2, U?.1 (VCCA), U?.1 (VCCA), U?.5 (EN), U?.5 (VCC), U?.8 (VCC), X?.1 (Tri-State), X?.4 (VDD)
- net +3V3: now also U?.8 (VCCB), U?.8 (VCCB), C?.1, C?.1, C?.1, C?.1, C?.1, C?.1, C?.1, C?.1, C?.1, C?.1, C?.1, C?.1, C?.1, C?.1, C?.1, C?.1, C?.1, C?.1, D?.2 (A), D?.2 (A), D?.2 (A), D?.2 (A), U?.8 (VCCB), U?.8 (VCCB)
- net 10MHZ_CLOCK_SOC: now also X?.3 (OUT)
- net CLICK_IRQ_SOC: now also U14.64 (IO28)
- net CLICK_PWM_SOC: now also U14.34 (IO43)
- net CLICK_RESET_SOC: now also U14.14 (IO18)
- net CLICK_RX: now also U?.7 (B1)
- net CLICK_TX: now also U?.6 (B2)
- net CS0_SOC: now also U14.79 (IO38)
- net EL_EVENT_SOC: now also U14.63 (IO27)
- net EL_RESET_SOC: now also U14.35 (IO44)
- net EL_RX: now also U?.7 (B1)
- net EL_TX: now also U?.6 (B2)
- net EL_WAKE_SOC: now also U14.78 (IO37)
- net FPGA_LED0: now also U14.28 (IO42), R?.2
- net FPGA_LED1: now also U14.37 (IO46), R?.2
- net FPGA_LED2: now also U14.38 (IO47), R?.2
- net GND: now also U?.4 (GND), U?.4 (GND), U?.4 (GND), C?.2, C?.2, C?.2, C?.2, C?.2, C?.2, C?.2, C?.2, C?.2, C?.2, C?.2, C?.2, C?.2, C?.2, C?.2, C?.2, C?.2, C?.2, C?.2, C?.2, C?.2, C?.2, C?.2, C?.2, C?.2, C?.2, C?.2, C?.2, C?.2, C?.2, C?.2, C?.2, C?.2, C?.2, C?.2, C?.2, C?.2, Q?.2 (E), Q?.2 (E), Q?.2 (E), Q?.2 (E), SW?.1, SW?.1, U?.2 (GND), U?.4 (GND), U?.4 (GND), U?.4 (GND), X?.2 (GND)
- net MISO0_SOC: now also U14.27 (IO41)
- net MOSI0_SOC: now also U14.80 (IO39)
- net PGM_FLASH_CLK: now also U?.6 (CLK)
- net PGM_FLASH_CS: now also U?.1 (~{CS})
- net PGM_FLASH_DATA0: now also U?.5 (DI(IO0))
- net PGM_FLASH_DATA1: now also U?.2 (DO(IO1))
- net PGM_FLASH_DATA2: now also U?.3 (IO2)
- net PGM_FLASH_DATA3: now also U?.7 (IO3)
- net RX0_SOC: now also U14.56 (IO7)
- net RX1_MUX0_SOC: now also U?.3 (A2)
- net RX1_MUX1_SOC: now also U14.3 (IO12), U?.3 (A2)
- net SCLK0_SOC: now also U14.26 (IO40)
- net TCK: now also U14.43 (IO0)
- net TDI: now also U14.44 (IO1)
- net TDO: now also U14.45 (IO2)
- net TMS: now also U14.46 (IO3)
- net TRST: now also U14.47 (IO4)
- net TX0_SOC: now also U14.57 (IO8)
- net TX1_MUX0_SOC: now also U?.2 (A1)
- net TX1_MUX1_SOC: now also U14.60 (IO11), U?.2 (A1)
- net USER_LED_SOC: now also U14.36 (IO45), R?.2
- net nRESET_SOC: now also U?.1 (*RESET)
- net CAMERA_VSYNC: now reaches U14.17 (IO21)
- net CAMERA_HSYNC: now reaches U14.18 (IO22)
- net CAMERA_PCLK: now reaches U14.61 (IO25)
- net CAMERA_MCLK: now reaches U14.62 (IO26)
- net CAMERA_D0: now reaches U14.65 (IO29)
- net CAMERA_D1: now reaches U14.66 (IO30)
- net CAMERA_D2: now reaches U14.67 (IO31)
- net CAMERA_D3: now reaches U14.68 (IO32)
- net CAMERA_D4: now reaches U14.74 (IO33)
- net CAMERA_D5: now reaches U14.75 (IO34)
- net CAMERA_D6: now reaches U14.76 (IO35)
- net CAMERA_D7: now reaches U14.77 (IO36)
- net USER_BUTTON: now reaches U14.8 (IO17)
- net USER_BUTTON: now also R?.2
- net 0.9V renamed 0.8V
- net 0.8V: no longer U?.1 (VCCA), U?.1 (VCCA), U?.1 (VCCA), U?.1 (VCCA), U?.1 (VCCA), U?.1 (VCCA), U?.1 (VCCA), U?.1 (VCCA)
- net el_event renamed EL_EVENT
- net el_reset renamed EL_RESET
- net el_wake renamed EL_WAKE
- net irq renamed CLICK_IRQ
- net pwm renamed CLICK_PWM
- net reset renamed CLICK_RESET
- net temp_alert renamed TEMP_ALERT
- new net: D?.1 (K), R?.2 (x4)
- new net: Q?.3 (C), R?.1 (x4)
- new net: Q?.1 (B), R?.1 (x4)
- new net: C?.1, R?.1, R?.1, SW?.2
- new net: SW?.2, U?.4 (*MR)
Other:
- note added: "TODO Fix Camera voltages Get SOC voltages sorted out"
- note added: "UART1 Connected to ExpressLink"
- note added: "UART1 Connected to Mikrobus"
- note removed: "TODO MODIFY JTAG for 1.8v I/O Find 10MHz 1.8v oscillator Find 1.8v QSPI Flash memory Fix Camera voltages Get SOC voltages sorted out"
- moved on the sheet: C?, R15, R16, R?, U?

Commit message: updates to the footprints
Parts:
- C26, C27, C28, C29, C30, C31, C38, C39, C40, C41, C42, C43, C44, C45, C46, C47, C48, C49, C50, C51, C52, C53, C54, C55, C56, C57, C58, C59, C6, C60, C61, C62, C63, C64, C65, C66, C67, C9: renamed from C?; footprint Capacitor_SMD:C_0603_1608Metric_Pad1.08x0.95mm_HandSolder -> Capacitor_SMD:C_0603_1608Metric
- D10, D11, D8, D9: renamed from D?; footprint (none) -> LED_SMD:LED_0603_1608Metric
- SW1, SW2: renamed from SW?; footprint (none) -> Button_Switch_SMD:SW_Push_1P1T-SH_NO_CK_KMR2xxG
- U10, U13, U15, U16, U17, U18, U19, U6, U7, U8, U9: renamed from U?; footprint PSON40P160X120X55-8N -> pi4uls3v302:PSON40P160X120X55-8N
- U5: renamed from U?; footprint 21-0057_U5-1_MXM -> MAX6842:MAX6842DUKD0&plus_T
- gave numbers to parts that had none: 20

Commit message: pcb updates including level shifter adjustments
Connections:
- net CS0 is gone; now on net EL_WAKE_SOC: U9.3 (A2)
- net PGM_FLASH_DATA2_SOC is gone; now on net PGM_FLASH_DATA2: U14.15 (IO19)
- net PGM_FLASH_DATA3_SOC is gone; now on net PGM_FLASH_DATA3: U14.16 (IO20)
- net SCLK0 is gone; now on net CLICK_IRQ_SOC: U10.2 (A1)
- net TEMP_ALERT is gone; now on net CS0_SOC: U9.2 (A1)
- net mikrobus and sensors/click_cs is gone; now on net EL_WAKE: U9.6 (B2)
- net mikrobus and sensors/click_miso is gone; now on net EL_EVENT: U10.6 (B2)
- net mikrobus and sensors/click_sck is gone; now on net CLICK_PWM: U10.7 (B1)
- net +3V3: now also U6.8 (VCCB)
- net CLICK_PWM: no longer U13.3 (A2)
- net CLICK_RX: no longer U16.7 (B1), U8.7 (B1)
- net CLICK_TX: now also U8.7 (B1); no longer U16.6 (B2), U8.6 (B2)
- net EL_EVENT: no longer U18.2 (A1)
- net EL_EVENT_SOC: now also U10.3 (A2)
- net EL_RX: now also U7.6 (B2); no longer U17.7 (B1), U7.7 (B1)
- net EL_TX: now also U7.7 (B1); no longer U17.6 (B2), U7.6 (B2)
- net EL_WAKE: no longer U18.3 (A2)
- net MOSI0_SOC: now also U8.3 (A2)
- net RX1_MUX0_SOC: now also U7.2 (A1); no longer U17.3 (A2), U7.3 (A2)
- net RX1_MUX1_SOC: now also U8.2 (A1); no longer U16.3 (A2), U8.3 (A2)
- net TX1_MUX0_SOC: now also U7.3 (A2); no longer U17.2 (A1), U7.2 (A1)
- net TX1_MUX1_SOC: no longer U16.2 (A1), U8.2 (A1)
- net mikrobus and sensors/temperature_alert: no longer U9.7 (B1)
- net 0.8V renamed +0V8
- net CLICK_IRQ: no longer names the net of U15.2 (A1)
- net CLICK_RESET: no longer names the net of U15.3 (A2)
- net EL_RESET: no longer names the net of U19.2 (A1)
- net EL_RESET_SOC renamed ~{EL_RESET_SOC}
- net ExpressLink/EL_EVENT: no longer names the net of U18.7 (B1)
- net ExpressLink/EL_WAKE: no longer names the net of U18.6 (B2)
- net ExpressLink/~{EL_RESET}: no longer names the net of U19.7 (B1)
- net MOSI0: no longer names the net of U13.2 (A1)
- net MOSI0: no longer U10.3 (A2)
- net mikrobus and sensors/click_int: no longer names the net of U15.7 (B1)
- net mikrobus and sensors/click_mosi: no longer names the net of U13.7 (B1)
- net mikrobus and sensors/click_pwm: no longer names the net of U13.6 (B2)
- net mikrobus and sensors/click_rst: no longer names the net of U15.6 (B2)
- net nRESET_SOC renamed ~{RESET_SOC}
- new net CLICK_CS: U9.7 (B1)
- new net CLICK_MOSI: U8.6 (B2)
- no-connect marks 1 -> 2
Other:
- moved on the sheet: C26, C27, C28, C29, C30, C31, C38, C39, C40, C41, C42, C43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
