File: OpenHW DevKit.kicad_sch (KiCad schematic)
At the start: 66 parts, among them J10 Conn_01x20, J4 Conn_01x02_Male, J7 Conn_01x20, J8 Conn_01x20, J9 Conn_01x20, Q1 MMBT3904, Q2 MMBT3904, SW1 SW_Push, SW2 SW_Push, U14 CORE-V-MCU, U3 W25Q32JWZP, U4 FXMA2102UMX, U6 NTB0104BQ,115, U7 NTB0104BQ,115, U8 NTB0104BQ,115, U9 NTB0104BQ,115, X1 ECS-2520MVLC-100-CN

Commit message: updated the QR code and added shield coupling to the usb connector
Changed lines of the file:
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@@
     )
   )
-  (symbol (lib_id "OpenHW:Devkit_QR") (at 408.94 231.14 0) (unit 1)
-    (in_bom yes) (on_board yes) (dnp no) (fields_autoplaced)
-    (property "Reference" "SYM*1" (at 410.9467 231.4568 0)
+  (symbol (lib_id "OpenHW:Devkit_QR") (at 43.18 233.68 0) (unit 1)
+    (in_bom yes) (on_board yes) (dnp no)
+    (property "Reference" "SYM*1" (at 45.72 233.68 0)
       (effects (font (size 1.27 1.27)) (justify left))
     )
-    (property "Value" "~" (at 408.94 231.14 0)
+    (property "Value" "~" (at 43.18 233.68 0)
       (effects (font (size 1.27 1.27)))
     )
-    (property "Footprint" "logos:devkits_qr" (at 408.94 233.68 0)
+    (property "Footprint" "logos:devkits_qr" (at 43.18 236.22 0)
       (effects (font (size 1.27 1.27)) hide)
     )
-    (property "Datasheet" "" (at 408.94 231.14 0)
+    (property "Datasheet" "" (at 43.18 233.68 0)
       (effects (font (size 1.27 1.27)) hide)
     )
