File: OpenHW DevKit.kicad_sch (KiCad schematic)
At the start: 66 parts, among them J10 Conn_01x20, J4 Conn_01x02_Male, J7 Conn_01x20, J8 Conn_01x20, J9 Conn_01x20, Q1 MMBT3904, Q2 MMBT3904, SW1 SW_Push, SW2 SW_Push, U14 CORE-V-MCU, U3 W25Q32JWZP, U4 FXMA2102UMX, U6 NTB0104BQ,115, U7 NTB0104BQ,115, U8 NTB0104BQ,115, U9 NTB0104BQ,115, X1 ECS-2520MVLC-100-CN

Commit message: pullup resistors on JTAG signals
Parts:
- added R43, R44, R45: 10k, Resistor_SMD:R_0603_1608Metric, symbol Device:R
Connections:
- net +1V8: now also R43.2, R44.2, R45.2
- net TDI: now also R45.1
- net TMS: now also R44.1
- net TRST: now also R43.1
Other:
- sheet jtag and uart ports: added nTRST; removed none

Commit message: swapped bootsel & test_mode pins
Connections:
- net BOOTSEL: now also J8.17 (Pin_17), U14.37 (IO44); no longer J8.19 (Pin_19), U14.39 (IO45)
- net TEST_MODE: now also J8.19 (Pin_19), U14.39 (IO45); no longer J8.17 (Pin_17), U14.37 (IO44)

Commit message: updated footprints, added the barrel power connector and test points
Parts:
- added TP10, TP11, TP12, TP13, TP14, TP15, TP16, TP17, TP18, TP19, TP25, TP27, TP28, TP29, TP30, TP31, TP32, TP33, TP34, TP35, TP36, TP37, TP38, TP39, TP40, TP41, TP42, TP43, TP44, TP45, TP46, TP47, TP48, TP49, TP50, TP51, TP52, TP53, TP54, TP55, TP56, TP57, TP58, TP59, TP60, TP61, TP62, TP63, TP64, TP65, TP66, TP67, TP68, TP69, TP7, TP70, TP71, TP72, TP73, TP74, TP75, TP8, TP9: TestPoint_Small, TestPoint:TestPoint_Pad_D1.0mm, symbol Connector:TestPoint_Small
Connections:
- net 10MHZ_CLOCK_SOC: now also TP25.1
- net CAMERA_D0: now also TP42.1
- net CAMERA_D1: now also TP48.1
- net CAMERA_D2: now also TP45.1
- net CAMERA_D3: now also TP47.1
- net CAMERA_D4: now also TP44.1
- net CAMERA_D5: now also TP39.1
- net CAMERA_D6: now also TP40.1
- net CAMERA_D7: now also TP43.1
- net CAMERA_HSYNC: now also TP31.1
- net CAMERA_MCLK: now also TP46.1
- net CAMERA_PCLK: now also TP41.1
- net CAMERA_VSYNC: now also TP32.1
- net CLICK_CS: now also TP64.1
- net CLICK_INT: now also TP62.1
- net CLICK_MISO: now also TP66.1
- net CLICK_MOSI: now also TP67.1
- net CLICK_PWM: now also TP63.1
- net CLICK_RESET_SOC: now also TP9.1
- net CLICK_RST: now also TP56.1
- net CLICK_RX: now also TP61.1
- net CLICK_SCK: now also TP65.1
- net CLICK_TX: now also TP60.1
- net CONSOLE_RX: now also TP52.1
- net CONSOLE_TX: now also TP53.1
- net CS0_SOC: now also TP51.1
- net EL_EVENT: now also TP59.1
- net EL_EVENT_SOC: now also TP30.1
- net EL_RXD: now also TP57.1
- net EL_TXD: now also TP58.1
- net EL_WAKE: now also TP54.1
- net EL_WAKE_SOC: now also TP29.1
- net FPGA_LED0: now also TP49.1
- net MISO0_SOC: now also TP34.1
- net MOSI0_SOC: now also TP35.1
- net PGM_FLASH_CLK: now also TP14.1
- net PGM_FLASH_CS: now also TP12.1
- net PGM_FLASH_DATA0: now also TP15.1
- net PGM_FLASH_DATA1: now also TP11.1
- net PGM_FLASH_DATA2: now also TP10.1
- net PGM_FLASH_DATA3: now also TP13.1
- net RX1_MUX0_SOC: now also TP8.1
- net RX1_MUX1_SOC: now also TP19.1
- net SCL: now also TP69.1
- net SCL0_SOC: now also TP37.1
- net SCLK0_SOC: now also TP33.1
- net SDA: now also TP68.1
- net SDA0_SOC: now also TP38.1
- net TCK: now also TP75.1
- net TDI: now also TP73.1
- net TDO: now also TP72.1
- net TMS: now also TP74.1
- net TRST: now also TP71.1
- net TX0_RXD: now also TP16.1
- net TX0_TXD: now also TP17.1
- net TX1_MUX0_SOC: now also TP7.1
- net TX1_MUX1_SOC: now also TP18.1
- net USER_BUTTON: now also TP28.1
- net USER_LED_SOC: now also TP36.1
- net ~{EL_RESET_SOC}: now also TP50.1
- net ~{EL_RESET}: now also TP55.1
- net ~{RESET_SOC}: now also TP27.1, TP70.1
Other:
- moved on the sheet: J10, J7, J8, J9

Commit message: Converted from QFP to BGA
Parts:
- U14: footprint Package_QFP:LQFP-80_12x12mm_P0.5mm -> core-v:BGA-80-22x22
Connections:
- net +0V8: now also U14.A9 (VDD_FPGA), U14.B8 (VDDC), U14.F2 (VDD_FPGA), U14.G12 (VDDC), U14.G2 (VDDC), U14.H12 (VDD_FPGA), U14.M6 (VDD_FPGA), U14.M7 (VDDC); no longer U14.11 (VDDC), U14.13 (VDD_FPGA), U14.33 (VDDC), U14.35 (VDD_FPGA), U14.51 (VDDC), U14.53 (VDD_FPGA), U14.71 (VDDC), U14.73 (VDD_FPGA)
- net +1V8: now also U14.B4 (AVDD2), U14.B5 (AVDD), U14.C8 (VDDIOC), U14.F1 (VDDIOC), U14.H13 (VDDIOC), U14.N6 (VDDIOC); no longer U14.12 (VDDIOC), U14.23 (AVDD2), U14.25 (AVDD), U14.34 (VDDIOC), U14.52 (VDDIOC), U14.72 (VDDIOC)
- net 10MHZ_CLOCK_SOC: now also U14.F12 (IO5); no longer U14.48 (IO5)
- net BOOTSEL: now also U14.C9 (IO44); no longer U14.37 (IO44)
- net CAMERA_D0: now also U14.L9 (IO29); no longer U14.66 (IO29)
- net CAMERA_D1: now also U14.L5 (IO30); no longer U14.77 (IO30)
- net CAMERA_D2: now also U14.L6 (IO31); no longer U14.74 (IO31)
- net CAMERA_D3: now also U14.M5 (IO32); no longer U14.76 (IO32)
- net CAMERA_D4: now also U14.M8 (IO33); no longer U14.68 (IO33)
- net CAMERA_D5: now also U14.M10 (IO34); no longer U14.63 (IO34)
- net CAMERA_D6: now also U14.N9 (IO35); no longer U14.64 (IO35)
- net CAMERA_D7: now also U14.N8 (IO36); no longer U14.67 (IO36)
- net CAMERA_HSYNC: now also U14.K12 (IO22); no longer U14.59 (IO22)
- net CAMERA_MCLK: now also U14.N5 (IO26); no longer U14.75 (IO26)
- net CAMERA_PCLK: now also U14.M9 (IO25); no longer U14.65 (IO25)
- net CAMERA_VSYNC: now also U14.L13 (IO21); no longer U14.60 (IO21)
- net CLICK_IRQ_SOC: now also U14.A10 (IO37); no longer U14.38 (IO37)
- net CLICK_PWM_SOC: now also U14.A11 (IO42); no longer U14.40 (IO42)
- net CLICK_RESET_SOC: now also U14.J2 (IO18); no longer U14.5 (IO18)
- net CS0_SOC: now also U14.N3 (IO38); no longer U14.80 (IO38)
- net EL_EVENT_SOC: now also U14.K13 (IO24); no longer U14.58 (IO24)
- net EL_WAKE_SOC: now also U14.J11 (IO23); no longer U14.57 (IO23)
- net FPGA_LED0: now also U14.N4 (IO28); no longer U14.78 (IO28)
- net GND: now also U14.A5 (AVSS), U14.A8 (VSSC), U14.B7 (VSSIOC), U14.F11 (VSSIOC), U14.G1 (VSSC), U14.G13 (VSSC), U14.H3 (VSSIOC), U14.L8 (VSSIOC), U14.N7 (VSSC); no longer U14.10 (VSSC), U14.24 (AVSS), U14.31 (VSSIOC), U14.32 (VSSC), U14.49 (VSSIOC), U14.50 (VSSC), U14.69 (VSSIOC), U14.70 (VSSC), U14.9 (VSSIOC)
- net MISO0_SOC: now also U14.C6 (IO41); no longer U14.29 (IO41)
- net MOSI0_SOC: now also U14.A7 (IO39); no longer U14.30 (IO39)
- net NB: now also U14.C13 (NB); no longer U14.41 (NB)
- net PB: now also U14.D13 (PB); no longer U14.42 (PB)
- net PGM_FLASH_CLK: now also U14.E1 (IO16); no longer U14.15 (IO16)
- net PGM_FLASH_CS: now also U14.H2 (IO13); no longer U14.8 (IO13)
- net PGM_FLASH_DATA0: now also U14.E2 (IO14); no longer U14.16 (IO14)
- net PGM_FLASH_DATA1: now also U14.H1 (IO15); no longer U14.7 (IO15)
- net PGM_FLASH_DATA2: now also U14.J3 (IO19); no longer U14.6 (IO19)
- net PGM_FLASH_DATA3: now also U14.F3 (IO20); no longer U14.14 (IO20)
- net POWER_DETECT: now also U14.H11 (POWER_DETECT); no longer U14.54 (POWER_DETECT)
- net RX1_MUX0_SOC: now also U14.J1 (IO12); no longer U14.4 (IO12)
- net RX1_MUX1_SOC: now also U14.C1 (IO10); no longer U14.20 (IO10)
- net SCL0_SOC: now also U14.N11 (IO46); no longer U14.61 (IO46)
- net SCLK0_SOC: now also U14.B6 (IO40); no longer U14.28 (IO40)
- net SDA0_SOC: now also U14.N10 (IO47); no longer U14.62 (IO47)
- net TCK: now also U14.E13 (IO0); no longer U14.44 (IO0)
- net TDI: now also U14.E11 (IO1); no longer U14.46 (IO1)
- net TDO: now also U14.E12 (IO2); no longer U14.45 (IO2)
- net TEST_MODE: now also U14.B10 (IO45); no longer U14.39 (IO45)
- net TMS: now also U14.D12 (IO3); no longer U14.43 (IO3)
- net TRST: now also U14.F13 (IO4); no longer U14.47 (IO4)
- net TX0_RXD: now also U14.E3 (IO7); no longer U14.17 (IO7)
- net TX0_TXD: now also U14.D1 (IO8); no longer U14.18 (IO8)
- net TX1_MUX0_SOC: now also U14.K2 (IO11); no longer U14.3 (IO11)
- net TX1_MUX1_SOC: now also U14.D2 (IO9); no longer U14.19 (IO9)
- net USER_BUTTON: now also U14.J12 (IO17); no longer U14.56 (IO17)
- net USER_LED_SOC: now also U14.B9 (IO27); no longer U14.36 (IO27)
- net VNW_N: now also U14.K1 (VNW_N); no longer U14.2 (VNW_N)
- net VPW_P: now also U14.L1 (VPW_P); no longer U14.1 (VPW_P)
- net ~{EL_RESET_SOC}: now also U14.M4 (IO43); no longer U14.79 (IO43)
- net ~{RESET_SOC}: now also U14.J13 (IO6); no longer U14.55 (IO6)
Changed lines of the file:
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@@
       (effects (font (size 1.27 1.27)))
     )
-    (property "Footprint" "Package_QFP:LQFP-80_12x12mm_P0.5mm" (at 129.54 74.93 0)
+    (property "Footprint" "core-v:BGA-80-22x22" (at 129.54 74.93 0)
       (effects (font (size 1.27 1.27)) hide)
     )
@@
       (effects (font (size 1.27 1.27)) hide)
     )
-    (pin "1")
-    (pin "10")
-    (pin "11")
-    (pin "12")
-    (pin "13")
-    (pin "14")
-    (pin "15")
-    (pin "16")
-    (pin "17")
-    (pin "18")
-    (pin "19")
-    (pin "2")
-    (pin "20")
-    (pin "23")
-    (pin "24")
-    (pin "25")
-    (pin "28")
-    (pin "29")
-    (pin "3")
-    (pin "30")
-    (pin "31")
-    (pin "32")
-    (pin "33")
-    (pin "34")
-    (pin "35")
-    (pin "36")
-    (pin "37")
-    (pin "38")
-    (pin "39")
-    (pin "4")
-    (pin "40")
-    (pin "41")
-    (pin "42")
-    (pin "43")
-    (pin "44")
-    (pin "45")
-    (pin "46")
-    (pin "47")
-    (pin "48")
-    (pin "49")
-    (pin "5")
-    (pin "50")
-    (pin "51")
-    (pin "52")
-    (pin "53")
-    (pin "54")
-    (pin "55")
-    (pin "56")
-    (pin "57")
-    (pin "58")
-    (pin "59")
-    (pin "6")
-    (pin "60")
-    (pin "61")
-    (pin "62")
-    (pin "63")
-    (pin "64")
-    (pin "65")
-    (pin "66")
-    (pin "67")
-    (pin "68")
-    (pin "69")
-    (pin "7")
-    (pin "70")
-    (pin "71")
-    (pin "72")
-    (pin "73")
-    (pin "74")
-    (pin "75")
-    (pin "76")
-    (pin "77")
-    (pin "78")
-    (pin "79")
-    (pin "8")
-    (pin "80")
-    (pin "9")
+    (pin "A10")
+    (pin "A11")
+    (pin "A5")
+    (pin "A7")
+    (pin "A8")
+    (pin "A9")
+    (pin "B10")
+    (pin "B4")
+    (pin "B5")
+    (pin "B6")
+    (pin "B7")
+    (pin "B8")
+    (pin "B9")
+    (pin "C1")
+    (pin "C13")
+    (pin "C6")
+    (pin "C8")
+    (pin "C9")
+    (pin "D1")
+    (pin "D12")
+    (pin "D13")
+    (pin "D2")
+    (pin "E1")
+    (pin "E11")
+    (pin "E12")
+    (pin "E13")
+    (pin "E2")
+    (pin "E3")
+    (pin "F1")
+    (pin "F11")
+    (pin "F12")
+    (pin "F13")
+    (pin "F2")
+    (pin "F3")
+    (pin "G1")
+    (pin "G12")
+    (pin "G13")
+    (pin "G2")
+    (pin "H1")
+    (pin "H11")
+    (pin "H12")
+    (pin "H13")
+    (pin "H2")
+    (pin "H3")
+    (pin "J1")
+    (pin "J11")
+    (pin "J12")
+    (pin "J13")
+    (pin "J2")
+    (pin "J3")
+    (pin "K1")
+    (pin "K12")
+    (pin "K13")
+    (pin "K2")
+    (pin "L1")
+    (pin "L13")
+    (pin "L5")
+    (pin "L6")
+    (pin "L8")
+    (pin "L9")
+    (pin "M10")
+    (pin "M4")
+    (pin "M5")
+    (pin "M6")
+    (pin "M7")
+    (pin "M8")
+    (pin "M9")
+    (pin "N10")
+    (pin "N11")
+    (pin "N3")
+    (pin "N4")
+    (pin "N5")
+    (pin "N6")
+    (pin "N7")
+    (pin "N8")
+    (pin "N9")
     (instances
       (project "OpenHW DevKit"

Commit message: Grounded the die paddle
Connections:
- net GND: now also U14.GND (VSSC)
Changed lines of the file:
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@@
   (junction (at 196.85 34.29) (diameter 0) (color 0 0 0 0)
   )
+  (junction (at 111.76 147.32) (diameter 0) (color 0 0 0 0)
+  )
   (junction (at 193.04 52.07) (diameter 0) (color 0 0 0 0)
   )
@@
     (stroke (width 0) (type default))
   )
-  (wire (pts (xy 106.68 147.32) (xy 116.84 147.32))
+  (wire (pts (xy 106.68 147.32) (xy 111.76 147.32))
     (stroke (width 0) (type default))
   )
@@
     (stroke (width 0) (type default))
   )
+  (wire (pts (xy 111.76 147.32) (xy 116.84 147.32))
+    (stroke (width 0) (type default))
+  )
   (wire (pts (xy 138.43 30.48) (xy 138.43 35.56))
     (stroke (width 0) (type default))
@@
     (stroke (width 0) (type default))
   )
+  (wire (pts (xy 111.76 149.86) (xy 116.84 149.86))
+    (stroke (width 0) (type default))
+  )
   (wire (pts (xy 370.84 90.17) (xy 393.7 90.17))
     (stroke (width 0) (type default))
@@
     (stroke (width 0) (type default))
   )
+  (wire (pts (xy 111.76 147.32) (xy 111.76 149.86))
+    (stroke (width 0) (type default))
+  )
   (wire (pts (xy 233.68 199.39) (xy 238.76 199.39))
     (stroke (width 0) (type default))
@@
     (pin "G13")
     (pin "G2")
+    (pin "GND")
     (pin "H1")
     (pin "H11")

Commit message: Added PDF and corrected AVDD net
Connections:
- net +0V8: now also J8.3 (Pin_3), J8.5 (Pin_5), U14.B4 (AVDD2), U14.B5 (AVDD)
- net +1V8: no longer J8.3 (Pin_3), J8.5 (Pin_5), U14.B4 (AVDD2), U14.B5 (AVDD)
Other:
- note removed: "Note: Verify these connections. Do we need bypass capacitors?"
Changed lines of the file:
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@@
   (junction (at 359.41 63.5) (diameter 0) (color 0 0 0 0)
   )
+  (junction (at 109.22 114.3) (diameter 0) (color 0 0 0 0)
+  )
   (junction (at 231.14 57.15) (diameter 0) (color 0 0 0 0)
   )
@@
   (junction (at 356.87 219.71) (diameter 0) (color 0 0 0 0)
   )
-  (junction (at 102.87 118.11) (diameter 0) (color 0 0 0 0)
-  )
   (junction (at 275.59 234.95) (diameter 0) (color 0 0 0 0)
   )
@@
   (junction (at 233.68 201.93) (diameter 0) (color 0 0 0 0)
   )
-  (junction (at 102.87 102.87) (diameter 0) (color 0 0 0 0)
-  )
   (junction (at 275.59 161.29) (diameter 0) (color 0 0 0 0)
   )
@@
   (junction (at 106.68 142.24) (diameter 0) (color 0 0 0 0)
   )
+  (junction (at 109.22 118.11) (diameter 0) (color 0 0 0 0)
+  )
   (junction (at 104.14 177.8) (diameter 0) (color 0 0 0 0)
   )
@@
   (no_connect (at 275.59 97.79))
   (no_connect (at 275.59 100.33))
-  (wire (pts (xy 275.59 102.87) (xy 279.4 102.87))
-    (stroke (width 0) (type default))
-  )
   (wire (pts (xy 233.68 130.81) (xy 238.76 130.81))
     (stroke (width 0) (type default))
@@
     (stroke (width 0) (type default))
   )
-  (wire (pts (xy 116.84 118.11) (xy 102.87 118.11))
+  (wire (pts (xy 116.84 118.11) (xy 109.22 118.11))
     (stroke (width 0) (type default))
   )
@@
     (stroke (width 0) (type default))
   )
+  (wire (pts (xy 275.59 102.87) (xy 279.4 102.87))
+    (stroke (width 0) (type default))
+  )
   (wire (pts (xy 92.71 156.21) (xy 92.71 163.83))
     (stroke (width 0) (type default))
@@
     (stroke (width 0) (type default))
   )
-  (wire (pts (xy 102.87 102.87) (xy 102.87 118.11))
-    (stroke (width 0) (type default))
-  )
   (wire (pts (xy 83.82 29.21) (xy 83.82 31.75))
     (stroke (width 0) (type default))
@@
     (stroke (width 0) (type default))
   )
-  (wire (pts (xy 275.59 107.95) (xy 279.4 107.95))
-    (stroke (width 0) (type default))
-  )
   (wire (pts (xy 109.22 91.44) (xy 116.84 91.44))
     (stroke (width 0) (type default))
@@
     (stroke (width 0) (type default))
   )
-  (wire (pts (xy 102.87 120.65) (xy 102.87 118.11))
+  (wire (pts (xy 109.22 120.65) (xy 109.22 118.11))
     (stroke (width 0) (type default))
   )
@@
     (stroke (width 0) (type default))
   )
+  (wire (pts (xy 109.22 114.3) (xy 109.22 118.11))
+    (stroke (width 0) (type default))
+  )
   (wire (pts (xy 105.41 251.46) (xy 105.41 254))
     (stroke (width 0) (type default))
@@
     (stroke (width 0) (type default))
   )
+  (wire (pts (xy 275.59 130.81) (xy 279.4 130.81))
+    (stroke (width 0) (type default))
+  )
   (wire (pts (xy 321.31 173.99) (xy 330.2 173.99))
     (stroke (width 0) (type default))
@@
     (stroke (width 0) (type default))
   )
-  (wire (pts (xy 275.59 130.81) (xy 279.4 130.81))
-    (stroke (width 0) (type default))
-  )
   (wire (pts (xy 46.99 44.45) (xy 50.8 44.45))
     (stroke (width 0) (type default))
@@
     (stroke (width 0) (type default))
   )
+  (wire (pts (xy 275.59 107.95) (xy 279.4 107.95))
+    (stroke (width 0) (type default))
+  )
   (wire (pts (xy 102.87 97.79) (xy 116.84 97.79))
     (stroke (width 0) (type default))
@@
     (stroke (width 0) (type default))
   )
-  (wire (pts (xy 116.84 120.65) (xy 102.87 120.65))
+  (wire (pts (xy 116.84 120.65) (xy 109.22 120.65))
     (stroke (width 0) (type default))
   )
@@
     (effects (font (size 1.27 1.27)) (justify left bottom))
   )
-  (text "Note: Verify these connections.\nDo we need bypass capacitors?"
-    (at 20.32 160.02 0)
-    (effects (font (size 2 2)) (justify left bottom))
-  )
   (text "Copyright and related rights are licensed under the Solderpad Hardware License, Version 2.1 (the \"License\");\nyou may not use this file except in compliance with the License.  You may obtain a copy of the License at\nhttp://solderpad.org/licenses/SHL-2.1. Unless required by applicable law or agreed to in writing, software,\nhardware and materials distributed under this License is distributed on an \"AS IS\" BASIS, WITHOUT WARRANTIES OR\nCONDITIONS OF ANY KIND, either express or implied. See the License for the specific language governing\npermissions and limitations under the License.\n"
     (at 314.96 247.65 0)
@@
     )
   )
-  (symbol (lib_id "power:+1V8") (at 279.4 107.95 270) (unit 1)
-    (in_bom yes) (on_board yes) (dnp no) (fields_autoplaced)
-    (property "Reference" "#PWR0117" (at 275.59 107.95 0)
-      (effects (font (size 1.27 1.27)) hide)
-    )
-    (property "Value" "+1V8" (at 282.575 108.2668 90)
-      (effects (font (size 1.27 1.27)) (justify left))
-    )
-    (property "Footprint" "" (at 279.4 107.95 0)
-      (effects (font (size 1.27 1.27)) hide)
-    )
-    (property "Datasheet" "" (at 279.4 107.95 0)
-      (effects (font (size 1.27 1.27)) hide)
-    )
-    (pin "1")
-    (instances
-      (project "OpenHW DevKit"
-        (path "/b0906e10-2fbc-4309-a8b4-6fc4cd1a5490"
-          (reference "#PWR0117") (unit 1)
-        )
-      )
-    )
-  )
   (symbol (lib_id "power:GND") (at 176.53 59.69 0) (mirror y) (unit 1)
     (in_bom yes) (on_board yes) (dnp no) (fields_autoplaced)
@@
     )
   )
+  (symbol (lib_id "power:+0V8") (at 279.4 107.95 270) (unit 1)
+    (in_bom yes) (on_board yes) (dnp no)
+    (property "Reference" "#PWR0115" (at 275.59 107.95 0)
+      (effects (font (size 1.27 1.27)) hide)
+    )
+    (property "Value" "+0V8" (at 282.575 108.2668 90)
+      (effects (font (size 1.27 1.27)) (justify left))
+    )
+    (property "Footprint" "" (at 279.4 107.95 0)
+      (effects (font (size 1.27 1.27)) hide)
+    )
+    (property "Datasheet" "" (at 279.4 107.95 0)
+      (effects (font (size 1.27 1.27)) hide)
+    )
+    (pin "1")
+    (instances
+      (project "OpenHW DevKit"
+        (path "/b0906e10-2fbc-4309-a8b4-6fc4cd1a5490"
+          (reference "#PWR0115") (unit 1)
+        )
+      )
+    )
+  )
   (symbol (lib_id "Connector:TestPoint_Small") (at 233.68 138.43 0) (unit 1)
     (in_bom yes) (on_board yes) (dnp no)
@@
     )
   )
+  (symbol (lib_id "power:+0V8") (at 279.4 102.87 270) (unit 1)
+    (in_bom yes) (on_board yes) (dnp no)
+    (property "Reference" "#PWR080" (at 275.59 102.87 0)
+      (effects (font (size 1.27 1.27)) hide)
+    )
+    (property "Value" "+0V8" (at 282.575 103.1868 90)
+      (effects (font (size 1.27 1.27)) (justify left))
+    )
+    (property "Footprint" "" (at 279.4 102.87 0)
+      (effects (font (size 1.27 1.27)) hide)
+    )
+    (property "Datasheet" "" (at 279.4 102.87 0)
+      (effects (font (size 1.27 1.27)) hide)
+    )
+    (pin "1")
+    (instances
+      (project "OpenHW DevKit"
+        (path "/b0906e10-2fbc-4309-a8b4-6fc4cd1a5490"
+          (reference "#PWR080") (unit 1)
+        )
+      )
+    )
+  )
   (symbol (lib_id "Connector:TestPoint_Small") (at 233.68 135.89 0) (unit 1)
     (in_bom yes) (on_board yes) (dnp no)
@@
     )
   )
+  (symbol (lib_id "power:+1V8") (at 279.4 130.81 270) (unit 1)
+    (in_bom yes) (on_board yes) (dnp no) (fields_autoplaced)
+    (property "Reference" "#PWR015" (at 275.59 130.81 0)
+      (effects (font (size 1.27 1.27)) hide)
+    )
+    (property "Value" "+1V8" (at 282.575 131.1268 90)
+      (effects (font (size 1.27 1.27)) (justify left))
+    )
+    (property "Footprint" "" (at 279.4 130.81 0)
+      (effects (font (size 1.27 1.27)) hide)
+    )
+    (property "Datasheet" "" (at 279.4 130.81 0)
+      (effects (font (size 1.27 1.27)) hide)
+    )
+    (pin "1")
+    (instances
+      (project "OpenHW DevKit"
+        (path "/b0906e10-2fbc-4309-a8b4-6fc4cd1a5490"
+          (reference "#PWR015") (unit 1)
+        )
+      )
+    )
+  )
   (symbol (lib_id "power:GND") (at 279.4 176.53 90) (unit 1)
     (in_bom yes) (on_board yes) (dnp no) (fields_autoplaced)
@@
     )
   )
-  (symbol (lib_id "power:+1V8") (at 279.4 130.81 270) (unit 1)
-    (in_bom yes) (on_board yes) (dnp no) (fields_autoplaced)
-    (property "Reference" "#PWR0121" (at 275.59 130.81 0)
-      (effects (font (size 1.27 1.27)) hide)
-    )
-    (property "Value" "+1V8" (at 282.575 131.1268 90)
-      (effects (font (size 1.27 1.27)) (justify left))
-    )
-    (property "Footprint" "" (at 279.4 130.81 0)
-      (effects (font (size 1.27 1.27)) hide)
-    )
-    (property "Datasheet" "" (at 279.4 130.81 0)
-      (effects (font (size 1.27 1.27)) hide)
-    )
-    (pin "1")
-    (instances
-      (project "OpenHW DevKit"
-        (path "/b0906e10-2fbc-4309-a8b4-6fc4cd1a5490"
-          (reference "#PWR0121") (unit 1)
-        )
-      )
-    )
-  )
   (symbol (lib_id "Connector:TestPoint_Small") (at 233.68 113.03 0) (unit 1)
     (in_bom yes) (on_board yes) (dnp no)
@@
         )
       )
-    )
-  )
-  (symbol (lib_id "power:+1V8") (at 279.4 102.87 270) (unit 1)
-    (in_bom yes) (on_board yes) (dnp no) (fields_autoplaced)
-    (property "Reference" "#PWR0115" (at 275.59 102.87 0)
-      (effects (font (size 1.27 1.27)) hide)
-    )
-    (property "Value" "+1V8" (at 282.575 103.1868 90)
-      (effects (font (size 1.27 1.27)) (justify left))
-    )
-    (property "Footprint" "" (at 279.4 102.87 0)
-      (effects (font (size 1.27 1.27)) hide)
-    )
-    (property "Datasheet" "" (at 279.4 102.87 0)
-      (effects (font (size 1.27 1.27)) hide)
-    )
-    (pin "1")
-    (instances
-      (project "OpenHW DevKit"
-        (path "/b0906e10-2fbc-4309-a8b4-6fc4cd1a5490"
-          (reference "#PWR0115") (unit 1)
-        )
-      )

Commit message: updated the graphics and moved files around for neatness
Parts:
- renumbered SYM*1 to QR-Code
Changed lines of the file:
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@@
   (symbol (lib_id "OpenHW:Devkit_QR") (at 43.18 233.68 0) (unit 1)
     (in_bom yes) (on_board yes) (dnp no)
-    (property "Reference" "SYM*1" (at 45.72 233.68 0)
+    (property "Reference" "QR-Code" (at 45.72 233.68 0)
       (effects (font (size 1.27 1.27)) (justify left))
     )
     (property "Value" "~" (at 43.18 233.68 0)
-      (effects (font (size 1.27 1.27)))
+      (effects (font (size 1.27 1.27)) hide)
     )
     (property "Footprint" "logos:devkits_qr" (at 43.18 236.22 0)
@@
       (project "OpenHW DevKit"
         (path "/b0906e10-2fbc-4309-a8b4-6fc4cd1a5490"
-          (reference "SYM*1") (unit 1)
+          (reference "QR-Code") (unit 1)
         )
       )

Commit message: minor save
Parts:
- renumbered QR-Code to QR-Code1
Changed lines of the file:
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@@
   (symbol (lib_id "OpenHW:Devkit_QR") (at 43.18 233.68 0) (unit 1)
     (in_bom yes) (on_board yes) (dnp no)
-    (property "Reference" "QR-Code" (at 45.72 233.68 0)
+    (property "Reference" "QR-Code1" (at 45.72 233.68 0)
       (effects (font (size 1.27 1.27)) (justify left))
     )
@@
       (project "OpenHW DevKit"
         (path "/b0906e10-2fbc-4309-a8b4-6fc4cd1a5490"
-          (reference "QR-Code") (unit 1)
+          (reference "QR-Code1") (unit 1)
         )
       )
