File: power.kicad_sch (KiCad schematic)
At the start: 1 part, among them J6 Barrel_Jack

Commit message: updates to the images and place holders for MCU footprint
Parts:
- added C26, C27, C28, C29, C30, C31, C32, C33: 1uF, Capacitor_SMD:C_0603_1608Metric, symbol Device:C_Small
- added D8: BAT760-7, Diode_SMD:SOD2513X120N, symbol bat760:BAT760-7
- added D9: MMBD4448HADW, Package_TO_SOT_SMD:SOT-363_SC-70-6, symbol Diode:MMBD4448HADW
- added U10: TLV71209_SOT23-5, Package_TO_SOT_SMD:SOT-23-5, symbol Regulator_Linear:TLV71209_SOT23-5
- added U11: LM1117-5.0, Package_TO_SOT_SMD:SOT-223-3_TabPin2, symbol Regulator_Linear:LM1117-5.0
- added U8: LM1117-3.3, Package_TO_SOT_SMD:SOT-223-3_TabPin2, symbol Regulator_Linear:LM1117-3.3
- added U9: LM1117-1.8, Package_TO_SOT_SMD:SOT-223-3_TabPin2, symbol Regulator_Linear:LM1117-1.8
Connections:
- net at J6.1: now also D8.A
- net GND: now reaches J6.2
- net GND: now also C26.2, C27.2, C28.2, C29.2, C30.2, C31.2, C32.2, C33.2, U10.2 (GND), U11.1 (GND), U8.1 (GND), U9.1 (GND)
- new net: C32.1, D8.C, D9.1 (K), U11.3 (VI)
- new net +1V8: C30.1, D9.3 (A), U9.2 (VO)
- new net +3V3: C28.1, C29.1, D9.4 (K), D9.6 (A), U10.1 (IN), U10.3 (EN), U8.2 (VO)
- new net +5V: C26.1, C27.1, C33.1, D9.2 (K), D9.5 (K), D9.6 (A), U11.2 (VO), U8.3 (VI), U9.3 (VI)
- new net 0.9V: C31.1, D9.3 (A), U10.5 (OUT)
Other:
- moved on the sheet: J6

Commit message: added solderpad license text to each sheet
Other:
- note added: "Copyright and related rights are licensed under the Solderpad Hardware License, Version 0.51 (the "License"); you may not use this file except in compliance with the License. You may obtain a copy of the License at http://solderpad.org/licenses/SHL-0.51. Unless required by applicable law or agreed to in writing, software, hardware and materials distributed under this License is distributed on an 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"
Changed lines of the file:
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@@
     (effects (font (size 1.27 1.27)) (justify left bottom))
+  )
+  (text "Copyright and related rights are licensed under the Solderpad Hardware License, Version 0.51 (the \"License\");\nyou may not use this file except in compliance with the License.  You may obtain a copy of the License at\nhttp://solderpad.org/licenses/SHL-0.51. Unless required by applicable law or agreed to in writing, software,\nhardware and materials distributed under this License is distributed on an \"AS IS\" BASIS, WITHOUT WARRANTIES OR\nCONDITIONS OF ANY KIND, either express or implied. See the License for the specific language governing\npermissions and limitations under the License.\n"
+    (at 179.07 179.07 0)
+    (effects (font (size 1 1)) (justify left bottom))
   )
   (global_label "0.9V" (shape input) (at 172.72 133.35 0) (fields_autoplaced)

Commit message: added the camera, temperature sensor and basic MCU symbol
Parts:
- removed C32, C33: 1uF, Capacitor_SMD:C_0603_1608Metric, symbol Device:C_Small
- removed D8: BAT760-7, Diode_SMD:SOD2513X120N, symbol bat760:BAT760-7
- removed unit 1 of D9
- removed J6: Barrel_Jack, Connector_BarrelJack:BarrelJack_CLIFF_FC681465S_SMT_Horizontal, symbol Connector:Barrel_Jack
- removed U11: LM1117-5.0, Package_TO_SOT_SMD:SOT-223-3_TabPin2, symbol Regulator_Linear:LM1117-5.0
Other:
- note added: "5v input from USB-C 3.3v, 1.8v, 0.9v outputs"
- note added: "Copyright and related rights are licensed under the Solderpad Hardware License, Version 2.1 (the "License"); you may not use this file except in compliance with the License. You may obtain a copy of the License at http://solderpad.org/licenses/SHL-2.1. Unless required by applicable law or agreed to in writing, software, hardware and materials distributed under this License is distributed on an "A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"
- note removed: "5v input from USB-C 6-12v input from 2.1mm Barrel 3.3v, 1.8v, 0.9v outputs"
- note removed: "Copyright and related rights are licensed under the Solderpad Hardware License, Version 0.51 (the "License"); you may not use this file except in compliance with the License. You may obtain a copy of the License at http://solderpad.org/licenses/SHL-0.51. Unless required by applicable law or agreed to in writing, software, hardware and materials distributed under this License is distributed on an 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"

Commit message: Power and Level Shifter updates
Parts:
- removed C26, C27, C28, C29, C30, C31: 1uF, Capacitor_SMD:C_0603_1608Metric, symbol Device:C_Small
- removed D9: MMBD4448HADW, Package_TO_SOT_SMD:SOT-363_SC-70-6, symbol Diode:MMBD4448HADW
- removed U10: TLV71209_SOT23-5, Package_TO_SOT_SMD:SOT-23-5, symbol Regulator_Linear:TLV71209_SOT23-5
- removed U8: LM1117-3.3, Package_TO_SOT_SMD:SOT-223-3_TabPin2, symbol Regulator_Linear:LM1117-3.3
- removed U9: LM1117-1.8, Package_TO_SOT_SMD:SOT-223-3_TabPin2, symbol Regulator_Linear:LM1117-1.8
- added C? (x3): 10uF, Capacitor_SMD:C_0603_1608Metric, symbol Device:C_Small
- added C? (x9): 22uF, symbol Device:C_Small
- added C? (x3): 100nF, Capacitor_SMD:C_0201_0603Metric, symbol Device:C_Small
- added L? (x3): 3.3uH, Inductor_SMD:L_Bourns-SRN4018, symbol pspice:INDUCTOR
- added R?: 31k, Resistor_SMD:R_0603_1608Metric, symbol Device:R_Small
- added R?: 13k, Resistor_SMD:R_0603_1608Metric, symbol Device:R_Small
- added R? (x2): 10k, Resistor_SMD:R_0603_1608Metric, symbol Device:R_Small
- added U? (x3): AP62300Z6, Package_TO_SOT_SMD:SOT-563, symbol Regulator_Switching:AP62300Z6
Connections:
- net +1V8: now also C?.1, C?.1, C?.1, L?.2, R?.1
- net +3V3: now also C?.1, C?.1, C?.1, L?.2, R?.1
- net +5V: now also C?.1, C?.1, C?.1, C?.1, C?.1, C?.1, U?.1 (VIN), U?.1 (VIN), U?.1 (VIN)
- net GND: now also C?.2, C?.2, C?.2, C?.2, C?.2, C?.2, C?.2, C?.2, C?.2, C?.2, C?.2, C?.2, R?.2, R?.2, U?.3 (GND), U?.3 (GND), U?.3 (GND)
- new net: R?.1, R?.2, U?.6 (FB) (x2)
- new net: L?.1, U?.4 (BST) (x3)
- new net: C?.2, U?.2 (SW) (x3)
- new net +0V8: C?.1, C?.1, C?.1, L?.2, U?.6 (FB)
Other:
- note added: "5v input from USB-C 3.3v, 1.8v, 0.8v outputs"
- note removed: "5v input from USB-C 3.3v, 1.8v, 0.9v outputs"

Commit message: updates to the footprints
Parts:
- C72, C73, C74: renamed from C?; footprint Capacitor_SMD:C_0201_0603Metric -> Capacitor_SMD:C_0603_1608Metric
- C75, C76, C77, C78, C79, C80, C81, C82, C83: renamed from C?; footprint (none) -> Capacitor_SMD:C_0603_1608Metric
- gave numbers to parts that had none: 13

Commit message: Changed to KiCAD 7 and updated to final pinout.
Parts:
- added TP2: 5v0, TestPoint:TestPoint_Loop_D2.54mm_Drill1.5mm_Beaded, symbol Connector:TestPoint
- added TP3: 3v3, TestPoint:TestPoint_Loop_D2.54mm_Drill1.5mm_Beaded, symbol Connector:TestPoint
- added TP4: 1v8, TestPoint:TestPoint_Loop_D2.54mm_Drill1.5mm_Beaded, symbol Connector:TestPoint
- added TP5: 0v8, TestPoint:TestPoint_Loop_D2.54mm_Drill1.5mm_Beaded, symbol Connector:TestPoint
- added TP6: GND, TestPoint:TestPoint_Loop_D2.54mm_Drill1.5mm_Beaded, symbol Connector:TestPoint
Connections:
- net +0V8: now also TP5.1
- net +1V8: now also TP4.1
- net +3V3: now also TP3.1
- net +5V: now also TP2.1
- net GND: now also TP6.1

Commit message: reset supervisor replacement and DRC cleanup
Parts:
- added C21, C22, C23: 150pF, Capacitor_SMD:C_0603_1608Metric, symbol Device:C_Small
- added R34: 65k, Resistor_SMD:R_0603_1608Metric, symbol Device:R_Small
- added R35, R37, R39: 10k, Resistor_SMD:R_0603_1608Metric, symbol Device:R_Small
- added R36: 32.5k, Resistor_SMD:R_0603_1608Metric, symbol Device:R_Small
- added R38: 7.5k, Resistor_SMD:R_0603_1608Metric, symbol Device:R_Small
- added U5 (x3): MP6400DG-01-LF-Z, QFN6_MP6400_MNP, symbol MP6400:MP6400DG-01-LF-Z
Connections:
- net +0V8: now also R38.1, U5.1 (VCC)
- net +1V8: now also R36.1, U5.1 (VCC)
- net +3V3: now also R34.1, U5.1 (VCC)
- net GND: now also C21.2, C22.2, C23.2, R35.2, R37.2, R39.2, U5.5 (GND), U5.5 (GND), U5.5 (GND), U5.7 (EPAD), U5.7 (EPAD), U5.7 (EPAD)
- new net: R38.2, R39.1, U5.2 (SENSE)
- new net: C23.1, U5.3 (CDELAY)
- new net: U5.4 (*MR), U5.6 (*RESET) (x2)
- new net: R36.2, R37.1, U5.2 (SENSE)
- new net: C22.1, U5.3 (CDELAY)
- new net: R34.2, R35.1, U5.2 (SENSE)
- new net: C21.1, U5.3 (CDELAY)
- new net ~{RESET_IN}: U5.4 (*MR)
- new net ~{RESET_OUT}: U5.6 (*RESET)
Other:
- note added: "All three voltages must be above their thresholds to release the RESET"
- note removed: "5v input from USB-C 3.3v, 1.8v, 0.8v outputs"
- moved on the sheet: C69, C70, C71, C72, C73, C74, C75, C76, C77, C78, C79, C80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

Commit message: updated pinout changes
Connections:
- net +0V8: no longer U5.1 (VCC)
- net +1V8: now also U5.1 (VCC)
Changed lines of the file:
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@@
   (junction (at 49.53 74.93) (diameter 0) (color 0 0 0 0)
   )
-  (junction (at 49.53 113.03) (diameter 0) (color 0 0 0 0)
-  )
   (junction (at 227.33 45.72) (diameter 0) (color 0 0 0 0)
   )
@@
     (stroke (width 0) (type default))
   )
-  (wire (pts (xy 49.53 113.03) (xy 58.42 113.03))
-    (stroke (width 0) (type default))
-  )
   (wire (pts (xy 109.22 119.38) (xy 113.03 119.38))
     (stroke (width 0) (type default))
@@
     (stroke (width 0) (type default))
   )
-  (wire (pts (xy 58.42 113.03) (xy 58.42 116.84))
+  (wire (pts (xy 58.42 111.76) (xy 58.42 116.84))
     (stroke (width 0) (type default))
   )
@@
         )
       )
+    )
+  )
+  (symbol (lib_id "power:+1V8") (at 58.42 111.76 0) (unit 1)
+    (in_bom yes) (on_board yes) (dnp no) (fields_autoplaced)
+    (property "Reference" "#PWR066" (at 58.42 115.57 0)
+      (effects (font (size 1.27 1.27)) hide)
+    )
+    (property "Value" "+1V8" (at 58.42 108.1842 0)
+      (effects (font (size 1.27 1.27)))
+    )
+    (property "Footprint" "" (at 58.42 111.76 0)
+      (effects (font (size 1.27 1.27)) hide)
+    )
+    (property "Datasheet" "" (at 58.42 111.76 0)
+      (effects (font (size 1.27 1.27)) hide)
+    )
+    (pin "1")
+    (instances
+      (project "OpenHW DevKit"
+        (path "/b0906e10-2fbc-4309-a8b4-6fc4cd1a5490/1d35af67-6e7f-4e50-89d3-ea3f7dca4687"
+          (reference "#PWR066") (unit 1)
+        )
+      )
