File: power.kicad_sch (KiCad schematic)
At the start: 42 parts, among them U23 AP62300Z6, U24 AP62300Z6, U25 AP62300Z6, U5 MP6400DG-01-LF-Z

Commit message: updated the QR code and added shield coupling to the usb connector
Other:
- moved on the sheet: C21, C22, C23, R34, R35, R36, R37, R38, R39, U5

Commit message: updated footprints, added the barrel power connector and test points
Parts:
- added D11: BAT760-7, diode:Diodes-SOD323-03_2017-0-0, symbol diode:BAT760-7
- added J12: PJ-002B, CUI_PJ-002B, symbol barrel:PJ-002B
- TP2: value 5v0 -> Vdc
- U? (x3): renamed from U5; footprint QFN6_MP6400_MNP -> MP6400:QFN6_MP6400_MNP
Connections:
- net GND: now also J12.2
- net +5V renamed +VDC
- net +VDC: now also D11.1 (CATHODE)
- new net: D11.2 (ANODE), J12.1
Other:
- moved on the sheet: TP2, TP3, TP4, TP5, TP6
