File: expresslink.kicad_sch (KiCad schematic)
At the start: 10 parts, among them J1 Conn_02x05_Odd_Even, J2 Conn_02x03_Odd_Even, U1 ESP32-C3-MINI-1, Y1 32.768kHz

Commit message: updates to the images and place holders for MCU footprint
Parts:
- added C34: 10uF, Capacitor_SMD:C_0603_1608Metric_Pad1.08x0.95mm_HandSolder, symbol Device:C_Small
- added R10: 1M, Resistor_SMD:R_0603_1608Metric_Pad0.98x0.95mm_HandSolder, symbol Device:R
Connections:
- net GND: now also C34.2
- net ~{EL_RESET}: now also C34.1
- net at C1.1, U1.12 (GPIO0/ADC1_CH0/XTAL_32K_P), Y1.1: now also R10.1
- net at C2.1, U1.13 (GPIO1/ADC1_CH1/XTAL_32K_N), Y1.2: now also R10.2
Other:
- moved on the sheet: C1, C2, C3, C4, R1, Y1

Commit message: added solderpad license text to each sheet
Other:
- note added: "Copyright and related rights are licensed under the Solderpad Hardware License, Version 0.51 (the "License"); you may not use this file except in compliance with the License. You may obtain a copy of the License at http://solderpad.org/licenses/SHL-0.51. Unless required by applicable law or agreed to in writing, software, hardware and materials distributed under this License is distributed on an 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"
Changed lines of the file:
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@@
     (stroke (width 0) (type default) (color 0 0 0 0))
+  )
+  (text "Copyright and related rights are licensed under the Solderpad Hardware License, Version 0.51 (the \"License\");\nyou may not use this file except in compliance with the License.  You may obtain a copy of the License at\nhttp://solderpad.org/licenses/SHL-0.51. Unless required by applicable law or agreed to in writing, software,\nhardware and materials distributed under this License is distributed on an \"AS IS\" BASIS, WITHOUT WARRANTIES OR\nCONDITIONS OF ANY KIND, either express or implied. See the License for the specific language governing\npermissions and limitations under the License.\n"
+    (at 180.34 177.8 0)
+    (effects (font (size 1 1)) (justify left bottom))
   )
   (text "ExpressLink" (at 139.7 43.18 0)

Commit message: added the camera, temperature sensor and basic MCU symbol
Other:
- note added: "AWS IoT ExpressLink"
- note added: "Copyright and related rights are licensed under the Solderpad Hardware License, Version 2.1 (the "License"); you may not use this file except in compliance with the License. You may obtain a copy of the License at http://solderpad.org/licenses/SHL-2.1. Unless required by applicable law or agreed to in writing, software, hardware and materials distributed under this License is distributed on an "A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"
- note removed: "Copyright and related rights are licensed under the Solderpad Hardware License, Version 0.51 (the "License"); you may not use this file except in compliance with the License. You may obtain a copy of the License at http://solderpad.org/licenses/SHL-0.51. Unless required by applicable law or agreed to in writing, software, hardware and materials distributed under this License is distributed on an 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"
- note removed: "ExpressLink"
Changed lines of the file:
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@@
     (stroke (width 0) (type default) (color 0 0 0 0))
   )
-  (text "Copyright and related rights are licensed under the Solderpad Hardware License, Version 0.51 (the \"License\");\nyou may not use this file except in compliance with the License.  You may obtain a copy of the License at\nhttp://solderpad.org/licenses/SHL-0.51. Unless required by applicable law or agreed to in writing, software,\nhardware and materials distributed under this License is distributed on an \"AS IS\" BASIS, WITHOUT WARRANTIES OR\nCONDITIONS OF ANY KIND, either express or implied. See the License for the specific language governing\npermissions and limitations under the License.\n"
+  (text "Copyright and related rights are licensed under the Solderpad Hardware License, Version 2.1 (the \"License\");\nyou may not use this file except in compliance with the License.  You may obtain a copy of the License at\nhttp://solderpad.org/licenses/SHL-2.1. Unless required by applicable law or agreed to in writing, software,\nhardware and materials distributed under this License is distributed on an \"AS IS\" BASIS, WITHOUT WARRANTIES OR\nCONDITIONS OF ANY KIND, either express or implied. See the License for the specific language governing\npermissions and limitations under the License.\n"
     (at 180.34 177.8 0)
     (effects (font (size 1 1)) (justify left bottom))
   )
-  (text "ExpressLink" (at 139.7 43.18 0)
+  (text "AWS IoT ExpressLink" (at 152.4 45.72 0)
     (effects (font (size 1.27 1.27)) (justify left bottom))
   )

Commit message: updates to the footprints
Parts:
- C1, C2, C3, C34, C4: footprint Capacitor_SMD:C_0603_1608Metric_Pad1.08x0.95mm_HandSolder -> Capacitor_SMD:C_0603_1608Metric
Changed lines of the file:
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@@
     (property "Reference" "C1" (id 0) (at 81.28 99.06 90))
     (property "Value" "12.5pF" (id 1) (at 81.28 100.33 90))
-    (property "Footprint" "Capacitor_SMD:C_0603_1608Metric_Pad1.08x0.95mm_HandSolder" (id 2) (at 81.28 102.87 0)
+    (property "Footprint" "Capacitor_SMD:C_0603_1608Metric" (id 2) (at 81.28 102.87 0)
       (effects (font (size 1.27 1.27)) hide)
     )
@@
     (property "Reference" "C2" (id 0) (at 81.28 115.57 90))
     (property "Value" "12.5pF" (id 1) (at 81.28 113.03 90))
-    (property "Footprint" "Capacitor_SMD:C_0603_1608Metric_Pad1.08x0.95mm_HandSolder" (id 2) (at 81.28 110.49 0)
+    (property "Footprint" "Capacitor_SMD:C_0603_1608Metric" (id 2) (at 81.28 110.49 0)
       (effects (font (size 1.27 1.27)) hide)
     )
@@
       (effects (font (size 1.27 1.27)) (justify right))
     )
-    (property "Footprint" "Capacitor_SMD:C_0603_1608Metric_Pad1.08x0.95mm_HandSolder" (id 2) (at 123.19 38.1 0)
+    (property "Footprint" "Capacitor_SMD:C_0603_1608Metric" (id 2) (at 123.19 38.1 0)
       (effects (font (size 1.27 1.27)) hide)
     )
@@
       (effects (font (size 1.27 1.27)) (justify right))
     )
-    (property "Footprint" "Capacitor_SMD:C_0603_1608Metric_Pad1.08x0.95mm_HandSolder" (id 2) (at 114.3 38.1 0)
+    (property "Footprint" "Capacitor_SMD:C_0603_1608Metric" (id 2) (at 114.3 38.1 0)
       (effects (font (size 1.27 1.27)) hide)
     )
@@
       (effects (font (size 1.27 1.27)) (justify right))
     )
-    (property "Footprint" "Capacitor_SMD:C_0603_1608Metric_Pad1.08x0.95mm_HandSolder" (id 2) (at 107.95 60.96 0)
-      (effects (font (size 1.27 1.27)) hide)
-    )
+    (property "Footprint" "Capacitor_SMD:C_0603_1608Metric" (id 2) (at 107.95 60.96 0)
+      (effects (font (size 1.27 1.27)) hide)
+    )

Commit message: Changed to KiCAD 7 and updated to final pinout.
Parts:
- C34: value 10uF -> 100nF

Commit message: updated 3d models and cleaned up the DRC
Parts:
- U1: footprint Espressif:ESP32-C3-MINI-1 -> espressif:ESP32-C3-MINI-1
Changed lines of the file:
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@@
       (effects (font (size 1.27 1.27)))
     )
-    (property "Footprint" "Espressif:ESP32-C3-MINI-1" (at 161.29 116.84 0)
+    (property "Footprint" "espressif:ESP32-C3-MINI-1" (at 161.29 116.84 0)
       (effects (font (size 1.27 1.27)) hide)
     )
