File: camera.kicad_sch (KiCad schematic)
At the start: 4 parts, among them J6 Conn_01x24, U12 AP2127K-2.8

Commit message: updated the graphics and moved files around for neatness
Parts:
- J6: symbol Connector_Generic:Conn_01x24 -> Connector_Generic_MountingPin:Conn_01x24_MountingPin
Connections:
- net GND: now also J6.MP (MountPin)
Changed lines of the file:
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@@
+    )
+  )
+  (symbol (lib_id "power:GND") (at 162.56 129.54 0) (unit 1)
+    (in_bom yes) (on_board yes) (dnp no) (fields_autoplaced)
+    (property "Reference" "#PWR0117" (at 162.56 135.89 0)
+      (effects (font (size 1.27 1.27)) hide)
+    )
+    (property "Value" "GND" (at 162.56 133.9834 0)
+      (effects (font (size 1.27 1.27)))
+    )
+    (property "Footprint" "" (at 162.56 129.54 0)
+      (effects (font (size 1.27 1.27)) hide)
+    )
+    (property "Datasheet" "" (at 162.56 129.54 0)
+      (effects (font (size 1.27 1.27)) hide)
+    )
+    (pin "1")
+    (instances
+      (project "OpenHW DevKit"
+        (path "/b0906e10-2fbc-4309-a8b4-6fc4cd1a5490/de268494-d8df-4048-8e82-8343b42749bc"
+          (reference "#PWR0117") (unit 1)
+        )
+      )
     )
   )
@@
     )
   )
-  (symbol (lib_id "Connector_Generic:Conn_01x24") (at 162.56 93.98 0) (unit 1)
+  (symbol (lib_id "Connector_Generic_MountingPin:Conn_01x24_MountingPin") (at 162.56 93.98 0) (unit 1)
     (in_bom yes) (on_board yes) (dnp no) (fields_autoplaced)
     (property "Reference" "J6" (at 164.592 94.4153 0)
@@
     (pin "8")
     (pin "9")
+    (pin "MP")
     (instances
       (project "OpenHW DevKit"
