File: kicad/OpenHW DevKit.kicad_sch (KiCad schematic)
At the start: 132 parts, among them J10 Conn_01x20, J4 Conn_01x02_Male, J7 Conn_01x20, J8 Conn_01x20, J9 Conn_01x20, Q1 MMBT3904, Q2 MMBT3904, SW1 SW_Push, SW2 SW_Push, U14 CORE-V-MCU, U3 W25Q32JWZP, U4 FXMA2102UMX, U6 NTB0104BQ,115, U7 NTB0104BQ,115, U8 NTB0104BQ,115, U9 NTB0104BQ,115, X1 ECS-2520MVLC-100-CN

Commit message: Corections made after testing V1
Parts:
- removed C24, C25: 100nF, Capacitor_SMD:C_0603_1608Metric, symbol Device:C_Small
Connections:
- net +0V8: no longer U14.B5 (AVDD)
- net +1V8: now also U14.B5 (AVDD); no longer JP2.1 (A), JP8.1 (A)
- net GND: now also JP2.1 (A), JP8.1 (A)
Other:
- moved on the sheet: R40, SW2

Commit message: changes to the power supply and minor edits to the silkscreen
Connections:
- net +0V8: no longer J8.5 (Pin_5)
- net +1V8: now also J8.5 (Pin_5)
Changed lines of the file:
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@@
-    )
-  )
-  (symbol (lib_id "power:+0V8") (at 279.4 107.95 270) (unit 1)
-    (in_bom yes) (on_board yes) (dnp no)
-    (property "Reference" "#PWR0115" (at 275.59 107.95 0)
-      (effects (font (size 1.27 1.27)) hide)
-    )
-    (property "Value" "+0V8" (at 282.575 108.2668 90)
-      (effects (font (size 1.27 1.27)) (justify left))
-    )
-    (property "Footprint" "" (at 279.4 107.95 0)
-      (effects (font (size 1.27 1.27)) hide)
-    )
-    (property "Datasheet" "" (at 279.4 107.95 0)
-      (effects (font (size 1.27 1.27)) hide)
-    )
-    (pin "1")
-    (instances
-      (project "OpenHW DevKit"
-        (path "/b0906e10-2fbc-4309-a8b4-6fc4cd1a5490"
-          (reference "#PWR0115") (unit 1)
-        )
-      )
     )
   )
@@
         )
       )
+    )
+  )
+  (symbol (lib_id "power:+1V8") (at 279.4 107.95 270) (unit 1)
+    (in_bom yes) (on_board yes) (dnp no) (fields_autoplaced)
+    (property "Reference" "#PWR086" (at 275.59 107.95 0)
+      (effects (font (size 1.27 1.27)) hide)
+    )
+    (property "Value" "+1V8" (at 282.575 108.2668 90)
+      (effects (font (size 1.27 1.27)) (justify left))
+    )
+    (property "Footprint" "" (at 279.4 107.95 0)
+      (effects (font (size 1.27 1.27)) hide)
+    )
+    (property "Datasheet" "" (at 279.4 107.95 0)
+      (effects (font (size 1.27 1.27)) hide)
+    )
+    (pin "1")
+    (instances
+      (project "OpenHW DevKit"
+        (path "/b0906e10-2fbc-4309-a8b4-6fc4cd1a5490"
+          (reference "#PWR086") (unit 1)
+        )
+      )
